File: sonar-v1-pcb/sonar.kicad_pcb (KiCad board)
At the start: 2 copper layers, 17 parts

Commit message: ragebait
Parts:
- added C1: 100nF, Capacitor_SMD:C_0402_1005Metric, F.Cu at (86.5, 73.0)
- added C10: 2.2nF, Capacitor_SMD:C_0402_1005Metric, F.Cu at (247.8, 79.6)
- added C11: 100nF, Capacitor_SMD:C_0402_1005Metric, F.Cu at (215.1, 91.5)
- added C12: 2.2nF, Capacitor_SMD:C_0402_1005Metric, F.Cu at (215.1, 93.5)
- added C13: 100nF, Capacitor_SMD:C_0402_1005Metric, F.Cu at (231.5, 77.6)
- added C14: 2.2nF, Capacitor_SMD:C_0402_1005Metric, F.Cu at (231.5, 79.6)
- added C15: 100nF, Capacitor_SMD:C_0402_1005Metric, F.Cu at (231.5, 91.5)
- added C16: 2.2nF, Capacitor_SMD:C_0402_1005Metric, F.Cu at (231.5, 93.5)
- added C17: 100nF, Capacitor_SMD:C_0402_1005Metric, F.Cu at (182.4, 63.7)
- added C18: 2.2nF, Capacitor_SMD:C_0402_1005Metric, F.Cu at (182.4, 65.7)
- added C19: 100nF, Capacitor_SMD:C_0402_1005Metric, F.Cu at (198.8, 49.8)
- added C2: 2.2nF, Capacitor_SMD:C_0402_1005Metric, F.Cu at (82.0, 78.5)
- added C20: 2.2nF, Capacitor_SMD:C_0402_1005Metric, F.Cu at (198.8, 51.8)
- added C21: 100nF, Capacitor_SMD:C_0402_1005Metric, F.Cu at (198.8, 63.7)
- added C22: 2.2nF, Capacitor_SMD:C_0402_1005Metric, F.Cu at (198.8, 65.7)
- added C23: 100nF, Capacitor_SMD:C_0402_1005Metric, F.Cu at (182.4, 91.5)
- added C24: 2.2nF, Capacitor_SMD:C_0402_1005Metric, F.Cu at (182.4, 93.5)
- added C25: 100nF, Capacitor_SMD:C_0402_1005Metric, F.Cu at (182.4, 49.8)
- added C26: 2.2nF, Capacitor_SMD:C_0402_1005Metric, F.Cu at (182.4, 51.8)
- added C27: 100nF, Capacitor_SMD:C_0402_1005Metric, F.Cu at (182.4, 77.6)
- added C28: 2.2nF, Capacitor_SMD:C_0402_1005Metric, F.Cu at (182.4, 79.6)
- added C29: 100nF, Capacitor_SMD:C_0402_1005Metric, F.Cu at (182.4, 105.4)
- added C3: 100nF, Capacitor_SMD:C_0402_1005Metric, F.Cu at (247.8, 63.7)
- added C30: 2.2nF, Capacitor_SMD:C_0402_1005Metric, F.Cu at (182.4, 107.4)
- added C31: 100nF, Capacitor_SMD:C_0402_1005Metric, F.Cu at (231.5, 63.7)
- added C32: 2.2nF, Capacitor_SMD:C_0402_1005Metric, F.Cu at (231.5, 65.7)
- added C33: 100nF, Capacitor_SMD:C_0402_1005Metric, F.Cu at (198.8, 77.6)
- added C34: 2.2nF, Capacitor_SMD:C_0402_1005Metric, F.Cu at (198.8, 79.6)
- added C35: 100nF, Capacitor_SMD:C_0402_1005Metric, F.Cu at (247.8, 49.8)
- added C36: 2.2nF, Capacitor_SMD:C_0402_1005Metric, F.Cu at (247.8, 51.8)
- added C37: 100nF, Capacitor_SMD:C_0402_1005Metric, F.Cu at (231.5, 49.8)
- added C38: 2.2nF, Capacitor_SMD:C_0402_1005Metric, F.Cu at (231.5, 51.8)
- added C39: 100nF, Capacitor_SMD:C_0402_1005Metric, F.Cu at (198.8, 105.4)
- added C4: 2.2nF, Capacitor_SMD:C_0402_1005Metric, F.Cu at (247.8, 65.7)
- added C40: 2.2nF, Capacitor_SMD:C_0402_1005Metric, F.Cu at (198.8, 107.4)
- added C41: 100nF, Capacitor_SMD:C_0402_1005Metric, F.Cu at (231.8, 33.4)
- added C42: 2.2nF, Capacitor_SMD:C_0402_1005Metric, F.Cu at (231.8, 35.4)
- added C43: 100nF, Capacitor_SMD:C_0402_1005Metric, F.Cu at (198.8, 91.5)
- added C44: 2.2nF, Capacitor_SMD:C_0402_1005Metric, F.Cu at (198.8, 93.5)
- added C45: 100nF, Capacitor_SMD:C_0402_1005Metric, F.Cu at (215.1, 63.7)
- added C46: 2.2nF, Capacitor_SMD:C_0402_1005Metric, F.Cu at (215.1, 65.7)
- added C47: 100nF, Capacitor_SMD:C_0402_1005Metric, F.Cu at (215.1, 49.8)
- added C48: 2.2nF, Capacitor_SMD:C_0402_1005Metric, F.Cu at (215.1, 51.8)
- added C5: 100nF, Capacitor_SMD:C_0402_1005Metric, F.Cu at (215.1, 77.6)
- added C6: 2.2nF, Capacitor_SMD:C_0402_1005Metric, F.Cu at (215.1, 79.6)
- added C7: 100nF, Capacitor_SMD:C_0402_1005Metric, F.Cu at (215.1, 105.4)
- added C8: 2.2nF, Capacitor_SMD:C_0402_1005Metric, F.Cu at (215.1, 107.4)
- added C9: 100nF, Capacitor_SMD:C_0402_1005Metric, F.Cu at (247.8, 77.6)
- added MK1: Microphone_Ultrasound, Sonar:MA40S4, F.Cu at (71.0, 77.1)
- added MK10: Microphone_Ultrasound, Sonar:MA40S4, F.Cu at (191.6, 46.6)
- added MK11: Microphone_Ultrasound, Sonar:MA40S4, F.Cu at (191.6, 60.5)
- added MK12: Microphone_Ultrasound, Sonar:MA40S4, F.Cu at (175.2, 88.3)
- added MK13: Microphone_Ultrasound, Sonar:MA40S4, F.Cu at (175.2, 46.6)
- added MK14: Microphone_Ultrasound, Sonar:MA40S4, F.Cu at (175.2, 74.4)
- added MK15: Microphone_Ultrasound, Sonar:MA40S4, F.Cu at (175.2, 102.2)
- added MK16: Microphone_Ultrasound, Sonar:MA40S4, F.Cu at (224.3, 60.5)
- added MK17: Microphone_Ultrasound, Sonar:MA40S4, F.Cu at (191.6, 74.4)
- added MK18: Microphone_Ultrasound, Sonar:MA40S4, F.Cu at (240.7, 46.6)
- added MK19: Microphone_Ultrasound, Sonar:MA40S4, F.Cu at (224.3, 46.6)
- added MK2: Microphone_Ultrasound, Sonar:MA40S4, F.Cu at (240.7, 60.5)
- added MK20: Microphone_Ultrasound, Sonar:MA40S4, F.Cu at (191.6, 102.2)
- added MK21: Microphone_Ultrasound, Sonar:MA40S4, F.Cu at (224.6, 30.2)
- added MK22: Microphone_Ultrasound, Sonar:MA40S4, F.Cu at (191.6, 88.3)
- added MK23: Microphone_Ultrasound, Sonar:MA40S4, F.Cu at (208.0, 60.5)
- added MK24: Microphone_Ultrasound, Sonar:MA40S4, F.Cu at (71.0, 91.0)
- added MK24: Microphone_Ultrasound, Sonar:MA40S4, F.Cu at (208.0, 46.6)
- added MK3: Microphone_Ultrasound, Sonar:MA40S4, F.Cu at (208.0, 74.4)
- added MK4: Microphone_Ultrasound, Sonar:MA40S4, F.Cu at (208.0, 102.2)
- added MK5: Microphone_Ultrasound, Sonar:MA40S4, F.Cu at (240.7, 74.4)
- added MK6: Microphone_Ultrasound, Sonar:MA40S4, F.Cu at (208.0, 88.3)
- added MK7: Microphone_Ultrasound, Sonar:MA40S4, F.Cu at (224.3, 74.4)
- added MK8: Microphone_Ultrasound, Sonar:MA40S4, F.Cu at (224.3, 88.3)
- added MK9: Microphone_Ultrasound, Sonar:MA40S4, F.Cu at (175.2, 60.5)
- added R1: 1M, Resistor_SMD:R_0402_1005Metric, F.Cu at (82.0, 73.0)
- added R10: 10k, Resistor_SMD:R_0402_1005Metric, F.Cu at (215.2, 71.7)
- added R11: 290k, Resistor_SMD:R_0402_1005Metric, F.Cu at (215.2, 73.7)
- added R12: 1k, Resistor_SMD:R_0402_1005Metric, F.Cu at (215.2, 75.7)
- added R13: 1M, Resistor_SMD:R_0402_1005Metric, F.Cu at (215.2, 97.5)
- added R14: 10k, Resistor_SMD:R_0402_1005Metric, F.Cu at (215.2, 99.5)
- added R15: 290k, Resistor_SMD:R_0402_1005Metric, F.Cu at (215.2, 101.5)
- added R16: 1k, Resistor_SMD:R_0402_1005Metric, F.Cu at (215.2, 103.5)
- added R17: 1M, Resistor_SMD:R_0402_1005Metric, F.Cu at (247.9, 69.7)
- added R18: 10k, Resistor_SMD:R_0402_1005Metric, F.Cu at (247.9, 71.7)
- added R19: 290k, Resistor_SMD:R_0402_1005Metric, F.Cu at (247.9, 73.7)
- added R2: 10k, Resistor_SMD:R_0402_1005Metric, F.Cu at (82.0, 68.0)
- added R20: 1k, Resistor_SMD:R_0402_1005Metric, F.Cu at (247.9, 75.7)
- added R21: 1M, Resistor_SMD:R_0402_1005Metric, F.Cu at (215.2, 83.6)
- added R22: 10k, Resistor_SMD:R_0402_1005Metric, F.Cu at (215.2, 85.6)
- added R23: 290k, Resistor_SMD:R_0402_1005Metric, F.Cu at (215.2, 87.6)
- added R24: 1k, Resistor_SMD:R_0402_1005Metric, F.Cu at (215.2, 89.6)
- added R25: 1M, Resistor_SMD:R_0402_1005Metric, F.Cu at (231.5, 69.7)
- added R26: 10k, Resistor_SMD:R_0402_1005Metric, F.Cu at (231.5, 71.7)
- added R27: 290k, Resistor_SMD:R_0402_1005Metric, F.Cu at (231.5, 73.7)
- added R28: 1k, Resistor_SMD:R_0402_1005Metric, F.Cu at (231.5, 75.7)
- added R29: 1M, Resistor_SMD:R_0402_1005Metric, F.Cu at (231.5, 83.6)
- added R3: 290k, Resistor_SMD:R_0402_1005Metric, F.Cu at (86.0, 68.0)
- added R30: 10k, Resistor_SMD:R_0402_1005Metric, F.Cu at (231.5, 85.6)
- added R31: 290k, Resistor_SMD:R_0402_1005Metric, F.Cu at (231.5, 87.6)
- added R32: 1k, Resistor_SMD:R_0402_1005Metric, F.Cu at (231.5, 89.6)
- added R33: 1M, Resistor_SMD:R_0402_1005Metric, F.Cu at (182.4, 55.8)
- added R34: 10k, Resistor_SMD:R_0402_1005Metric, F.Cu at (182.4, 57.8)
- added R35: 290k, Resistor_SMD:R_0402_1005Metric, F.Cu at (182.4, 59.8)
- added R36: 1k, Resistor_SMD:R_0402_1005Metric, F.Cu at (182.4, 61.8)
- added R37: 1M, Resistor_SMD:R_0402_1005Metric, F.Cu at (198.8, 41.9)
- added R38: 10k, Resistor_SMD:R_0402_1005Metric, F.Cu at (198.8, 43.9)
- added R39: 290k, Resistor_SMD:R_0402_1005Metric, F.Cu at (198.8, 45.9)
- added R4: 1k, Resistor_SMD:R_0402_1005Metric, F.Cu at (85.0, 63.5)
- added R40: 1k, Resistor_SMD:R_0402_1005Metric, F.Cu at (198.8, 47.9)
- added R41: 1M, Resistor_SMD:R_0402_1005Metric, F.Cu at (198.8, 55.8)
- added R42: 10k, Resistor_SMD:R_0402_1005Metric, F.Cu at (198.8, 57.8)
- added R43: 290k, Resistor_SMD:R_0402_1005Metric, F.Cu at (198.8, 59.8)
- added R44: 1k, Resistor_SMD:R_0402_1005Metric, F.Cu at (198.8, 61.8)
- added R45: 1M, Resistor_SMD:R_0402_1005Metric, F.Cu at (182.4, 83.6)
- added R46: 10k, Resistor_SMD:R_0402_1005Metric, F.Cu at (182.4, 85.6)
- added R47: 290k, Resistor_SMD:R_0402_1005Metric, F.Cu at (182.4, 87.6)
- added R48: 1k, Resistor_SMD:R_0402_1005Metric, F.Cu at (182.4, 89.6)
- added R49: 1M, Resistor_SMD:R_0402_1005Metric, F.Cu at (182.4, 41.9)
- added R5: 1M, Resistor_SMD:R_0402_1005Metric, F.Cu at (247.9, 55.8)
- added R50: 10k, Resistor_SMD:R_0402_1005Metric, F.Cu at (182.4, 43.9)
- added R51: 290k, Resistor_SMD:R_0402_1005Metric, F.Cu at (182.4, 45.9)
- added R52: 1k, Resistor_SMD:R_0402_1005Metric, F.Cu at (182.4, 47.9)
- added R53: 1M, Resistor_SMD:R_0402_1005Metric, F.Cu at (182.4, 69.7)
- added R54: 10k, Resistor_SMD:R_0402_1005Metric, F.Cu at (182.4, 71.7)
- added R55: 290k, Resistor_SMD:R_0402_1005Metric, F.Cu at (182.4, 73.7)
- added R56: 1k, Resistor_SMD:R_0402_1005Metric, F.Cu at (182.4, 75.7)
- added R57: 1M, Resistor_SMD:R_0402_1005Metric, F.Cu at (182.4, 97.5)
- added R58: 10k, Resistor_SMD:R_0402_1005Metric, F.Cu at (182.4, 99.5)
- added R59: 290k, Resistor_SMD:R_0402_1005Metric, F.Cu at (182.4, 101.5)
- added R6: 10k, Resistor_SMD:R_0402_1005Metric, F.Cu at (247.9, 57.8)
- added R60: 1k, Resistor_SMD:R_0402_1005Metric, F.Cu at (182.4, 103.5)
- added R61: 1M, Resistor_SMD:R_0402_1005Metric, F.Cu at (231.5, 55.8)
- added R62: 10k, Resistor_SMD:R_0402_1005Metric, F.Cu at (231.5, 57.8)
- added R63: 290k, Resistor_SMD:R_0402_1005Metric, F.Cu at (231.5, 59.8)
- added R64: 1k, Resistor_SMD:R_0402_1005Metric, F.Cu at (231.5, 61.8)
- added R65: 1M, Resistor_SMD:R_0402_1005Metric, F.Cu at (198.8, 69.7)
- added R66: 10k, Resistor_SMD:R_0402_1005Metric, F.Cu at (198.8, 71.7)
- added R67: 290k, Resistor_SMD:R_0402_1005Metric, F.Cu at (198.8, 73.7)
- added R68: 1k, Resistor_SMD:R_0402_1005Metric, F.Cu at (198.8, 75.7)
- added R69: 1M, Resistor_SMD:R_0402_1005Metric, F.Cu at (247.9, 41.9)
- added R7: 290k, Resistor_SMD:R_0402_1005Metric, F.Cu at (247.9, 59.8)
- added R70: 10k, Resistor_SMD:R_0402_1005Metric, F.Cu at (247.9, 43.9)
- added R71: 290k, Resistor_SMD:R_0402_1005Metric, F.Cu at (247.9, 45.9)
- added R72: 1k, Resistor_SMD:R_0402_1005Metric, F.Cu at (247.9, 47.9)
- added R73: 1M, Resistor_SMD:R_0402_1005Metric, F.Cu at (231.5, 41.9)
- added R74: 10k, Resistor_SMD:R_0402_1005Metric, F.Cu at (231.5, 43.9)
- added R75: 290k, Resistor_SMD:R_0402_1005Metric, F.Cu at (231.5, 45.9)
- added R76: 1k, Resistor_SMD:R_0402_1005Metric, F.Cu at (231.5, 47.9)
- added R77: 1M, Resistor_SMD:R_0402_1005Metric, F.Cu at (198.8, 97.5)
- added R78: 10k, Resistor_SMD:R_0402_1005Metric, F.Cu at (198.8, 99.5)
- added R79: 290k, Resistor_SMD:R_0402_1005Metric, F.Cu at (198.8, 101.5)
- added R8: 1k, Resistor_SMD:R_0402_1005Metric, F.Cu at (247.9, 61.8)
- added R80: 1k, Resistor_SMD:R_0402_1005Metric, F.Cu at (198.8, 103.5)
- added R81: 1M, Resistor_SMD:R_0402_1005Metric, F.Cu at (231.8, 25.4)
- added R82: 10k, Resistor_SMD:R_0402_1005Metric, F.Cu at (231.8, 27.4)
- added R83: 290k, Resistor_SMD:R_0402_1005Metric, F.Cu at (231.8, 29.4)
- added R84: 1k, Resistor_SMD:R_0402_1005Metric, F.Cu at (231.8, 31.4)
- added R85: 1M, Resistor_SMD:R_0402_1005Metric, F.Cu at (198.8, 83.6)
- added R86: 10k, Resistor_SMD:R_0402_1005Metric, F.Cu at (198.8, 85.6)
- added R87: 290k, Resistor_SMD:R_0402_1005Metric, F.Cu at (198.8, 87.6)
- added R88: 1k, Resistor_SMD:R_0402_1005Metric, F.Cu at (198.8, 89.6)
- added R89: 1M, Resistor_SMD:R_0402_1005Metric, F.Cu at (215.2, 55.8)
- added R9: 1M, Resistor_SMD:R_0402_1005Metric, F.Cu at (215.2, 69.7)
- added R90: 10k, Resistor_SMD:R_0402_1005Metric, F.Cu at (215.2, 57.8)
- added R91: 290k, Resistor_SMD:R_0402_1005Metric, F.Cu at (215.2, 59.8)
- added R92: 1k, Resistor_SMD:R_0402_1005Metric, F.Cu at (215.2, 61.8)
- added R93: 1M, Resistor_SMD:R_0402_1005Metric, F.Cu at (215.2, 41.9)
- added R94: 10k, Resistor_SMD:R_0402_1005Metric, F.Cu at (215.2, 43.9)
- added R95: 290k, Resistor_SMD:R_0402_1005Metric, F.Cu at (215.2, 45.9)
- added R96: 1k, Resistor_SMD:R_0402_1005Metric, F.Cu at (215.2, 47.9)
- added U1: AD7606, Package_QFP:LQFP-64_10x10mm_P0.5mm, F.Cu at (193.2, 31.7)
- added U10: AD7606, Package_QFP:LQFP-64_10x10mm_P0.5mm, F.Cu at (209.7, 31.7)
- added U19: AD7606, Package_QFP:LQFP-64_10x10mm_P0.5mm, F.Cu at (175.8, 31.7)
- MK12: moved to B.Cu
- turned MK12 to 180 degrees
