File: sonar-v1-pcb/sonar.kicad_pcb (KiCad board)
At the start: 2 copper layers, 16 parts, among them U1 ADS8568SPM, U4 ADS8568SPM, U7 ADS8568SPM

Commit message: added some adc shit
Parts:
- added C1: 1.6nf, Capacitor_SMD:C_0201_0603Metric, F.Cu at (74.1, 64.9)
- added C10: 1.6nf, Capacitor_SMD:C_0201_0603Metric, F.Cu at (74.1, 38.5)
- added C11: 1.6nf, Capacitor_SMD:C_0201_0603Metric, F.Cu at (74.1, 78.1)
- added C12: 1.6nf, Capacitor_SMD:C_0201_0603Metric, F.Cu at (47.5, 38.5)
- added C13: 1.6nf, Capacitor_SMD:C_0201_0603Metric, F.Cu at (34.2, 78.1)
- added C14: 1.6nf, Capacitor_SMD:C_0201_0603Metric, F.Cu at (60.8, 51.7)
- added C15: 1.6nf, Capacitor_SMD:C_0201_0603Metric, F.Cu at (87.4, 64.9)
- added C16: 1.6nf, Capacitor_SMD:C_0201_0603Metric, F.Cu at (34.2, 91.3)
- added C17: 1.6nf, Capacitor_SMD:C_0201_0603Metric, F.Cu at (47.5, 91.3)
- added C18: 1.6nf, Capacitor_SMD:C_0201_0603Metric, F.Cu at (60.8, 64.9)
- added C19: 1.6nf, Capacitor_SMD:C_0201_0603Metric, F.Cu at (34.2, 51.7)
- added C2: 1.6nf, Capacitor_SMD:C_0201_0603Metric, F.Cu at (79.8, 85.3)
- added C20: 1.6nf, Capacitor_SMD:C_0201_0603Metric, F.Cu at (87.4, 38.5)
- added C21: 1.6nf, Capacitor_SMD:C_0201_0603Metric, F.Cu at (47.5, 64.9)
- added C22: 1.6nf, Capacitor_SMD:C_0201_0603Metric, F.Cu at (34.2, 38.5)
- added C23: 1.6nf, Capacitor_SMD:C_0201_0603Metric, F.Cu at (60.8, 38.5)
- added C24: 1.6nf, Capacitor_SMD:C_0201_0603Metric, F.Cu at (74.1, 51.7)
- added C3: 1.6nf, Capacitor_SMD:C_0201_0603Metric, F.Cu at (96.5, 70.0)
- added C4: 1.6nf, Capacitor_SMD:C_0201_0603Metric, F.Cu at (60.8, 91.3)
- added C5: 1.6nf, Capacitor_SMD:C_0201_0603Metric, F.Cu at (60.8, 78.1)
- added C6: 1.6nf, Capacitor_SMD:C_0201_0603Metric, F.Cu at (34.2, 64.9)
- added C7: 1.6nf, Capacitor_SMD:C_0201_0603Metric, F.Cu at (47.5, 51.7)
- added C8: 1.6nf, Capacitor_SMD:C_0201_0603Metric, F.Cu at (87.4, 51.7)
- added C9: 1.6nf, Capacitor_SMD:C_0201_0603Metric, F.Cu at (47.5, 78.1)
- added MK10: Microphone_Ultrasound, Sonar:MA40S4, F.Cu at (91.0, 128.7)
- added MK11: Microphone_Ultrasound, Sonar:MA40S4, F.Cu at (122.8, 155.6)
- added MK12: Microphone_Ultrasound, Sonar:MA40S4, F.Cu at (59.2, 169.0)
- added MK13: Microphone_Ultrasound, Sonar:MA40S4, F.Cu at (59.2, 142.1)
- added MK14: Microphone_Ultrasound, Sonar:MA40S4, F.Cu at (75.1, 169.0)
- added MK15: Microphone_Ultrasound, Sonar:MA40S4, F.Cu at (106.9, 155.6)
- added MK16: Microphone_Ultrasound, Sonar:MA40S4, F.Cu at (59.2, 155.6)
- added MK17: Microphone_Ultrasound, Sonar:MA40S4, F.Cu at (75.1, 155.6)
- added MK18: Microphone_Ultrasound, Sonar:MA40S4, F.Cu at (122.8, 142.1)
- added MK19: Microphone_Ultrasound, Sonar:MA40S4, F.Cu at (107.8, 112.3)
- added MK20: Microphone_Ultrasound, Sonar:MA40S4, F.Cu at (106.9, 128.7)
- added MK21: Microphone_Ultrasound, Sonar:MA40S4, F.Cu at (75.1, 142.1)
- added MK22: Microphone_Ultrasound, Sonar:MA40S4, F.Cu at (106.9, 169.0)
- added MK23: Microphone_Ultrasound, Sonar:MA40S4, F.Cu at (75.1, 128.7)
- added MK24: Microphone_Ultrasound, Sonar:MA40S4, F.Cu at (91.0, 142.1)
- added MK4: Microphone_Ultrasound, Sonar:MA40S4, F.Cu at (91.0, 169.0)
- added MK5: Microphone_Ultrasound, Sonar:MA40S4, F.Cu at (91.0, 155.6)
- added MK6: Microphone_Ultrasound, Sonar:MA40S4, F.Cu at (59.2, 128.7)
- added MK7: Microphone_Ultrasound, Sonar:MA40S4, F.Cu at (122.8, 128.7)
- added MK8: Microphone_Ultrasound, Sonar:MA40S4, F.Cu at (106.9, 142.1)
- added MK9: Microphone_Ultrasound, Sonar:MA40S4, F.Cu at (91.9, 112.3)
- added R100: 1k, Resistor_SMD:R_0201_0603Metric, F.Cu at (60.8, 94.8)
- added R101: 1k, Resistor_SMD:R_0201_0603Metric, F.Cu at (60.8, 81.6)
- added R102: 1k, Resistor_SMD:R_0201_0603Metric, F.Cu at (34.2, 68.4)
- added R103: 1k, Resistor_SMD:R_0201_0603Metric, F.Cu at (47.5, 55.2)
- added R104: 1k, Resistor_SMD:R_0201_0603Metric, F.Cu at (87.4, 55.2)
- added R105: 1k, Resistor_SMD:R_0201_0603Metric, F.Cu at (47.5, 81.6)
- added R106: 1k, Resistor_SMD:R_0201_0603Metric, F.Cu at (74.1, 42.0)
- added R107: 1k, Resistor_SMD:R_0201_0603Metric, F.Cu at (74.1, 81.6)
- added R108: 1k, Resistor_SMD:R_0201_0603Metric, F.Cu at (47.5, 42.0)
- added R109: 1k, Resistor_SMD:R_0201_0603Metric, F.Cu at (34.2, 81.6)
- added R110: 1k, Resistor_SMD:R_0201_0603Metric, F.Cu at (60.8, 55.2)
- added R111: 1k, Resistor_SMD:R_0201_0603Metric, F.Cu at (87.4, 68.4)
- added R112: 1k, Resistor_SMD:R_0201_0603Metric, F.Cu at (34.2, 94.8)
- added R113: 1k, Resistor_SMD:R_0201_0603Metric, F.Cu at (47.5, 94.8)
- added R114: 1k, Resistor_SMD:R_0201_0603Metric, F.Cu at (60.8, 68.4)
- added R115: 1k, Resistor_SMD:R_0201_0603Metric, F.Cu at (34.2, 55.2)
- added R116: 1k, Resistor_SMD:R_0201_0603Metric, F.Cu at (87.4, 42.0)
- added R117: 1k, Resistor_SMD:R_0201_0603Metric, F.Cu at (47.5, 68.4)
- added R118: 1k, Resistor_SMD:R_0201_0603Metric, F.Cu at (34.2, 42.0)
- added R119: 1k, Resistor_SMD:R_0201_0603Metric, F.Cu at (60.8, 42.0)
- added R12: 100k, Resistor_SMD:R_0201_0603Metric, F.Cu at (93.1, 73.9)
- added R120: 1k, Resistor_SMD:R_0201_0603Metric, F.Cu at (74.1, 55.2)
- added R13: 10k, Resistor_SMD:R_0201_0603Metric, F.Cu at (98.0, 164.2)
- added R14: 100k, Resistor_SMD:R_0201_0603Metric, F.Cu at (98.0, 165.9)
- added R15: 1k, Resistor_SMD:R_0201_0603Metric, F.Cu at (98.0, 167.7)
- added R16: 100k, Resistor_SMD:R_0201_0603Metric, F.Cu at (60.8, 93.0)
- added R17: 10k, Resistor_SMD:R_0201_0603Metric, F.Cu at (98.0, 150.7)
- added R18: 100k, Resistor_SMD:R_0201_0603Metric, F.Cu at (98.0, 152.4)
- added R19: 1k, Resistor_SMD:R_0201_0603Metric, F.Cu at (98.0, 154.2)
- added R20: 100k, Resistor_SMD:R_0201_0603Metric, F.Cu at (60.8, 79.8)
- added R21: 10k, Resistor_SMD:R_0201_0603Metric, F.Cu at (66.2, 123.8)
- added R22: 100k, Resistor_SMD:R_0201_0603Metric, F.Cu at (66.2, 125.5)
- added R23: 1k, Resistor_SMD:R_0201_0603Metric, F.Cu at (66.2, 127.3)
- added R24: 100k, Resistor_SMD:R_0201_0603Metric, F.Cu at (34.2, 66.6)
- added R25: 10k, Resistor_SMD:R_0201_0603Metric, F.Cu at (129.8, 123.8)
- added R26: 100k, Resistor_SMD:R_0201_0603Metric, F.Cu at (129.8, 125.5)
- added R27: 1k, Resistor_SMD:R_0201_0603Metric, F.Cu at (129.8, 127.3)
- added R28: 100k, Resistor_SMD:R_0201_0603Metric, F.Cu at (47.5, 53.4)
- added R29: 10k, Resistor_SMD:R_0201_0603Metric, F.Cu at (113.9, 137.2)
- added R30: 100k, Resistor_SMD:R_0201_0603Metric, F.Cu at (113.9, 139.0)
- added R31: 1k, Resistor_SMD:R_0201_0603Metric, F.Cu at (113.9, 140.8)
- added R32: 100k, Resistor_SMD:R_0201_0603Metric, F.Cu at (87.4, 53.4)
- added R33: 10k, Resistor_SMD:R_0201_0603Metric, F.Cu at (98.9, 107.5)
- added R34: 100k, Resistor_SMD:R_0201_0603Metric, F.Cu at (98.9, 109.2)
- added R35: 1k, Resistor_SMD:R_0201_0603Metric, F.Cu at (98.9, 111.0)
- added R36: 100k, Resistor_SMD:R_0201_0603Metric, F.Cu at (47.5, 79.8)
- added R37: 10k, Resistor_SMD:R_0201_0603Metric, F.Cu at (98.0, 123.8)
- added R38: 100k, Resistor_SMD:R_0201_0603Metric, F.Cu at (98.0, 125.5)
- added R39: 1k, Resistor_SMD:R_0201_0603Metric, F.Cu at (98.0, 127.3)
- added R4: 100k, Resistor_SMD:R_0201_0603Metric, F.Cu at (74.1, 66.6)
- added R40: 100k, Resistor_SMD:R_0201_0603Metric, F.Cu at (74.1, 40.2)
- added R41: 10k, Resistor_SMD:R_0201_0603Metric, F.Cu at (129.8, 150.7)
- added R42: 100k, Resistor_SMD:R_0201_0603Metric, F.Cu at (129.8, 152.4)
- added R43: 1k, Resistor_SMD:R_0201_0603Metric, F.Cu at (129.8, 154.2)
- added R44: 100k, Resistor_SMD:R_0201_0603Metric, F.Cu at (74.1, 79.8)
- added R45: 10k, Resistor_SMD:R_0201_0603Metric, F.Cu at (66.2, 164.2)
- added R46: 100k, Resistor_SMD:R_0201_0603Metric, F.Cu at (66.2, 165.9)
- added R47: 1k, Resistor_SMD:R_0201_0603Metric, F.Cu at (66.2, 167.7)
- added R48: 100k, Resistor_SMD:R_0201_0603Metric, F.Cu at (47.5, 40.2)
- added R49: 10k, Resistor_SMD:R_0201_0603Metric, F.Cu at (66.2, 137.2)
- added R50: 100k, Resistor_SMD:R_0201_0603Metric, F.Cu at (66.2, 139.0)
- added R51: 1k, Resistor_SMD:R_0201_0603Metric, F.Cu at (66.2, 140.8)
- added R52: 100k, Resistor_SMD:R_0201_0603Metric, F.Cu at (34.2, 79.8)
- added R53: 10k, Resistor_SMD:R_0201_0603Metric, F.Cu at (82.1, 164.2)
- added R54: 100k, Resistor_SMD:R_0201_0603Metric, F.Cu at (82.1, 165.9)
- added R55: 1k, Resistor_SMD:R_0201_0603Metric, F.Cu at (82.1, 167.7)
- added R56: 100k, Resistor_SMD:R_0201_0603Metric, F.Cu at (60.8, 53.4)
- added R57: 10k, Resistor_SMD:R_0201_0603Metric, F.Cu at (113.9, 150.7)
- added R58: 100k, Resistor_SMD:R_0201_0603Metric, F.Cu at (113.9, 152.4)
- added R59: 1k, Resistor_SMD:R_0201_0603Metric, F.Cu at (113.9, 154.2)
- added R60: 100k, Resistor_SMD:R_0201_0603Metric, F.Cu at (87.4, 66.6)
- added R61: 10k, Resistor_SMD:R_0201_0603Metric, F.Cu at (66.2, 150.7)
- added R62: 100k, Resistor_SMD:R_0201_0603Metric, F.Cu at (66.2, 152.4)
- added R63: 1k, Resistor_SMD:R_0201_0603Metric, F.Cu at (66.2, 154.2)
- added R64: 100k, Resistor_SMD:R_0201_0603Metric, F.Cu at (34.2, 93.0)
- added R65: 10k, Resistor_SMD:R_0201_0603Metric, F.Cu at (82.1, 150.7)
- added R66: 100k, Resistor_SMD:R_0201_0603Metric, F.Cu at (82.1, 152.4)
- added R67: 1k, Resistor_SMD:R_0201_0603Metric, F.Cu at (82.1, 154.2)
- added R68: 100k, Resistor_SMD:R_0201_0603Metric, F.Cu at (47.5, 93.0)
- added R69: 10k, Resistor_SMD:R_0201_0603Metric, F.Cu at (129.8, 137.2)
- added R70: 100k, Resistor_SMD:R_0201_0603Metric, F.Cu at (129.8, 139.0)
- added R71: 1k, Resistor_SMD:R_0201_0603Metric, F.Cu at (129.8, 140.8)
- added R72: 100k, Resistor_SMD:R_0201_0603Metric, F.Cu at (60.8, 66.6)
- added R73: 10k, Resistor_SMD:R_0201_0603Metric, F.Cu at (114.8, 107.5)
- added R74: 100k, Resistor_SMD:R_0201_0603Metric, F.Cu at (114.8, 109.2)
- added R75: 1k, Resistor_SMD:R_0201_0603Metric, F.Cu at (114.8, 111.0)
- added R76: 100k, Resistor_SMD:R_0201_0603Metric, F.Cu at (34.2, 53.4)
- added R77: 10k, Resistor_SMD:R_0201_0603Metric, F.Cu at (113.9, 123.8)
- added R78: 100k, Resistor_SMD:R_0201_0603Metric, F.Cu at (113.9, 125.5)
- added R79: 1k, Resistor_SMD:R_0201_0603Metric, F.Cu at (113.9, 127.3)
- added R8: 100k, Resistor_SMD:R_0201_0603Metric, F.Cu at (79.8, 87.1)
- added R80: 100k, Resistor_SMD:R_0201_0603Metric, F.Cu at (87.4, 40.2)
- added R81: 10k, Resistor_SMD:R_0201_0603Metric, F.Cu at (82.1, 137.2)
- added R82: 100k, Resistor_SMD:R_0201_0603Metric, F.Cu at (82.1, 139.0)
- added R83: 1k, Resistor_SMD:R_0201_0603Metric, F.Cu at (82.1, 140.8)
- added R84: 100k, Resistor_SMD:R_0201_0603Metric, F.Cu at (47.5, 66.6)
- added R85: 10k, Resistor_SMD:R_0201_0603Metric, F.Cu at (113.9, 164.2)
- added R86: 100k, Resistor_SMD:R_0201_0603Metric, F.Cu at (113.9, 165.9)
- added R87: 1k, Resistor_SMD:R_0201_0603Metric, F.Cu at (113.9, 167.7)
- added R88: 100k, Resistor_SMD:R_0201_0603Metric, F.Cu at (34.2, 40.2)
- added R89: 10k, Resistor_SMD:R_0201_0603Metric, F.Cu at (82.1, 123.8)
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Connections:
- R1 pad 2: /eight_transducer_array/GND -> /eight_transducer_array/10V
- R11 pad 1: Net-(U9--) -> Net-(U7--)
- R5 pad 1: Net-(U5--) (its old number) -> Net-(U4--)
- R5 pad 2: /eight_transducer_array1/GND -> /eight_transducer_array1/10V
- R6 pad 1: Net-(U5--) (its old number) -> Net-(U4--)
- R9 pad 2: /eight_transducer_array2/GND -> /eight_transducer_array2/10V
- U1 pad 1: unconnected-(U1-HVSS-Pad1) -> /eight_transducer_array/GND
- U1 pad 14: unconnected-(U1-AVDD-Pad14) -> /eight_transducer_array/15V
- U1 pad 15: /eight_transducer_array/GND -> /eight_transducer_array/10V
- U1 pad 16: unconnected-(U1-DB15_SDO_D-Pad16) -> /eight_transducer_array/read_out_bus.db15
- U1 pad 17: unconnected-(U1-DB14_SDO_C-Pad17) -> /eight_transducer_array/read_out_bus.db14
- U1 pad 18: unconnected-(U1-DB13_SDO_B-Pad18) -> /eight_transducer_array/read_out_bus.db13
- U1 pad 19: unconnected-(U1-DB12_SDO_A-Pad19) -> /eight_transducer_array/read_out_bus.db12
- U1 pad 20: unconnected-(U1-DB11_REFBUFEN_N-Pad20) -> /eight_transducer_array/read_out_bus.db11
- U1 pad 21: unconnected-(U1-DB10_SCLK-Pad21) -> /eight_transducer_array/read_out_bus.db10
- U1 pad 22: unconnected-(U1-DB9_SDI-Pad22) -> /eight_transducer_array/read_out_bus.db9
- U1 pad 23: unconnected-(U1-DB8_DCEN-Pad23) -> /eight_transducer_array/read_out_bus.db8
- U1 pad 24: /eight_transducer_array/GND -> /eight_transducer_array/10V
- U1 pad 25: unconnected-(U1-DVDD-Pad25) -> /eight_transducer_array/15V
- U1 pad 26: unconnected-(U1-DB7-Pad26) -> /eight_transducer_array/read_out_bus.db7
- U1 pad 27: unconnected-(U1-DB6_SEL_B-Pad27) -> /eight_transducer_array/read_out_bus.db6
- U1 pad 28: unconnected-(U1-DB5_SEL_CD-Pad28) -> /eight_transducer_array/read_out_bus.db5
- U1 pad 29: unconnected-(U1-DB4-Pad29) -> /eight_transducer_array/read_out_bus.db4
- U1 pad 30: unconnected-(U1-DB3_DCIN_A-Pad30) -> /eight_transducer_array/read_out_bus.db3
- U1 pad 31: unconnected-(U1-DB2_DCIN_B-Pad31) -> /eight_transducer_array/read_out_bus.db2
- U1 pad 32: unconnected-(U1-DB1_DCIN_C-Pad32) -> /eight_transducer_array/read_out_bus.db1
- U1 pad 33: unconnected-(U1-DB0_DCIN_D-Pad33) -> /eight_transducer_array/read_out_bus.db0
- U1 pad 4: unconnected-(U1-AVDD-Pad4) -> /eight_transducer_array/15V
- U1 pad 44: /eight_transducer_array/GND -> /eight_transducer_array/10V
- U1 pad 45: unconnected-(U1-AVDD-Pad45) -> /eight_transducer_array/15V
- U1 pad 48: unconnected-(U1-HVDD-Pad48) -> /eight_transducer_array/20V
- U1 pad 5: /eight_transducer_array/GND -> /eight_transducer_array/10V
- U1 pad 51: /eight_transducer_array/GND -> /eight_transducer_array/10V
- U1 pad 52: unconnected-(U1-AVDD-Pad52) -> /eight_transducer_array/15V
- U1 pad 57: unconnected-(U1-AVDD-Pad57) -> /eight_transducer_array/15V
- U1 pad 58: /eight_transducer_array/GND -> /eight_transducer_array/10V
- U1 pad 61: unconnected-(U1-AVDD-Pad61) -> /eight_transducer_array/15V
- U1 pad 62: /eight_transducer_array/GND -> /eight_transducer_array/10V
- U4 pad 1: unconnected-(U4-HVSS-Pad1) -> Net-(U4-+)
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
Commit message: fix bandpass
Parts:
- removed U10, U11, U12, U13, U14, U15, U16, U17, U19, U2, U20, U21, U22, U23, U24, U25, U26, U27, U28, U29, U3, U30, U31, U32, U33, U34, U36, U37, U38, U39, U4, U40, U41, U42, U43, U44, U45, U46, U47, U48, U49, U5, U50, U51, U6, U7, U8, U9: ~, Package_TO_SOT_SMD:SOT-23-5
- added C25: 10uF, Capacitor_SMD:C_0402_1005Metric, F.Cu at (222.7, 89.2)
- added C26: 10uF, Capacitor_SMD:C_0402_1005Metric, F.Cu at (230.5, 89.2)
- added C27: 10uF, Capacitor_SMD:C_0402_1005Metric, F.Cu at (215.0, 89.2)
- added C28: 10uF, Capacitor_SMD:C_0402_1005Metric, F.Cu at (222.7, 91.2)
- added C29: 10uF, Capacitor_SMD:C_0402_1005Metric, F.Cu at (230.5, 91.2)
- added C30: 10uF, Capacitor_SMD:C_0402_1005Metric, F.Cu at (215.0, 91.2)
- added C31: 10uF, Capacitor_SMD:C_0402_1005Metric, F.Cu at (222.7, 93.2)
- added C32: 10uF, Capacitor_SMD:C_0402_1005Metric, F.Cu at (230.5, 93.2)
- added C33: 10uF, Capacitor_SMD:C_0402_1005Metric, F.Cu at (215.0, 93.2)
- added C34: 10uF, Capacitor_SMD:C_0402_1005Metric, F.Cu at (222.7, 95.1)
- added C35: 10uF, Capacitor_SMD:C_0402_1005Metric, F.Cu at (230.5, 95.1)
- added C36: 10uF, Capacitor_SMD:C_0402_1005Metric, F.Cu at (215.0, 95.1)
- added C37: 10uF, Capacitor_SMD:C_0402_1005Metric, F.Cu at (222.7, 97.1)
- added C38: 10uF, Capacitor_SMD:C_0402_1005Metric, F.Cu at (230.5, 97.1)
- added C39: 10uF, Capacitor_SMD:C_0402_1005Metric, F.Cu at (215.0, 97.1)
- added C40: 0.1uF, Capacitor_SMD:C_0402_1005Metric, F.Cu at (222.7, 99.1)
- added C41: 0.1uF, Capacitor_SMD:C_0402_1005Metric, F.Cu at (230.5, 99.1)
- added C42: 0.1uF, Capacitor_SMD:C_0402_1005Metric, F.Cu at (215.0, 99.1)
- added C43: 10uF, Capacitor_SMD:C_0402_1005Metric, F.Cu at (222.7, 101.0)
- added C44: 0.1uF, Capacitor_SMD:C_0402_1005Metric, F.Cu at (222.7, 103.0)
- added C45: 10uF, Capacitor_SMD:C_0402_1005Metric, F.Cu at (230.5, 101.0)
- added C46: 0.1uF, Capacitor_SMD:C_0402_1005Metric, F.Cu at (230.5, 103.0)
- added C47: 10uF, Capacitor_SMD:C_0402_1005Metric, F.Cu at (215.0, 101.0)
- added C48: 0.1uF, Capacitor_SMD:C_0402_1005Metric, F.Cu at (215.0, 103.0)
- added R121: 100k, Resistor_SMD:R_0402_1005Metric, F.Cu at (225.6, 89.2)
- added R122: 100k, Resistor_SMD:R_0402_1005Metric, F.Cu at (233.4, 89.2)
- added R123: 100k, Resistor_SMD:R_0402_1005Metric, F.Cu at (217.8, 89.2)
- added R124: 100k, Resistor_SMD:R_0402_1005Metric, F.Cu at (225.6, 91.2)
- added R125: 100k, Resistor_SMD:R_0402_1005Metric, F.Cu at (233.4, 91.2)
- added R126: 100k, Resistor_SMD:R_0402_1005Metric, F.Cu at (217.8, 91.2)
- added R127: 100k, Resistor_SMD:R_0402_1005Metric, F.Cu at (225.6, 93.2)
- added R128: 100k, Resistor_SMD:R_0402_1005Metric, F.Cu at (233.4, 93.2)
- added R129: 100k, Resistor_SMD:R_0402_1005Metric, F.Cu at (217.8, 93.2)
- added R130: 100k, Resistor_SMD:R_0402_1005Metric, F.Cu at (225.6, 95.2)
- added R131: 100k, Resistor_SMD:R_0402_1005Metric, F.Cu at (233.4, 95.2)
- added R132: 100k, Resistor_SMD:R_0402_1005Metric, F.Cu at (217.8, 95.2)
- added TP1: TestPoint_Probe, TestPoint:TestPoint_Pad_D1.0mm, F.Cu at (316.5, 290.0)
- added TP10: TestPoint_Probe, TestPoint:TestPoint_Pad_D1.0mm, F.Cu at (148.8, 80.9)
- added TP11: TestPoint_Probe, TestPoint:TestPoint_Pad_D1.0mm, F.Cu at (170.9, 80.9)
- added TP12: TestPoint_Probe, TestPoint:TestPoint_Pad_D1.0mm, F.Cu at (148.8, 55.6)
- added TP13: TestPoint_Probe, TestPoint:TestPoint_Pad_D1.0mm, F.Cu at (143.2, 55.6)
- added TP14: TestPoint_Probe, TestPoint:TestPoint_Pad_D1.0mm, F.Cu at (154.3, 68.2)
- added TP15: TestPoint_Probe, TestPoint:TestPoint_Pad_D1.0mm, F.Cu at (165.4, 80.9)
- added TP16: TestPoint_Probe, TestPoint:TestPoint_Pad_D1.0mm, F.Cu at (143.2, 80.9)
- added TP17: TestPoint_Probe, TestPoint:TestPoint_Pad_D1.0mm, F.Cu at (176.5, 55.6)
- added TP18: TestPoint_Probe, TestPoint:TestPoint_Pad_D1.0mm, F.Cu at (159.8, 80.9)
- added TP19: TestPoint_Probe, TestPoint:TestPoint_Pad_D1.0mm, F.Cu at (137.7, 68.2)
- added TP2: TestPoint_Probe, TestPoint:TestPoint_Pad_D1.0mm, F.Cu at (143.2, 68.2)
- added TP20: TestPoint_Probe, TestPoint:TestPoint_Pad_D1.0mm, F.Cu at (154.3, 55.6)
- added TP21: TestPoint_Probe, TestPoint:TestPoint_Pad_D1.0mm, F.Cu at (165.4, 55.6)
- added TP22: TestPoint_Probe, TestPoint:TestPoint_Pad_D1.0mm, F.Cu at (176.5, 80.9)
- added TP23: TestPoint_Probe, TestPoint:TestPoint_Pad_D1.0mm, F.Cu at (148.8, 68.2)
- added TP24: TestPoint_Probe, TestPoint:TestPoint_Pad_D1.0mm, F.Cu at (154.3, 80.9)
- added TP25: TestPoint_Probe, TestPoint:TestPoint_Pad_D1.0mm, F.Cu at (309.0, 296.0)
- added TP26: TestPoint_Probe, TestPoint:TestPoint_Pad_D1.0mm, F.Cu at (143.2, 71.8)
- added TP27: TestPoint_Probe, TestPoint:TestPoint_Pad_D1.0mm, F.Cu at (170.9, 59.1)
- added TP28: TestPoint_Probe, TestPoint:TestPoint_Pad_D1.0mm, F.Cu at (170.9, 71.8)
- added TP29: TestPoint_Probe, TestPoint:TestPoint_Pad_D1.0mm, F.Cu at (165.4, 71.8)
- added TP3: TestPoint_Probe, TestPoint:TestPoint_Pad_D1.0mm, F.Cu at (170.9, 55.6)
- added TP30: TestPoint_Probe, TestPoint:TestPoint_Pad_D1.0mm, F.Cu at (137.7, 84.5)
- added TP31: TestPoint_Probe, TestPoint:TestPoint_Pad_D1.0mm, F.Cu at (159.8, 59.1)
- added TP32: TestPoint_Probe, TestPoint:TestPoint_Pad_D1.0mm, F.Cu at (159.8, 71.8)
- added TP33: TestPoint_Probe, TestPoint:TestPoint_Pad_D1.0mm, F.Cu at (137.7, 59.1)
- added TP34: TestPoint_Probe, TestPoint:TestPoint_Pad_D1.0mm, F.Cu at (148.8, 84.5)
- added TP35: TestPoint_Probe, TestPoint:TestPoint_Pad_D1.0mm, F.Cu at (170.9, 84.5)
- added TP36: TestPoint_Probe, TestPoint:TestPoint_Pad_D1.0mm, F.Cu at (148.8, 59.1)
- added TP37: TestPoint_Probe, TestPoint:TestPoint_Pad_D1.0mm, F.Cu at (143.2, 59.1)
- added TP38: TestPoint_Probe, TestPoint:TestPoint_Pad_D1.0mm, F.Cu at (154.3, 71.8)
- added TP39: TestPoint_Probe, TestPoint:TestPoint_Pad_D1.0mm, F.Cu at (165.4, 84.5)
- added TP4: TestPoint_Probe, TestPoint:TestPoint_Pad_D1.0mm, F.Cu at (170.9, 68.2)
- added TP40: TestPoint_Probe, TestPoint:TestPoint_Pad_D1.0mm, F.Cu at (143.2, 84.5)
- added TP41: TestPoint_Probe, TestPoint:TestPoint_Pad_D1.0mm, F.Cu at (176.5, 59.1)
- added TP42: TestPoint_Probe, TestPoint:TestPoint_Pad_D1.0mm, F.Cu at (159.8, 84.5)
- added TP43: TestPoint_Probe, TestPoint:TestPoint_Pad_D1.0mm, F.Cu at (137.7, 71.8)
- added TP44: TestPoint_Probe, TestPoint:TestPoint_Pad_D1.0mm, F.Cu at (154.3, 59.1)
- added TP45: TestPoint_Probe, TestPoint:TestPoint_Pad_D1.0mm, F.Cu at (165.4, 59.1)
- added TP46: TestPoint_Probe, TestPoint:TestPoint_Pad_D1.0mm, F.Cu at (176.5, 84.5)
- added TP47: TestPoint_Probe, TestPoint:TestPoint_Pad_D1.0mm, F.Cu at (148.8, 71.8)
- added TP48: TestPoint_Probe, TestPoint:TestPoint_Pad_D1.0mm, F.Cu at (154.3, 84.5)
- added TP49: TestPoint_Probe, TestPoint:TestPoint_Pad_D1.0mm, F.Cu at (316.0, 295.5)
- added TP5: TestPoint_Probe, TestPoint:TestPoint_Pad_D1.0mm, F.Cu at (165.4, 68.2)
- added TP50: TestPoint_Probe, TestPoint:TestPoint_Pad_D1.0mm, F.Cu at (143.2, 75.3)
- added TP51: TestPoint_Probe, TestPoint:TestPoint_Pad_D1.0mm, F.Cu at (170.9, 62.7)
- added TP52: TestPoint_Probe, TestPoint:TestPoint_Pad_D1.0mm, F.Cu at (170.9, 75.3)
- added TP53: TestPoint_Probe, TestPoint:TestPoint_Pad_D1.0mm, F.Cu at (165.4, 75.3)
- added TP54: TestPoint_Probe, TestPoint:TestPoint_Pad_D1.0mm, F.Cu at (137.7, 88.0)
- added TP55: TestPoint_Probe, TestPoint:TestPoint_Pad_D1.0mm, F.Cu at (159.8, 62.7)
- added TP56: TestPoint_Probe, TestPoint:TestPoint_Pad_D1.0mm, F.Cu at (159.8, 75.3)
- added TP57: TestPoint_Probe, TestPoint:TestPoint_Pad_D1.0mm, F.Cu at (137.7, 62.7)
- added TP58: TestPoint_Probe, TestPoint:TestPoint_Pad_D1.0mm, F.Cu at (148.8, 88.0)
- added TP59: TestPoint_Probe, TestPoint:TestPoint_Pad_D1.0mm, F.Cu at (170.9, 88.0)
- added TP6: TestPoint_Probe, TestPoint:TestPoint_Pad_D1.0mm, F.Cu at (137.7, 80.9)
- added TP60: TestPoint_Probe, TestPoint:TestPoint_Pad_D1.0mm, F.Cu at (148.8, 62.7)
- added TP61: TestPoint_Probe, TestPoint:TestPoint_Pad_D1.0mm, F.Cu at (143.2, 62.7)
- added TP62: TestPoint_Probe, TestPoint:TestPoint_Pad_D1.0mm, F.Cu at (154.3, 75.3)
- added TP63: TestPoint_Probe, TestPoint:TestPoint_Pad_D1.0mm, F.Cu at (165.4, 88.0)
- added TP64: TestPoint_Probe, TestPoint:TestPoint_Pad_D1.0mm, F.Cu at (143.2, 88.0)
- added TP65: TestPoint_Probe, TestPoint:TestPoint_Pad_D1.0mm, F.Cu at (176.5, 62.7)
- added TP66: TestPoint_Probe, TestPoint:TestPoint_Pad_D1.0mm, F.Cu at (159.8, 88.0)
- added TP67: TestPoint_Probe, TestPoint:TestPoint_Pad_D1.0mm, F.Cu at (137.7, 75.3)
- added TP68: TestPoint_Probe, TestPoint:TestPoint_Pad_D1.0mm, F.Cu at (154.3, 62.7)
- added TP69: TestPoint_Probe, TestPoint:TestPoint_Pad_D1.0mm, F.Cu at (165.4, 62.7)
- added TP7: TestPoint_Probe, TestPoint:TestPoint_Pad_D1.0mm, F.Cu at (159.8, 55.6)
- added TP70: TestPoint_Probe, TestPoint:TestPoint_Pad_D1.0mm, F.Cu at (176.5, 88.0)
- added TP71: TestPoint_Probe, TestPoint:TestPoint_Pad_D1.0mm, F.Cu at (148.8, 75.3)
- added TP72: TestPoint_Probe, TestPoint:TestPoint_Pad_D1.0mm, F.Cu at (154.3, 88.0)
- added TP73: TestPoint_Probe, TestPoint:TestPoint_Pad_D1.0mm, F.Cu at (314.0, 296.0)
- added TP74: TestPoint_Probe, TestPoint:TestPoint_Pad_D1.0mm, F.Cu at (195.1, 114.8)
- added TP75: TestPoint_Probe, TestPoint:TestPoint_Pad_D1.0mm, F.Cu at (195.1, 119.8)
- added TP76: TestPoint_Probe, TestPoint:TestPoint_Pad_D1.0mm, F.Cu at (184.9, 129.9)
- added TP77: TestPoint_Probe, TestPoint:TestPoint_Pad_D1.0mm, F.Cu at (195.1, 124.9)
- added TP78: TestPoint_Probe, TestPoint:TestPoint_Pad_D1.0mm, F.Cu at (184.9, 114.8)
- added TP79: TestPoint_Probe, TestPoint:TestPoint_Pad_D1.0mm, F.Cu at (184.9, 119.8)
- added TP8: TestPoint_Probe, TestPoint:TestPoint_Pad_D1.0mm, F.Cu at (159.8, 68.2)
- added TP80: TestPoint_Probe, TestPoint:TestPoint_Pad_D1.0mm, F.Cu at (184.9, 124.9)
- added TP81: TestPoint_Probe, TestPoint:TestPoint_Pad_D1.0mm, F.Cu at (174.8, 114.8)
- added TP82: TestPoint_Probe, TestPoint:TestPoint_Pad_D1.0mm, F.Cu at (174.8, 135.0)
- added TP83: TestPoint_Probe, TestPoint:TestPoint_Pad_D1.0mm, F.Cu at (195.1, 129.9)
- added TP84: TestPoint_Probe, TestPoint:TestPoint_Pad_D1.0mm, F.Cu at (174.8, 124.9)
- added TP85: TestPoint_Probe, TestPoint:TestPoint_Pad_D1.0mm, F.Cu at (190.0, 114.8)
- added TP86: TestPoint_Probe, TestPoint:TestPoint_Pad_D1.0mm, F.Cu at (179.9, 129.9)
- added TP87: TestPoint_Probe, TestPoint:TestPoint_Pad_D1.0mm, F.Cu at (190.0, 129.9)
- added TP88: TestPoint_Probe, TestPoint:TestPoint_Pad_D1.0mm, F.Cu at (174.8, 119.8)
- added TP89: TestPoint_Probe, TestPoint:TestPoint_Pad_D1.0mm, F.Cu at (179.9, 124.9)
- added TP9: TestPoint_Probe, TestPoint:TestPoint_Pad_D1.0mm, F.Cu at (135.0, 54.0)
- added TP90: TestPoint_Probe, TestPoint:TestPoint_Pad_D1.0mm, F.Cu at (190.0, 124.9)
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Connections:
- C1 pad 2: /eight_transducer_array/10V -> /eight_transducer_array/GND
- C10 pad 2: /eight_transducer_array2/10V -> /eight_transducer_array2/GND
- C11 pad 2: /eight_transducer_array/10V -> /eight_transducer_array/GND
- C12 pad 2: /eight_transducer_array1/10V -> /eight_transducer_array1/GND
- C13 pad 2: /eight_transducer_array1/10V -> /eight_transducer_array1/GND
- C14 pad 2: /eight_transducer_array2/10V -> /eight_transducer_array2/GND
- C15 pad 2: /eight_transducer_array/10V -> /eight_transducer_array/GND
- C16 pad 2: /eight_transducer_array1/10V -> /eight_transducer_array1/GND
- C17 pad 2: /eight_transducer_array2/10V -> /eight_transducer_array2/GND
- C18 pad 2: /eight_transducer_array/10V -> /eight_transducer_array/GND
- C19 pad 2: /eight_transducer_array1/10V -> /eight_transducer_array1/GND
- C2 pad 2: /eight_transducer_array1/10V -> /eight_transducer_array1/GND
- C20 pad 2: /eight_transducer_array2/10V -> /eight_transducer_array2/GND
- C21 pad 2: /eight_transducer_array2/10V -> /eight_transducer_array2/GND
- C22 pad 2: /eight_transducer_array/10V -> /eight_transducer_array/GND
- C23 pad 2: /eight_transducer_array1/10V -> /eight_transducer_array1/GND
- C24 pad 2: /eight_transducer_array2/10V -> /eight_transducer_array2/GND
- C3 pad 2: /eight_transducer_array2/10V -> /eight_transducer_array2/GND
- C4 pad 2: /eight_transducer_array/10V -> /eight_transducer_array/GND
- C5 pad 2: /eight_transducer_array/10V -> /eight_transducer_array/GND
- C6 pad 2: /eight_transducer_array1/10V -> /eight_transducer_array1/GND
- C7 pad 2: /eight_transducer_array2/10V -> /eight_transducer_array2/GND
- C8 pad 2: /eight_transducer_array/10V -> /eight_transducer_array/GND
- C9 pad 2: /eight_transducer_array1/10V -> /eight_transducer_array1/GND
- MK1 pad 2: /eight_transducer_array/10V -> /eight_transducer_array/GND
- MK10 pad 2: /eight_transducer_array2/10V -> /eight_transducer_array2/GND
- MK11 pad 2: /eight_transducer_array/10V -> /eight_transducer_array/GND
- MK12 pad 2: /eight_transducer_array1/10V -> /eight_transducer_array1/GND
- MK13 pad 2: /eight_transducer_array1/10V -> /eight_transducer_array1/GND
- MK14 pad 2: /eight_transducer_array2/10V -> /eight_transducer_array2/GND
- MK15 pad 2: /eight_transducer_array/10V -> /eight_transducer_array/GND
- MK16 pad 2: /eight_transducer_array1/10V -> /eight_transducer_array1/GND
- MK17 pad 2: /eight_transducer_array2/10V -> /eight_transducer_array2/GND
- MK18 pad 2: /eight_transducer_array/10V -> /eight_transducer_array/GND
- MK19 pad 2: /eight_transducer_array1/10V -> /eight_transducer_array1/GND
- MK2 pad 2: /eight_transducer_array1/10V -> /eight_transducer_array1/GND
- MK20 pad 2: /eight_transducer_array2/10V -> /eight_transducer_array2/GND
- MK21 pad 2: /eight_transducer_array2/10V -> /eight_transducer_array2/GND
- MK22 pad 2: /eight_transducer_array/10V -> /eight_transducer_array/GND
- MK23 pad 2: /eight_transducer_array1/10V -> /eight_transducer_array1/GND
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Other:
- board outline added: 10 x 10 mm
- copper layers 2 -> 4

Commit message: kept cooking
Parts:
- removed U35: ADS8568SPM, Package_QFP:LQFP-64-1EP_10x10mm_P0.5mm_EP6.5x6.5mm_ThermalVias
- removed U53, U54, U55, U56, U57, U58, U59, U60, U61, U62, U63, U64, U65, U66, U67, U68, U69, U70, U71, U72, U73, U74, U75, U76: Opamp_Dual, Package_SO:TSSOP-8_3x3mm_P0.65mm
- added C49: 1.6nF, Capacitor_SMD:C_0402_1005Metric, F.Cu at (268.4, 67.0)
- added C50: 100nF, Capacitor_SMD:C_0402_1005Metric, F.Cu at (263.5, 80.1)
- added C51: 1.6nF, Capacitor_SMD:C_0402_1005Metric, F.Cu at (263.5, 82.1)
- added C52: 1.6nF, Capacitor_SMD:C_0402_1005Metric, F.Cu at (263.5, 84.1)
- added C53: 100nF, Capacitor_SMD:C_0402_1005Metric, F.Cu at (251.7, 70.3)
- added C54: 1.6nF, Capacitor_SMD:C_0402_1005Metric, F.Cu at (251.7, 72.3)
- added C55: 1.6nF, Capacitor_SMD:C_0402_1005Metric, F.Cu at (251.7, 74.2)
- added C56: 10uF, Capacitor_SMD:C_0402_1005Metric, F.Cu at (263.5, 62.4)
- added C57: 10uF, Capacitor_SMD:C_0402_1005Metric, F.Cu at (263.5, 64.3)
- added C58: 0.1uF, Capacitor_SMD:C_0402_1005Metric, F.Cu at (263.5, 66.3)
- added C59: 0.1uF, Capacitor_SMD:C_0402_1005Metric, F.Cu at (263.5, 68.3)
- added C60: 10uF, Capacitor_SMD:C_0402_1005Metric, F.Cu at (263.5, 70.3)
- added C61: 10uF, Capacitor_SMD:C_0402_1005Metric, F.Cu at (263.5, 72.2)
- added C62: 10uF, Capacitor_SMD:C_0402_1005Metric, F.Cu at (263.5, 74.2)
- added C63: 10uF, Capacitor_SMD:C_0402_1005Metric, F.Cu at (263.5, 76.2)
- added C64: 100nF, Capacitor_SMD:C_0402_1005Metric, F.Cu at (251.7, 62.4)
- added C65: 1.6nF, Capacitor_SMD:C_0402_1005Metric, F.Cu at (251.7, 64.3)
- added C66: 1.6nF, Capacitor_SMD:C_0402_1005Metric, F.Cu at (251.7, 66.3)
- added C67: 100nF, Capacitor_SMD:C_0402_1005Metric, F.Cu at (275.3, 46.6)
- added C68: 1.6nF, Capacitor_SMD:C_0402_1005Metric, F.Cu at (275.3, 48.5)
- added C69: 1.6nF, Capacitor_SMD:C_0402_1005Metric, F.Cu at (275.3, 50.5)
- added C70: 100nF, Capacitor_SMD:C_0402_1005Metric, F.Cu at (246.8, 38.6)
- added C71: 1.6nF, Capacitor_SMD:C_0402_1005Metric, F.Cu at (246.8, 40.6)
- added C72: 1.6nF, Capacitor_SMD:C_0402_1005Metric, F.Cu at (246.8, 42.6)
- added C73: 100nF, Capacitor_SMD:C_0402_1005Metric, F.Cu at (263.5, 38.6)
- added C74: 1.6nF, Capacitor_SMD:C_0402_1005Metric, F.Cu at (263.5, 40.6)
- added C75: 1.6nF, Capacitor_SMD:C_0402_1005Metric, F.Cu at (263.5, 42.6)
- added C76: 100nF, Capacitor_SMD:C_0402_1005Metric, F.Cu at (251.7, 38.6)
- added C77: 1.6nF, Capacitor_SMD:C_0402_1005Metric, F.Cu at (251.7, 40.6)
- added C78: 1.6nF, Capacitor_SMD:C_0402_1005Metric, F.Cu at (251.7, 42.6)
- added C79: 100nF, Capacitor_SMD:C_0402_1005Metric, F.Cu at (251.7, 46.6)
- added C80: 1.6nF, Capacitor_SMD:C_0402_1005Metric, F.Cu at (251.7, 48.5)
- added C81: 1.6nF, Capacitor_SMD:C_0402_1005Metric, F.Cu at (251.7, 50.5)
- added C82: 100nF, Capacitor_SMD:C_0402_1005Metric, F.Cu at (263.5, 54.5)
- added C83: 1.6nF, Capacitor_SMD:C_0402_1005Metric, F.Cu at (263.5, 56.4)
- added C84: 1.6nF, Capacitor_SMD:C_0402_1005Metric, F.Cu at (263.5, 58.4)
- added C85: 100nF, Capacitor_SMD:C_0402_1005Metric, F.Cu at (263.5, 46.6)
- added C86: 1.6nF, Capacitor_SMD:C_0402_1005Metric, F.Cu at (263.5, 48.5)
- added C87: 1.6nF, Capacitor_SMD:C_0402_1005Metric, F.Cu at (263.5, 50.5)
- added C88: 100nF, Capacitor_SMD:C_0402_1005Metric, F.Cu at (275.3, 54.5)
- added C89: 1.6nF, Capacitor_SMD:C_0402_1005Metric, F.Cu at (275.3, 56.4)
- added C90: 1.6nF, Capacitor_SMD:C_0402_1005Metric, F.Cu at (275.3, 58.4)
- added C91: 100nF, Capacitor_SMD:C_0402_1005Metric, F.Cu at (251.7, 54.5)
- added C92: 1.6nF, Capacitor_SMD:C_0402_1005Metric, F.Cu at (251.7, 56.4)
- added C93: 1.6nF, Capacitor_SMD:C_0402_1005Metric, F.Cu at (251.7, 58.4)
- added C94: 100nF, Capacitor_SMD:C_0402_1005Metric, F.Cu at (275.3, 38.6)
- added C95: 1.6nF, Capacitor_SMD:C_0402_1005Metric, F.Cu at (275.3, 40.6)
- added C96: 1.6nF, Capacitor_SMD:C_0402_1005Metric, F.Cu at (275.3, 42.6)
- added F1: 1.1A, Diode_SMD:D_1206_3216Metric, F.Cu at (253.1, 85.6)
- added U10: Opamp_Dual, Package_SO:TSSOP-8_3x3mm_P0.65mm, F.Cu at (241.9, 60.7)
- added U11: Opamp_Dual, Package_SO:TSSOP-8_3x3mm_P0.65mm, F.Cu at (241.9, 65.3)
- added U12: Opamp_Dual, Package_SO:TSSOP-8_3x3mm_P0.65mm, F.Cu at (279.4, 72.4)
- added U13: Opamp_Dual, Package_SO:TSSOP-8_3x3mm_P0.65mm, F.Cu at (270.4, 72.4)
- added U14: Opamp_Dual, Package_SO:TSSOP-8_3x3mm_P0.65mm, F.Cu at (270.4, 85.7)
- added U15: Opamp_Dual, Package_SO:TSSOP-8_3x3mm_P0.65mm, F.Cu at (279.4, 63.7)
- added U16: Opamp_Dual, Package_SO:TSSOP-8_3x3mm_P0.65mm, F.Cu at (279.4, 85.7)
- added U17: Opamp_Dual, Package_SO:TSSOP-8_3x3mm_P0.65mm, F.Cu at (270.4, 63.7)
- added U19: Opamp_Dual, Package_SO:TSSOP-8_3x3mm_P0.65mm, F.Cu at (256.6, 71.6)
- added U2: Opamp_Dual, Package_SO:TSSOP-8_3x3mm_P0.65mm, F.Cu at (270.4, 79.0)
- added U21: Opamp_Dual, Package_SO:TSSOP-8_3x3mm_P0.65mm, F.Cu at (256.6, 63.7)
- added U22: Opamp_Dual, Package_SO:TSSOP-8_3x3mm_P0.65mm, F.Cu at (280.2, 47.9)
- added U23: Opamp_Dual, Package_SO:TSSOP-8_3x3mm_P0.65mm, F.Cu at (241.9, 40.0)
- added U24: Opamp_Dual, Package_SO:TSSOP-8_3x3mm_P0.65mm, F.Cu at (241.9, 44.7)
- added U25: Opamp_Dual, Package_SO:TSSOP-8_3x3mm_P0.65mm, F.Cu at (241.9, 49.3)
- added U26: Opamp_Dual, Package_SO:TSSOP-8_3x3mm_P0.65mm, F.Cu at (268.4, 40.0)
- added U27: Opamp_Dual, Package_SO:TSSOP-8_3x3mm_P0.65mm, F.Cu at (256.6, 40.0)
- added U28: Opamp_Dual, Package_SO:TSSOP-8_3x3mm_P0.65mm, F.Cu at (256.6, 47.9)
- added U29: Opamp_Dual, Package_SO:TSSOP-8_3x3mm_P0.65mm, F.Cu at (268.4, 55.8)
- added U30: Opamp_Dual, Package_SO:TSSOP-8_3x3mm_P0.65mm, F.Cu at (268.4, 47.9)
- added U31: Opamp_Dual, Package_SO:TSSOP-8_3x3mm_P0.65mm, F.Cu at (280.2, 55.8)
- added U32: Opamp_Dual, Package_SO:TSSOP-8_3x3mm_P0.65mm, F.Cu at (256.6, 55.8)
- added U33: Opamp_Dual, Package_SO:TSSOP-8_3x3mm_P0.65mm, F.Cu at (280.2, 40.0)
- added U4: Opamp_Dual, Package_SO:TSSOP-8_3x3mm_P0.65mm, F.Cu at (253.7, 79.6)
- added U5: Opamp_Dual, Package_SO:TSSOP-8_3x3mm_P0.65mm, F.Cu at (241.9, 72.0)
- added U6: Opamp_Dual, Package_SO:TSSOP-8_3x3mm_P0.65mm, F.Cu at (241.9, 76.7)
- added U7: Opamp_Dual, Package_SO:TSSOP-8_3x3mm_P0.65mm, F.Cu at (241.9, 81.3)
- added U8: Opamp_Dual, Package_SO:TSSOP-8_3x3mm_P0.65mm, F.Cu at (279.4, 79.0)
- added U9: Opamp_Dual, Package_SO:TSSOP-8_3x3mm_P0.65mm, F.Cu at (241.9, 56.0)
- C1, C12, C13, C16, C17, C18, C19, C2, C5, C6, C7, C8: value 1.6nF -> 10uF
- C14, C15, C3, C4: value 1.6nF -> 0.1uF
- C20, C23, C9: value 1.6nF -> 100nF
- C25, C27, C28, C30, C31, C33, C34, C36, C37, C39, C43, C45: value 10uF -> 1.6nF
- C26, C29, C32, C35, C38, C47: value 10uF -> 100nF
- C40, C42, C46, C48: value 0.1uF -> 1.6nF
- C41, C44: value 0.1uF -> 100nF
- R1, R13, R21, R33, R41, R53, R61, R73, R77, R85, R9: value 10k -> 100k
- R100, R102, R105, R107, R11, R110, R112, R115, R117, R120, R23, R3, R31, R43, R51, R63, R7, R71, R75, R87, R95, R97: value 1k -> 100k
- R104, R109, R114, R119, R15, R35, R55, R79, R99: value 1k -> 10k
- R121, R123, R126, R128, R131, R14, R22, R24, R32, R34, R42, R44, R52, R54, R62, R64, R72, R78, R8, R86, R88, R96: value 100k -> 1k
- R124, R129, R20, R30, R40, R50, R6, R60, R70, R84, R94: value 100k -> 10k
- R17, R29, R37, R49, R5, R57, R69, R81, R93: value 10k -> 1k
- U18: value ADS8568SPM -> Opamp_Dual; footprint Package_QFP:LQFP-64-1EP_10x10mm_P0.5mm_EP6.5x6.5mm_ThermalVias -> Package_SO:TSSOP-8_3x3mm_P0.65mm
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Connections:
- C1 pad 1: Net-(U53A-+) -> /eight_transducer_array/GND
- C1 pad 2: /eight_transducer_array/GND -> /eight_transducer_array/10V
- C10 pad 1: Net-(U62A-+) -> Net-(U2A-+)
- C10 pad 2: /eight_transducer_array2/GND -> /eight_transducer_array/GND
- C11 pad 1: Net-(U63A-+) -> Net-(C11-Pad1)
- C11 pad 2: /eight_transducer_array/GND -> Net-(U2A--)
- C12 pad 1: Net-(U64A-+) -> /eight_transducer_array1/GND
- C12 pad 2: /eight_transducer_array1/GND -> /eight_transducer_array1/10V
- C13 pad 1: Net-(U65A-+) -> /eight_transducer_array1/-10V
- C14 pad 1: Net-(U66A-+) -> /eight_transducer_array1/GND
- C14 pad 2: /eight_transducer_array2/GND -> /eight_transducer_array1/10V
- C15 pad 1: Net-(U67A-+) -> /eight_transducer_array1/-10V
- C15 pad 2: /eight_transducer_array/GND -> /eight_transducer_array1/GND
- C16 pad 1: Net-(U68A-+) -> /eight_transducer_array1/GND
- C16 pad 2: /eight_transducer_array1/GND -> Net-(U3-REFAP)
- C17 pad 1: Net-(U69A-+) -> /eight_transducer_array1/GND
- C17 pad 2: /eight_transducer_array2/GND -> Net-(U3-REFBP)
- C18 pad 1: Net-(U70A-+) -> /eight_transducer_array1/GND
- C18 pad 2: /eight_transducer_array/GND -> Net-(U3-REFCP)
- C19 pad 1: Net-(U71A-+) -> /eight_transducer_array1/GND
- C19 pad 2: /eight_transducer_array1/GND -> Net-(U3-REFDP)
- C2 pad 1: Net-(U54A-+) -> /eight_transducer_array/-10V
- C2 pad 2: /eight_transducer_array1/GND -> /eight_transducer_array/GND
- C20 pad 1: Net-(U72A-+) -> /eight_transducer_array1/2.5V
- C20 pad 2: /eight_transducer_array2/GND -> /eight_transducer_array1/-2.5V
- C21 pad 1: Net-(U73A-+) -> Net-(U4A-+)
- C21 pad 2: /eight_transducer_array2/GND -> /eight_transducer_array1/GND
- C22 pad 1: Net-(U74A-+) -> Net-(C22-Pad1)
- C22 pad 2: /eight_transducer_array/GND -> Net-(U4A--)
- C23 pad 1: Net-(U75A-+) -> /eight_transducer_array/2.5V
- C23 pad 2: /eight_transducer_array1/GND -> /eight_transducer_array/-2.5V
- C24 pad 1: Net-(U76A-+) -> Net-(U6A-+)
- C24 pad 2: /eight_transducer_array2/GND -> /eight_transducer_array/GND
- C25 pad 1: /eight_transducer_array/GND -> Net-(C25-Pad1)
- C25 pad 2: Net-(U1-REFAP) -> Net-(U6A--)
- C26 pad 1: /eight_transducer_array1/GND -> /eight_transducer_array/2.5V
- C26 pad 2: Net-(U18-REFAP) -> /eight_transducer_array/-2.5V
- C27 pad 1: /eight_transducer_array2/GND -> Net-(U8A-+)
- C27 pad 2: Net-(U35-REFAP) -> /eight_transducer_array/GND
- C28 pad 1: /eight_transducer_array/GND -> Net-(C28-Pad1)
- C28 pad 2: Net-(U1-REFBP) -> Net-(U8A--)
- C29 pad 1: /eight_transducer_array1/GND -> /eight_transducer_array1/2.5V
- C29 pad 2: Net-(U18-REFBP) -> /eight_transducer_array1/-2.5V
- C3 pad 1: Net-(U55A-+) -> /eight_transducer_array/GND
- C3 pad 2: /eight_transducer_array2/GND -> /eight_transducer_array/10V
- C30 pad 1: /eight_transducer_array2/GND -> Net-(U10A-+)
- C30 pad 2: Net-(U35-REFBP) -> /eight_transducer_array1/GND
- C31 pad 1: /eight_transducer_array/GND -> Net-(C31-Pad1)
- C31 pad 2: Net-(U1-REFCP) -> Net-(U10A--)
- C32 pad 1: /eight_transducer_array1/GND -> /eight_transducer_array1/2.5V
- C32 pad 2: Net-(U18-REFCP) -> /eight_transducer_array1/-2.5V
- C33 pad 1: /eight_transducer_array2/GND -> Net-(U12A-+)
- C33 pad 2: Net-(U35-REFCP) -> /eight_transducer_array1/GND
- C34 pad 1: /eight_transducer_array/GND -> Net-(C34-Pad1)
- C34 pad 2: Net-(U1-REFDP) -> Net-(U12A--)
- C35 pad 1: /eight_transducer_array1/GND -> /eight_transducer_array/2.5V
- C35 pad 2: Net-(U18-REFDP) -> /eight_transducer_array/-2.5V
- C36 pad 1: /eight_transducer_array2/GND -> Net-(U13A-+)
- C36 pad 2: Net-(U35-REFDP) -> /eight_transducer_array/GND
- C37 pad 1: /eight_transducer_array/GND -> Net-(C37-Pad1)
- C37 pad 2: /eight_transducer_array/10V -> Net-(U13A--)
- C38 pad 1: /eight_transducer_array1/GND -> /eight_transducer_array1/2.5V
- C38 pad 2: /eight_transducer_array1/10V -> /eight_transducer_array1/-2.5V
- C39 pad 1: /eight_transducer_array2/GND -> Net-(U14A-+)
- C39 pad 2: /eight_transducer_array2/10V -> /eight_transducer_array1/GND
- C4 pad 1: Net-(U56A-+) -> /eight_transducer_array/-10V
- C40 pad 1: /eight_transducer_array/GND -> Net-(C40-Pad1)
- C40 pad 2: /eight_transducer_array/10V -> Net-(U14A--)
- C41 pad 1: /eight_transducer_array1/GND -> /eight_transducer_array1/2.5V
- C41 pad 2: /eight_transducer_array1/10V -> /eight_transducer_array1/-2.5V
- C42 pad 1: /eight_transducer_array2/GND -> Net-(U15A-+)
- C42 pad 2: /eight_transducer_array2/10V -> /eight_transducer_array1/GND
- C43 pad 1: /eight_transducer_array/-10V -> Net-(C43-Pad1)
- C43 pad 2: /eight_transducer_array/GND -> Net-(U15A--)
- C44 pad 1: /eight_transducer_array/-10V -> /eight_transducer_array1/2.5V
- C44 pad 2: /eight_transducer_array/GND -> /eight_transducer_array1/-2.5V
- C45 pad 1: /eight_transducer_array1/-10V -> Net-(U16A-+)
- C46 pad 1: /eight_transducer_array1/-10V -> Net-(C46-Pad1)
- C46 pad 2: /eight_transducer_array1/GND -> Net-(U16A--)
- C47 pad 1: /eight_transducer_array2/-10V -> /eight_transducer_array/2.5V
- C47 pad 2: /eight_transducer_array2/GND -> /eight_transducer_array/-2.5V
- C48 pad 1: /eight_transducer_array2/-10V -> Net-(U17A-+)
- C48 pad 2: /eight_transducer_array2/GND -> /eight_transducer_array/GND
- C5 pad 1: Net-(U57A-+) -> /eight_transducer_array/GND
- C5 pad 2: /eight_transducer_array/GND -> Net-(U1-REFAP)
- C6 pad 1: Net-(U58A-+) -> /eight_transducer_array/GND
- C6 pad 2: /eight_transducer_array1/GND -> Net-(U1-REFBP)
- C7 pad 1: Net-(U59A-+) -> /eight_transducer_array/GND
- C7 pad 2: /eight_transducer_array2/GND -> Net-(U1-REFCP)
- C8 pad 1: Net-(U60A-+) -> /eight_transducer_array/GND
- C8 pad 2: /eight_transducer_array/GND -> Net-(U1-REFDP)
- C9 pad 1: Net-(U61A-+) -> /eight_transducer_array/2.5V
- C9 pad 2: /eight_transducer_array1/GND -> /eight_transducer_array/-2.5V
- MK10 pad 2: /eight_transducer_array2/GND -> /eight_transducer_array1/GND
- MK14 pad 2: /eight_transducer_array2/GND -> /eight_transducer_array/GND
- MK15 pad 2: /eight_transducer_array/GND -> /eight_transducer_array2/GND
- MK16 pad 2: /eight_transducer_array1/GND -> /eight_transducer_array2/GND
- MK19 pad 2: /eight_transducer_array1/GND -> /eight_transducer_array2/GND
- MK23 pad 2: /eight_transducer_array1/GND -> /eight_transducer_array2/GND
- MK3 pad 2: /eight_transducer_array2/GND -> /eight_transducer_array/GND
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