File: sonar-v1-pcb/sonar.kicad_pcb (KiCad board)
At the start: 4 copper layers, 10 x 10 mm, 381 parts, among them U1 ADS8568SPM, U10 Opamp_Dual, U11 Opamp_Dual, U12 Opamp_Dual, U13 Opamp_Dual, U14 Opamp_Dual, U15 Opamp_Dual, U16 Opamp_Dual, U17 Opamp_Dual, U18 Opamp_Dual, U19 Opamp_Dual, U2 Opamp_Dual, U21 Opamp_Dual, U22 Opamp_Dual, U23 Opamp_Dual, U24 Opamp_Dual, U25 Opamp_Dual, U26 Opamp_Dual, U27 Opamp_Dual, U28 Opamp_Dual, U29 Opamp_Dual, U30 Opamp_Dual, U31 Opamp_Dual, U32 Opamp_Dual, U33 Opamp_Dual, U4 Opamp_Dual, U5 Opamp_Dual, U6 Opamp_Dual, U7 Opamp_Dual, U8 Opamp_Dual, U9 Opamp_Dual

Commit message: Switch to audio not just ultrasonic.
Parts:
- removed MK1, MK10, MK11, MK12, MK13, MK14, MK15, MK16, MK17, MK18, MK19, MK2, MK20, MK21, MK22, MK23, MK24, MK3, MK4, MK5, MK6, MK7, MK8, MK9: Microphone_Ultrasound, Sonar:MA40S4
- removed TP49, TP50, TP53, TP54, TP57, TP58, TP61, TP62, TP65, TP66, TP69, TP70, TP73, TP74, TP77, TP78, TP81, TP82, TP85, TP86, TP89, TP90, TP93, TP94: TestPoint_Probe, TestPoint:TestPoint_Pad_D1.0mm
- added J2: DF40C-80DS-0.4V51, Sonar:CONN80_DF40C-80DS_HIR, F.Cu at (166.1, 17.9)
- added MK25: SPV08A0LR5H-1, Sonar:MIC_SPV08A0LR5H-1, F.Cu at (253.8, 109.2)
- added MK26: SPV08A0LR5H-1, Sonar:MIC_SPV08A0LR5H-1, F.Cu at (265.9, 115.5)
- added MK27: SPV08A0LR5H-1, Sonar:MIC_SPV08A0LR5H-1, F.Cu at (265.9, 102.9)
- added MK28: SPV08A0LR5H-1, Sonar:MIC_SPV08A0LR5H-1, F.Cu at (253.8, 102.9)
- added MK29: SPV08A0LR5H-1, Sonar:MIC_SPV08A0LR5H-1, F.Cu at (259.9, 115.5)
- added MK30: SPV08A0LR5H-1, Sonar:MIC_SPV08A0LR5H-1, F.Cu at (259.9, 109.2)
- added MK31: SPV08A0LR5H-1, Sonar:MIC_SPV08A0LR5H-1, F.Cu at (253.8, 115.5)
- added MK32: SPV08A0LR5H-1, Sonar:MIC_SPV08A0LR5H-1, F.Cu at (272.0, 109.2)
- added MK33: SPV08A0LR5H-1, Sonar:MIC_SPV08A0LR5H-1, F.Cu at (265.9, 121.8)
- added MK34: SPV08A0LR5H-1, Sonar:MIC_SPV08A0LR5H-1, F.Cu at (259.9, 121.8)
- added MK35: SPV08A0LR5H-1, Sonar:MIC_SPV08A0LR5H-1, F.Cu at (272.0, 102.9)
- added MK36: SPV08A0LR5H-1, Sonar:MIC_SPV08A0LR5H-1, F.Cu at (272.0, 115.5)
- added MK37: SPV08A0LR5H-1, Sonar:MIC_SPV08A0LR5H-1, F.Cu at (265.9, 109.2)
- added MK38: SPV08A0LR5H-1, Sonar:MIC_SPV08A0LR5H-1, F.Cu at (259.9, 102.9)
- added MK39: SPV08A0LR5H-1, Sonar:MIC_SPV08A0LR5H-1, F.Cu at (281.3, 111.3)
- added MK40: SPV08A0LR5H-1, Sonar:MIC_SPV08A0LR5H-1, F.Cu at (299.5, 105.0)
- added MK41: SPV08A0LR5H-1, Sonar:MIC_SPV08A0LR5H-1, F.Cu at (281.3, 105.0)
- added MK42: SPV08A0LR5H-1, Sonar:MIC_SPV08A0LR5H-1, F.Cu at (253.8, 121.8)
- added MK43: SPV08A0LR5H-1, Sonar:MIC_SPV08A0LR5H-1, F.Cu at (293.4, 105.0)
- added MK44: SPV08A0LR5H-1, Sonar:MIC_SPV08A0LR5H-1, F.Cu at (281.3, 123.9)
- added MK45: SPV08A0LR5H-1, Sonar:MIC_SPV08A0LR5H-1, F.Cu at (305.6, 105.0)
- added MK46: SPV08A0LR5H-1, Sonar:MIC_SPV08A0LR5H-1, F.Cu at (244.5, 124.5)
- added MK47: SPV08A0LR5H-1, Sonar:MIC_SPV08A0LR5H-1, F.Cu at (281.3, 117.6)
- added MK48: SPV08A0LR5H-1, Sonar:MIC_SPV08A0LR5H-1, F.Cu at (287.4, 105.0)
- added R133: 5.1k, Resistor_SMD:R_0402_1005Metric, F.Cu at (145.4, 40.6)
- added R134: 5.1k, Resistor_SMD:R_0402_1005Metric, F.Cu at (145.4, 42.6)
- added R135: 100k, Resistor_SMD:R_0402_1005Metric, F.Cu at (148.5, 32.5)
- added TP97: TestPoint_Probe, TestPoint:TestPoint_Pad_D1.0mm, F.Cu at (145.5, 33.0)
- added TP98: TestPoint_Probe, TestPoint:TestPoint_Pad_D1.0mm, F.Cu at (145.5, 36.1)
- added U20: ADS8568SPM, Package_QFP:LQFP-64-1EP_10x10mm_P0.5mm_EP5x5mm_ThermalVias, F.Cu at (188.3, 18.8)
- added U3: ADS8568SPM, Package_QFP:LQFP-64-1EP_10x10mm_P0.5mm_EP5x5mm_ThermalVias, F.Cu at (129.8, 32.8)
- U1: footprint Package_QFP:LQFP-64-1EP_10x10mm_P0.5mm_EP6.5x6.5mm_ThermalVias -> Package_QFP:LQFP-64-1EP_10x10mm_P0.5mm_EP5x5mm_ThermalVias
- moved U1 42.8 mm to (142.8, 13.2)
- moved U26 34.6 mm to (302.0, 48.4)
- moved U29 34.6 mm to (302.0, 64.2)
- moved U30 34.6 mm to (302.0, 56.3)
- moved C79 34.6 mm to (285.2, 55.0)
- moved C80 34.6 mm to (285.2, 57.0)
- moved C81 34.6 mm to (285.2, 58.9)
- moved C91 34.6 mm to (285.2, 62.9)
- moved C92 34.6 mm to (285.2, 64.9)
- moved C93 34.6 mm to (285.2, 66.8)
- moved R123 34.6 mm to (251.4, 97.6)
- moved R125 34.6 mm to (267.0, 99.6)
- moved R126 34.6 mm to (251.4, 99.6)
- moved R128 34.6 mm to (267.0, 101.6)
- moved R129 34.6 mm to (251.4, 101.6)
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Connections:
- R103 pad 2: Net-(MK19--) -> Net-(MK43-OUT)
- R108 pad 2: Net-(MK20--) -> Net-(MK44-OUT)
- R113 pad 2: Net-(MK21--) -> Net-(MK45-OUT)
- R118 pad 2: Net-(MK22--) -> Net-(MK46-OUT)
- R123 pad 2: Net-(MK23--) -> Net-(MK47-OUT)
- R128 pad 2: Net-(MK24--) -> Net-(MK48-OUT)
- R14 pad 2: Net-(MK2--) -> Net-(MK26-OUT)
- R19 pad 2: Net-(MK3--) -> Net-(MK27-OUT)
- R24 pad 2: Net-(MK4--) -> Net-(MK28-OUT)
- R29 pad 2: Net-(MK5--) -> Net-(MK29-OUT)
- R34 pad 2: Net-(MK6--) -> Net-(MK30-OUT)
- R39 pad 2: Net-(MK7--) -> Net-(MK31-OUT)
- R44 pad 2: Net-(MK8--) -> Net-(MK32-OUT)
- R49 pad 2: Net-(MK9--) -> Net-(MK33-OUT)
- R5 pad 2: Net-(MK1--) -> Net-(MK25-OUT)
- R54 pad 2: Net-(MK10--) -> Net-(MK34-OUT)
- R59 pad 2: Net-(MK11--) -> Net-(MK35-OUT)
- R64 pad 2: Net-(MK12--) -> Net-(MK36-OUT)
- R69 pad 2: Net-(MK13--) -> Net-(MK37-OUT)
- R78 pad 2: Net-(MK14--) -> Net-(MK38-OUT)
- R83 pad 2: Net-(MK15--) -> Net-(MK39-OUT)
- R88 pad 2: Net-(MK16--) -> Net-(MK40-OUT)
- R93 pad 2: Net-(MK17--) -> Net-(MK41-OUT)
- R98 pad 2: Net-(MK18--) -> Net-(MK42-OUT)
- TP1 pad 1: /eight_transducer_array/GND -> Net-(MK25-OUT)
- TP10 pad 1: Net-(MK3--) -> Net-(MK30-OUT)
- TP13 pad 1: /eight_transducer_array/GND -> Net-(MK31-OUT)
- TP14 pad 1: Net-(MK4--) -> Net-(MK32-OUT)
- TP17 pad 1: /eight_transducer_array1/GND -> Net-(MK33-OUT)
- TP18 pad 1: Net-(MK5--) -> Net-(MK34-OUT)
- TP2 pad 1: Net-(MK1--) -> Net-(MK26-OUT)
- TP21 pad 1: /eight_transducer_array1/GND -> Net-(MK35-OUT)
- TP22 pad 1: Net-(MK6--) -> Net-(MK36-OUT)
- TP25 pad 1: /eight_transducer_array/GND -> Net-(MK37-OUT)
- TP26 pad 1: Net-(MK7--) -> Net-(MK38-OUT)
- TP29 pad 1: /eight_transducer_array1/GND -> Net-(MK39-OUT)
- TP30 pad 1: Net-(MK8--) -> Net-(MK40-OUT)
- TP33 pad 1: /eight_transducer_array1/GND -> Net-(MK41-OUT)
- TP34 pad 1: Net-(MK9--) -> Net-(MK42-OUT)
- TP37 pad 1: /eight_transducer_array1/GND -> Net-(MK43-OUT)
- TP38 pad 1: Net-(MK10--) -> Net-(MK44-OUT)
- TP41 pad 1: /eight_transducer_array/GND -> Net-(MK45-OUT)
- TP42 pad 1: Net-(MK11--) -> Net-(MK46-OUT)
- TP45 pad 1: /eight_transducer_array1/GND -> Net-(MK47-OUT)
- TP46 pad 1: Net-(MK12--) -> Net-(MK48-OUT)
- TP5 pad 1: /eight_transducer_array1/GND -> Net-(MK27-OUT)
- TP6 pad 1: Net-(MK2--) -> Net-(MK28-OUT)
- TP9 pad 1: /eight_transducer_array/GND -> Net-(MK29-OUT)
- U1 pad 16: /eight_transducer_array/read_out_bus.db15 -> /adc_bus_a.db15
- U1 pad 17: /eight_transducer_array/read_out_bus.db14 -> /adc_bus_a.db14
- U1 pad 18: /eight_transducer_array/read_out_bus.db13 -> /adc_bus_a.db13
- U1 pad 19: /eight_transducer_array/read_out_bus.db12 -> /adc_bus_a.db12
- U1 pad 20: /eight_transducer_array/read_out_bus.db11 -> /adc_bus_a.db11
- U1 pad 21: /eight_transducer_array/read_out_bus.db10 -> /adc_bus_a.db10
- U1 pad 22: /eight_transducer_array/read_out_bus.db9 -> /adc_bus_a.db9
- U1 pad 23: /eight_transducer_array/read_out_bus.db8 -> /adc_bus_a.db8
- U1 pad 26: /eight_transducer_array/read_out_bus.db7 -> /adc_bus_a.db7
- U1 pad 27: /eight_transducer_array/read_out_bus.db6 -> /adc_bus_a.db6
- U1 pad 28: /eight_transducer_array/read_out_bus.db5 -> /adc_bus_a.db5
- U1 pad 29: /eight_transducer_array/read_out_bus.db4 -> /adc_bus_a.db4
- U1 pad 30: /eight_transducer_array/read_out_bus.db3 -> /adc_bus_a.db3
- U1 pad 31: /eight_transducer_array/read_out_bus.db2 -> /adc_bus_a.db2
- U1 pad 32: /eight_transducer_array/read_out_bus.db1 -> /adc_bus_a.db1
- U1 pad 33: /eight_transducer_array/read_out_bus.db0 -> /adc_bus_a.db0
- U1 pad 8: /eight_transducer_array/read_out_bus.par_ser_select -> /adc_bus_a.par_ser_select

Commit message: Josh cooking some more.
Parts:
- removed C1, C12, C13, C16, C17, C18, C19, C2, C5, C56, C57, C6, C60, C61, C62, C63, C7, C8: 10uF, Capacitor_SMD:C_0402_1005Metric
- removed C10, C11, C21, C22, C24, C25, C27, C28, C30, C31, C33, C34, C36, C37, C39, C40, C42, C43, C45, C46, C48, C49, C51, C52, C54, C55, C65, C66, C68, C69, C71, C72, C74, C75, C77, C78, C80, C81, C83, C84, C86, C87, C89, C90, C92, C93, C95, C96: 1.6nF, Capacitor_SMD:C_0402_1005Metric
- removed C14, C15, C3, C4, C58, C59: 0.1uF, Capacitor_SMD:C_0402_1005Metric
- removed C20, C23, C26, C29, C32, C35, C38, C41, C44, C47, C50, C53, C64, C67, C70, C73, C76, C79, C82, C85, C88, C9, C91, C94: 100nF, Capacitor_SMD:C_0402_1005Metric
- removed F1: 1.1A, Diode_SMD:D_1206_3216Metric
- removed J2: DF40C-80DS-0.4V51, Sonar:CONN80_DF40C-80DS_HIR
- removed LS1: Speaker_Ultrasound, Sonar:MA40S4
- removed MK25, MK26, MK27, MK28, MK29, MK30, MK31, MK32, MK33, MK34, MK35, MK36, MK37, MK38, MK39, MK40, MK41, MK42, MK43, MK44, MK45, MK46, MK47, MK48: SPV08A0LR5H-1, Sonar:MIC_SPV08A0LR5H-1
- removed R1, R10, R100, R102, R105, R107, R11, R110, R112, R115, R117, R12, R120, R122, R125, R127, R13, R130, R132, R135, R16, R18, R2, R21, R23, R26, R28, R3, R31, R33, R36, R38, R4, R41, R43, R46, R48, R51, R53, R56, R58, R61, R63, R66, R68, R7, R71, R73, R74, R75, R76, R77, R80, R82, R85, R87, R9, R90, R92, R95, R97: 100k, Resistor_SMD:R_0402_1005Metric
- removed R101, R103, R106, R108, R111, R113, R116, R118, R121, R123, R126, R128, R131, R14, R17, R19, R22, R24, R27, R29, R32, R34, R37, R39, R42, R44, R47, R49, R5, R52, R54, R57, R59, R62, R64, R67, R69, R72, R78, R8, R81, R83, R86, R88, R91, R93, R96, R98: 1k, Resistor_SMD:R_0402_1005Metric
- removed R104, R109, R114, R119, R124, R129, R15, R20, R25, R30, R35, R40, R45, R50, R55, R6, R60, R65, R70, R79, R84, R89, R94, R99: 10k, Resistor_SMD:R_0402_1005Metric
- removed R133, R134: 5.1k, Resistor_SMD:R_0402_1005Metric
- removed TP1, TP10, TP11, TP12, TP13, TP14, TP15, TP16, TP17, TP18, TP19, TP2, TP20, TP21, TP22, TP23, TP24, TP25, TP26, TP27, TP28, TP29, TP3, TP30, TP31, TP32, TP33, TP34, TP35, TP36, TP37, TP38, TP39, TP4, TP40, TP41, TP42, TP43, TP44, TP45, TP46, TP47, TP48, TP5, TP51, TP52, TP55, TP56, TP59, TP6, TP60, TP63, TP64, TP67, TP68, TP7, TP71, TP72, TP75, TP76, TP79, TP8, TP80, TP83, TP84, TP87, TP88, TP9, TP91, TP92, TP95, TP96, TP97, TP98: TestPoint_Probe, TestPoint:TestPoint_Pad_D1.0mm
- removed U1, U20, U3: ADS8568SPM, Package_QFP:LQFP-64-1EP_10x10mm_P0.5mm_EP5x5mm_ThermalVias
- removed U10, U11, U12, U13, U14, U15, U16, U17, U18, U19, U2, U21, U22, U23, U24, U25, U26, U27, U28, U29, U30, U31, U32, U33, U4, U5, U6, U7, U8, U9: Opamp_Dual, Package_SO:TSSOP-8_3x3mm_P0.65mm
- added C1001: 3.3nF, Capacitor_SMD:C_0402_1005Metric, F.Cu at (-41.9, 64.9)
- added C1002: 100nF, Capacitor_SMD:C_0402_1005Metric, F.Cu at (-41.9, 66.9)
- added C1003: 1.6nF, Capacitor_SMD:C_0402_1005Metric, F.Cu at (-41.9, 68.8)
- added C1101: 3.3nF, Capacitor_SMD:C_0402_1005Metric, F.Cu at (-27.0, 77.5)
- added C1102: 100nF, Capacitor_SMD:C_0402_1005Metric, F.Cu at (-27.0, 79.4)
- added C1103: 1.6nF, Capacitor_SMD:C_0402_1005Metric, F.Cu at (-27.0, 81.4)
- added C1201: 3.3nF, Capacitor_SMD:C_0402_1005Metric, F.Cu at (-74.6, 81.8)
- added C1202: 100nF, Capacitor_SMD:C_0402_1005Metric, F.Cu at (-74.6, 83.7)
- added C1203: 1.6nF, Capacitor_SMD:C_0402_1005Metric, F.Cu at (-74.6, 85.7)
- added C1301: 3.3nF, Capacitor_SMD:C_0402_1005Metric, F.Cu at (-12.1, 77.5)
- added C1302: 100nF, Capacitor_SMD:C_0402_1005Metric, F.Cu at (-12.1, 79.4)
- added C1303: 1.6nF, Capacitor_SMD:C_0402_1005Metric, F.Cu at (-12.1, 81.4)
- added C1401: 3.3nF, Capacitor_SMD:C_0402_1005Metric, F.Cu at (-56.8, 102.6)
- added C1402: 100nF, Capacitor_SMD:C_0402_1005Metric, F.Cu at (-56.8, 104.6)
- added C1403: 1.6nF, Capacitor_SMD:C_0402_1005Metric, F.Cu at (-56.8, 106.5)
- added C1501: 3.3nF, Capacitor_SMD:C_0402_1005Metric, F.Cu at (-27.0, 90.0)
- added C1502: 100nF, Capacitor_SMD:C_0402_1005Metric, F.Cu at (-27.0, 92.0)
- added C1503: 1.6nF, Capacitor_SMD:C_0402_1005Metric, F.Cu at (-27.0, 94.0)
- added C1601: 3.3nF, Capacitor_SMD:C_0402_1005Metric, F.Cu at (-41.9, 90.0)
- added C1602: 100nF, Capacitor_SMD:C_0402_1005Metric, F.Cu at (-41.9, 92.0)
- added C1603: 1.6nF, Capacitor_SMD:C_0402_1005Metric, F.Cu at (-41.9, 94.0)
- added C1701: 1uF, Capacitor_SMD:C_0402_1005Metric, F.Cu at (-99.9, 40.3)
- added C1702: 1uF, Capacitor_SMD:C_0402_1005Metric, F.Cu at (-99.9, 42.3)
- added C1703: 1uF, Capacitor_SMD:C_0402_1005Metric, F.Cu at (-99.9, 44.2)
- added C1704: 1uF, Capacitor_SMD:C_0402_1005Metric, F.Cu at (-99.9, 46.2)
- added C1705: 1uF, Capacitor_SMD:C_0402_1005Metric, F.Cu at (-97.0, 40.3)
- added C1706: 10uF, Capacitor_SMD:C_0402_1005Metric, F.Cu at (-97.0, 42.3)
- added C1707: 10uF, Capacitor_SMD:C_0402_1005Metric, F.Cu at (-97.0, 44.2)
- added C1708: 10uF, Capacitor_SMD:C_0402_1005Metric, F.Cu at (-97.0, 46.2)
- added C1709: 10uF, Capacitor_SMD:C_0402_1005Metric, F.Cu at (-94.2, 40.3)
- added C1710: 470nF, Capacitor_SMD:C_0402_1005Metric, F.Cu at (-94.2, 42.3)
- added C1711: 10uF, Capacitor_SMD:C_0402_1005Metric, F.Cu at (-94.2, 44.2)
- added C1712: 0.1uF, Capacitor_SMD:C_0402_1005Metric, F.Cu at (-94.2, 46.2)
- added C1713: 40uF, Capacitor_SMD:C_0402_1005Metric, F.Cu at (-91.3, 40.3)
- added C1714: 1uF, Capacitor_SMD:C_0402_1005Metric, F.Cu at (-91.3, 42.3)
- added C1715: 10uF, Capacitor_SMD:C_0402_1005Metric, F.Cu at (-91.3, 44.2)
- added C1716: 0.1uF, Capacitor_SMD:C_0402_1005Metric, F.Cu at (-91.3, 46.2)
- added C1801: 3.3nF, Capacitor_SMD:C_0402_1005Metric, F.Cu at (-56.8, 77.5)
- added C1802: 100nF, Capacitor_SMD:C_0402_1005Metric, F.Cu at (-56.8, 79.4)
- added C1803: 1.6nF, Capacitor_SMD:C_0402_1005Metric, F.Cu at (-56.8, 81.4)
- added C1901: 3.3nF, Capacitor_SMD:C_0402_1005Metric, F.Cu at (-67.6, 47.7)
- added C1902: 100nF, Capacitor_SMD:C_0402_1005Metric, F.Cu at (-67.6, 49.6)
- added C1903: 1.6nF, Capacitor_SMD:C_0402_1005Metric, F.Cu at (-67.6, 51.6)
- added C2001: 3.3nF, Capacitor_SMD:C_0402_1005Metric, F.Cu at (-44.3, 25.9)
- added C2002: 100nF, Capacitor_SMD:C_0402_1005Metric, F.Cu at (-44.3, 27.8)
- added C2003: 1.6nF, Capacitor_SMD:C_0402_1005Metric, F.Cu at (-44.3, 29.8)
- added C201: 1uF, Capacitor_SMD:C_0402_1005Metric, F.Cu at (-99.9, 89.0)
- added C202: 1uF, Capacitor_SMD:C_0402_1005Metric, F.Cu at (-99.9, 90.9)
- added C203: 1uF, Capacitor_SMD:C_0402_1005Metric, F.Cu at (-99.9, 92.9)
- added C204: 1uF, Capacitor_SMD:C_0402_1005Metric, F.Cu at (-99.9, 94.9)
- added C205: 1uF, Capacitor_SMD:C_0402_1005Metric, F.Cu at (-97.0, 89.0)
- added C206: 10uF, Capacitor_SMD:C_0402_1005Metric, F.Cu at (-97.0, 90.9)
- added C207: 10uF, Capacitor_SMD:C_0402_1005Metric, F.Cu at (-97.0, 92.9)
- added C208: 10uF, Capacitor_SMD:C_0402_1005Metric, F.Cu at (-97.0, 94.9)
- added C209: 10uF, Capacitor_SMD:C_0402_1005Metric, F.Cu at (-94.2, 89.0)
- added C210: 470nF, Capacitor_SMD:C_0402_1005Metric, F.Cu at (-94.2, 90.9)
- added C2101: 3.3nF, Capacitor_SMD:C_0402_1005Metric, F.Cu at (-41.9, 102.6)
- added C2102: 100nF, Capacitor_SMD:C_0402_1005Metric, F.Cu at (-41.9, 104.6)
- added C2103: 1.6nF, Capacitor_SMD:C_0402_1005Metric, F.Cu at (-41.9, 106.5)
- added C211: 10uF, Capacitor_SMD:C_0402_1005Metric, F.Cu at (-94.2, 92.9)
- added C212: 0.1uF, Capacitor_SMD:C_0402_1005Metric, F.Cu at (-94.2, 94.9)
- added C213: 40uF, Capacitor_SMD:C_0402_1005Metric, F.Cu at (-91.3, 89.0)
- added C214: 1uF, Capacitor_SMD:C_0402_1005Metric, F.Cu at (-91.3, 90.9)
- added C215: 10uF, Capacitor_SMD:C_0402_1005Metric, F.Cu at (-91.3, 92.9)
- added C216: 0.1uF, Capacitor_SMD:C_0402_1005Metric, F.Cu at (-91.3, 94.9)
- added C2201: 3.3nF, Capacitor_SMD:C_0402_1005Metric, F.Cu at (-27.0, 64.9)
- added C2202: 100nF, Capacitor_SMD:C_0402_1005Metric, F.Cu at (-27.0, 66.9)
- added C2203: 1.6nF, Capacitor_SMD:C_0402_1005Metric, F.Cu at (-27.0, 68.8)
- added C2301: 3.3nF, Capacitor_SMD:C_0402_1005Metric, F.Cu at (-41.9, 52.3)
- added C2302: 100nF, Capacitor_SMD:C_0402_1005Metric, F.Cu at (-41.9, 54.3)
- added C2303: 1.6nF, Capacitor_SMD:C_0402_1005Metric, F.Cu at (-41.9, 56.3)
- added C2401: 3.3nF, Capacitor_SMD:C_0402_1005Metric, F.Cu at (-56.8, 52.3)
- added C2402: 100nF, Capacitor_SMD:C_0402_1005Metric, F.Cu at (-56.8, 54.3)
- added C2403: 1.6nF, Capacitor_SMD:C_0402_1005Metric, F.Cu at (-56.8, 56.3)
- added C2501: 3.3nF, Capacitor_SMD:C_0402_1005Metric, F.Cu at (-74.6, 94.3)
- added C2502: 100nF, Capacitor_SMD:C_0402_1005Metric, F.Cu at (-74.6, 96.3)
- added C2503: 1.6nF, Capacitor_SMD:C_0402_1005Metric, F.Cu at (-74.6, 98.3)
- added C2601: 3.3nF, Capacitor_SMD:C_0402_1005Metric, F.Cu at (-27.0, 52.3)
- added C2602: 100nF, Capacitor_SMD:C_0402_1005Metric, F.Cu at (-27.0, 54.3)
- added C2603: 1.6nF, Capacitor_SMD:C_0402_1005Metric, F.Cu at (-27.0, 56.3)
- added C2701: 3.3nF, Capacitor_SMD:C_0402_1005Metric, F.Cu at (-74.6, 106.9)
- added C2702: 100nF, Capacitor_SMD:C_0402_1005Metric, F.Cu at (-74.6, 108.9)
- added C2703: 1.6nF, Capacitor_SMD:C_0402_1005Metric, F.Cu at (-74.6, 110.8)
- added C2801: 3.3nF, Capacitor_SMD:C_0402_1005Metric, F.Cu at (-12.1, 64.9)
- added C2802: 100nF, Capacitor_SMD:C_0402_1005Metric, F.Cu at (-12.1, 66.9)
- added C2803: 1.6nF, Capacitor_SMD:C_0402_1005Metric, F.Cu at (-12.1, 68.8)
- added C2901: 1uF, Capacitor_SMD:C_0402_1005Metric, F.Cu at (-67.8, 25.9)
- added C2902: 1uF, Capacitor_SMD:C_0402_1005Metric, F.Cu at (-67.8, 27.8)
- added C2905: 22uF, Capacitor_SMD:C_0402_1005Metric, F.Cu at (-67.8, 29.8)
- added C2906: 22uF, Capacitor_SMD:C_0402_1005Metric, F.Cu at (-67.8, 31.8)
- added C2907: 22uF, Capacitor_SMD:C_0402_1005Metric, F.Cu at (-67.8, 33.7)
- added C2908: 22uF, Capacitor_SMD:C_0402_1005Metric, F.Cu at (-67.8, 35.7)
- added C2909: 22uF, Capacitor_SMD:C_0402_1005Metric, F.Cu at (-64.9, 25.9)
- added C2910: 470nF, Capacitor_SMD:C_0402_1005Metric, F.Cu at (-64.9, 27.8)
- added C2911: 2.2nF, Capacitor_SMD:C_0402_1005Metric, F.Cu at (-64.9, 29.8)
- added C2912: 10uF, Capacitor_SMD:C_0402_1005Metric, F.Cu at (-64.9, 31.8)
- added C2913: 10uF, Capacitor_SMD:C_0402_1005Metric, F.Cu at (-64.9, 33.7)
- added C2914: 1uF, Capacitor_SMD:C_0402_1005Metric, F.Cu at (-64.9, 35.7)
- added C2915: 1uF, Capacitor_SMD:C_0402_1005Metric, F.Cu at (-62.0, 25.9)
- added C2916: 4.7nF, Capacitor_SMD:C_0402_1005Metric, F.Cu at (-62.0, 27.8)
- added C2917: 0.1uF, Capacitor_SMD:C_0402_1005Metric, F.Cu at (-62.0, 29.8)
- added C301: 3.3nF, Capacitor_SMD:C_0402_1005Metric, F.Cu at (-56.8, 64.9)
- added C302: 100nF, Capacitor_SMD:C_0402_1005Metric, F.Cu at (-56.8, 66.9)
- added C303: 1.6nF, Capacitor_SMD:C_0402_1005Metric, F.Cu at (-56.8, 68.8)
- added C401: 1uF, Capacitor_SMD:C_0402_1005Metric, F.Cu at (-99.9, 64.6)
- added C402: 1uF, Capacitor_SMD:C_0402_1005Metric, F.Cu at (-99.9, 66.6)
- added C403: 1uF, Capacitor_SMD:C_0402_1005Metric, F.Cu at (-99.9, 68.6)
- added C404: 1uF, Capacitor_SMD:C_0402_1005Metric, F.Cu at (-99.9, 70.5)
- added C405: 1uF, Capacitor_SMD:C_0402_1005Metric, F.Cu at (-97.0, 64.6)
- added C406: 10uF, Capacitor_SMD:C_0402_1005Metric, F.Cu at (-97.0, 66.6)
- added C407: 10uF, Capacitor_SMD:C_0402_1005Metric, F.Cu at (-97.0, 68.6)
- added C408: 10uF, Capacitor_SMD:C_0402_1005Metric, F.Cu at (-97.0, 70.5)
- added C409: 10uF, Capacitor_SMD:C_0402_1005Metric, F.Cu at (-94.2, 64.6)
- added C410: 470nF, Capacitor_SMD:C_0402_1005Metric, F.Cu at (-94.2, 66.6)
- added C411: 10uF, Capacitor_SMD:C_0402_1005Metric, F.Cu at (-94.2, 68.6)
- added C412: 0.1uF, Capacitor_SMD:C_0402_1005Metric, F.Cu at (-94.2, 70.5)
- added C413: 40uF, Capacitor_SMD:C_0402_1005Metric, F.Cu at (-91.3, 64.6)
- added C414: 1uF, Capacitor_SMD:C_0402_1005Metric, F.Cu at (-91.3, 66.6)
- added C415: 10uF, Capacitor_SMD:C_0402_1005Metric, F.Cu at (-91.3, 68.6)
- added C416: 0.1uF, Capacitor_SMD:C_0402_1005Metric, F.Cu at (-91.3, 70.5)
- added C501: 3.3nF, Capacitor_SMD:C_0402_1005Metric, F.Cu at (-8.70, 25.9)
- added C502: 100nF, Capacitor_SMD:C_0402_1005Metric, F.Cu at (-8.70, 27.8)
- added C503: 1.6nF, Capacitor_SMD:C_0402_1005Metric, F.Cu at (-8.70, 29.8)
- added C601: 3.3nF, Capacitor_SMD:C_0402_1005Metric, F.Cu at (-56.8, 90.0)
- added C602: 100nF, Capacitor_SMD:C_0402_1005Metric, F.Cu at (-56.8, 92.0)
- added C603: 1.6nF, Capacitor_SMD:C_0402_1005Metric, F.Cu at (-56.8, 94.0)
- added C701: 3.3nF, Capacitor_SMD:C_0402_1005Metric, F.Cu at (-12.1, 52.3)
- added C702: 100nF, Capacitor_SMD:C_0402_1005Metric, F.Cu at (-12.1, 54.3)
- added C703: 1.6nF, Capacitor_SMD:C_0402_1005Metric, F.Cu at (-12.1, 56.3)
- added C801: 3.3nF, Capacitor_SMD:C_0402_1005Metric, F.Cu at (-26.5, 25.9)
- added C802: 100nF, Capacitor_SMD:C_0402_1005Metric, F.Cu at (-26.5, 27.8)
- added C803: 1.6nF, Capacitor_SMD:C_0402_1005Metric, F.Cu at (-26.5, 29.8)
- added C901: 3.3nF, Capacitor_SMD:C_0402_1005Metric, F.Cu at (-41.9, 77.5)
- added C902: 100nF, Capacitor_SMD:C_0402_1005Metric, F.Cu at (-41.9, 79.4)
- added C903: 1.6nF, Capacitor_SMD:C_0402_1005Metric, F.Cu at (-41.9, 81.4)
- added F2901: 1.1A, Diode_SMD:D_1206_3216Metric, F.Cu at (-72.5, 38.8)
- added J101: DF40C-80DS-0.4V51, Sonar:CONN80_DF40C-80DS_HIR, F.Cu at (-29.6, 98.4)
- added J2901: USB_C_Receptacle_PowerOnly_6P, Connector_TE-Connectivity:TE_2834006-1_1x01_P4.0mm_Horizontal, F.Cu at (-78.3, 32.9)
- added L2901: 2.2uH, Inductor_SMD:L_0402_1005Metric, F.Cu at (-64.7, 37.7)
- added LS3001: Speaker_Ultrasound, Sonar:MA40S4, F.Cu at (-76.3, 68.4)
- added MK1001: SPV0142LR5H-1, Sonar:MIC_SPV08A0LR5H-1, F.Cu at (-38.8, 66.6)
- added MK1101: SPV0142LR5H-1, Sonar:MIC_SPV08A0LR5H-1, F.Cu at (-23.9, 79.1)
- added MK1201: SPV0142LR5H-1, Sonar:MIC_SPV08A0LR5H-1, F.Cu at (-71.5, 83.4)
- added MK1301: SPV0142LR5H-1, Sonar:MIC_SPV08A0LR5H-1, F.Cu at (-8.95, 79.1)
- added MK1401: SPV0142LR5H-1, Sonar:MIC_SPV08A0LR5H-1, F.Cu at (-53.7, 104.3)
- added MK1501: SPV0142LR5H-1, Sonar:MIC_SPV08A0LR5H-1, F.Cu at (-23.9, 91.7)
- added MK1601: SPV0142LR5H-1, Sonar:MIC_SPV08A0LR5H-1, F.Cu at (-38.8, 91.7)
- added MK1801: SPV0142LR5H-1, Sonar:MIC_SPV08A0LR5H-1, F.Cu at (-53.7, 79.1)
- added MK1901: SPV0142LR5H-1, Sonar:MIC_SPV08A0LR5H-1, F.Cu at (-70.4, 58.5)
- added MK2001: SPV0142LR5H-1, Sonar:MIC_SPV08A0LR5H-1, F.Cu at (-47.0, 36.7)
- added MK2101: SPV0142LR5H-1, Sonar:MIC_SPV08A0LR5H-1, F.Cu at (-38.8, 104.3)
- added MK2201: SPV0142LR5H-1, Sonar:MIC_SPV08A0LR5H-1, F.Cu at (-23.9, 66.6)
- added MK2301: SPV0142LR5H-1, Sonar:MIC_SPV08A0LR5H-1, F.Cu at (-38.8, 54.0)
- added MK2401: SPV0142LR5H-1, Sonar:MIC_SPV08A0LR5H-1, F.Cu at (-53.7, 54.0)
- added MK2501: SPV0142LR5H-1, Sonar:MIC_SPV08A0LR5H-1, F.Cu at (-71.5, 96.0)
- added MK2601: SPV0142LR5H-1, Sonar:MIC_SPV08A0LR5H-1, F.Cu at (-23.9, 54.0)
- added MK2701: SPV0142LR5H-1, Sonar:MIC_SPV08A0LR5H-1, F.Cu at (-71.5, 108.6)
- added MK2801: SPV0142LR5H-1, Sonar:MIC_SPV08A0LR5H-1, F.Cu at (-8.95, 66.6)
- added MK301: SPV0142LR5H-1, Sonar:MIC_SPV08A0LR5H-1, F.Cu at (-53.7, 66.6)
- added MK501: SPV0142LR5H-1, Sonar:MIC_SPV08A0LR5H-1, F.Cu at (-11.5, 36.7)
- added MK601: SPV0142LR5H-1, Sonar:MIC_SPV08A0LR5H-1, F.Cu at (-53.7, 91.7)
- added MK701: SPV0142LR5H-1, Sonar:MIC_SPV08A0LR5H-1, F.Cu at (-8.95, 54.0)
- added MK801: SPV0142LR5H-1, Sonar:MIC_SPV08A0LR5H-1, F.Cu at (-29.3, 36.7)
- added MK901: SPV0142LR5H-1, Sonar:MIC_SPV08A0LR5H-1, F.Cu at (-38.8, 79.1)
- added R1001: 1k, Resistor_SMD:R_0402_1005Metric, F.Cu at (-47.8, 60.2)
- added R1002: 1k, Resistor_SMD:R_0402_1005Metric, F.Cu at (-47.8, 62.2)
- added R1003: 100k, Resistor_SMD:R_0402_1005Metric, F.Cu at (-47.8, 64.2)
- added R1004: 100k, Resistor_SMD:R_0402_1005Metric, F.Cu at (-47.8, 66.2)
- added R1005: 10k, Resistor_SMD:R_0402_1005Metric, F.Cu at (-47.8, 68.2)
- added R1101: 1k, Resistor_SMD:R_0402_1005Metric, F.Cu at (-32.9, 72.8)
- added R1102: 1k, Resistor_SMD:R_0402_1005Metric, F.Cu at (-32.9, 74.8)
- added R1103: 100k, Resistor_SMD:R_0402_1005Metric, F.Cu at (-32.9, 76.8)
- added R1104: 100k, Resistor_SMD:R_0402_1005Metric, F.Cu at (-32.9, 78.8)
- added R1105: 10k, Resistor_SMD:R_0402_1005Metric, F.Cu at (-32.9, 80.8)
- added R1201: 1k, Resistor_SMD:R_0402_1005Metric, F.Cu at (-80.5, 77.1)
- added R1202: 1k, Resistor_SMD:R_0402_1005Metric, F.Cu at (-80.5, 79.1)
- added R1203: 100k, Resistor_SMD:R_0402_1005Metric, F.Cu at (-80.5, 81.1)
- added R1204: 100k, Resistor_SMD:R_0402_1005Metric, F.Cu at (-80.5, 83.1)
- added R1205: 10k, Resistor_SMD:R_0402_1005Metric, F.Cu at (-80.5, 85.1)
- added R1301: 1k, Resistor_SMD:R_0402_1005Metric, F.Cu at (-18.0, 72.8)
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Other:
- board size 10 x 10 mm -> 70 x 100 mm
- board text added: "Made with by Josh and George"
- board text added: "♥"

Commit message: formatting lol
Parts:
- removed C2916: 4.7nF, Capacitor_SMD:C_0402_1005Metric
- removed F2901: 1.1A, Diode_SMD:D_1206_3216Metric
- removed J2901: USB_C_Receptacle_PowerOnly_6P, Connector_TE-Connectivity:TE_2834006-1_1x01_P4.0mm_Horizontal
- removed R2901, R2902: 5.1k, Resistor_SMD:R_0402_1005Metric
- removed TP2903, TP2904, TP2906: TestPoint_Probe, TestPoint:TestPoint_Pad_D1.0mm
- removed U1902, U1903, U2002, U2003, U502, U503, U802, U803: Opamp_Dual, Package_SO:TSSOP-8_3x3mm_P0.65mm
- added C1: 4.7uF, Sonar:C_0603_1608Metric, F.Cu at (-99.2, -8.00)
- added C3: 100nF, Sonar:C_0603_1608Metric, F.Cu at (-99.2, -5.49)
- added C4: 4.7uF, Sonar:C_0603_1608Metric, F.Cu at (-99.2, -2.98)
- added FB1: 120R @ 100MHz, Sonar:L_0603_1608Metric, F.Cu at (-99.2, -0.47)
- added Q1: AO3415, Sonar:SOT-23, F.Cu at (-75.9, -7.03)
- added Q2: AO3415, Sonar:SOT-23, F.Cu at (-75.9, 1.93)
- added R1: 5.1k, Sonar:R_0603_1608Metric, F.Cu at (-99.2, 2.04)
- added R2: 5.1k, Sonar:R_0603_1608Metric, F.Cu at (-99.2, 4.55)
- added R3: 100k, Sonar:R_0603_1608Metric, F.Cu at (-76.4, -3.55)
- added R5: 100k, Sonar:R_0603_1608Metric, F.Cu at (-76.4, 5.41)
- added U1: XT60_M, Sonar:XT60_M_VERTICAL, F.Cu at (-88.8, -3.12)
- added U4: AP63301WU-7, Sonar:TSOT-23-6, F.Cu at (-98.7, 14.6)
- added USB1: TYPE-C 6P, Sonar:TYPE-C-SMD_TYPE-C-6P_1, F.Cu at (69.7, 62.2)
- J101: moved to B.Cu
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Connections:
- C1001 pad 2: /GND -> GND
- C1101 pad 2: /GND -> GND
- C1201 pad 2: /GND -> GND
- C1301 pad 2: /GND -> GND
- C1401 pad 2: /GND -> GND
- C1501 pad 2: /GND -> GND
- C1601 pad 2: /GND -> GND
- C1701 pad 1: /GND -> GND
- C1702 pad 1: /GND -> GND
- C1703 pad 1: /GND -> GND
- C1704 pad 1: /GND -> GND
- C1705 pad 1: /GND -> GND
- C1706 pad 1: /GND -> GND
- C1707 pad 1: /GND -> GND
- C1708 pad 1: /GND -> GND
- C1709 pad 1: /GND -> GND
- C1710 pad 2: /GND -> GND
- C1711 pad 1: /GND -> GND
- C1712 pad 1: /GND -> GND
- C1713 pad 1: /GND -> GND
- C1714 pad 1: /GND -> GND
- C1715 pad 2: /GND -> GND
- C1716 pad 2: /GND -> GND
- C1801 pad 2: /GND -> GND
- C1901 pad 1: Net-(U1902A-+) -> Net-(U1901A-+)
- C1901 pad 2: /GND -> GND
- C1903 pad 2: Net-(U1902A--) -> Net-(U1901A--)
- C2001 pad 1: Net-(U2002A-+) -> Net-(U2001A-+)
- C2001 pad 2: /GND -> GND
- C2003 pad 2: Net-(U2002A--) -> Net-(U2001A--)
- C201 pad 1: /GND -> GND
- C202 pad 1: /GND -> GND
- C203 pad 1: /GND -> GND
- C204 pad 1: /GND -> GND
- C205 pad 1: /GND -> GND
- C206 pad 1: /GND -> GND
- C207 pad 1: /GND -> GND
- C208 pad 1: /GND -> GND
- C209 pad 1: /GND -> GND
- C210 pad 2: /GND -> GND
- C2101 pad 2: /GND -> GND
- C211 pad 1: /GND -> GND
- C212 pad 1: /GND -> GND
- C213 pad 1: /GND -> GND
- C214 pad 1: /GND -> GND
- C215 pad 2: /GND -> GND
- C216 pad 2: /GND -> GND
- C2201 pad 2: /GND -> GND
- C2301 pad 2: /GND -> GND
- C2401 pad 2: /GND -> GND
- C2501 pad 2: /GND -> GND
- C2601 pad 2: /GND -> GND
- C2701 pad 2: /GND -> GND
- C2801 pad 2: /GND -> GND
- C2901 pad 2: /GND -> /power_supply/GND
- C2902 pad 1: /GND -> /power_supply/GND
- C2905 pad 1: /GND -> /power_supply/GND
- C2906 pad 1: /GND -> /power_supply/GND
- C2907 pad 1: /GND -> /power_supply/GND
- C2908 pad 1: /GND -> /power_supply/GND
- C2909 pad 1: /GND -> /power_supply/GND
- C2911 pad 2: /GND -> /power_supply/GND
- C2912 pad 2: /GND -> /power_supply/GND
- C2913 pad 2: /GND -> /power_supply/GND
- C2914 pad 2: /GND -> /power_supply/GND
- C2915 pad 1: /GND -> /power_supply/GND
- C2917 pad 1: /GND -> /power_supply/GND
- C301 pad 2: /GND -> GND
- C401 pad 1: /GND -> GND
- C402 pad 1: /GND -> GND
- C403 pad 1: /GND -> GND
- C404 pad 1: /GND -> GND
- C405 pad 1: /GND -> GND
- C406 pad 1: /GND -> GND
- C407 pad 1: /GND -> GND
- C408 pad 1: /GND -> GND
- C409 pad 1: /GND -> GND
- C410 pad 2: /GND -> GND
- C411 pad 1: /GND -> GND
- C412 pad 1: /GND -> GND
- C413 pad 1: /GND -> GND
- C414 pad 1: /GND -> GND
- C415 pad 2: /GND -> GND
- C416 pad 2: /GND -> GND
- C501 pad 1: Net-(U502A-+) -> Net-(U501A-+)
- C501 pad 2: /GND -> GND
- C503 pad 2: Net-(U502A--) -> Net-(U501A--)
- C601 pad 2: /GND -> GND
- C701 pad 2: /GND -> GND
- C801 pad 1: Net-(U802A-+) -> Net-(U801A-+)
- C801 pad 2: /GND -> GND
- C803 pad 2: Net-(U802A--) -> Net-(U801A--)
- C901 pad 2: /GND -> GND
- J101 pad 1: /GND -> GND
- J101 pad 18: /GND -> GND
- J101 pad 20: /GND -> GND
- J101 pad 37: /GND -> GND
- J101 pad 41: /GND -> GND
- MK1001 pad 3: /GND -> GND
- MK1101 pad 3: /GND -> GND
- MK1201 pad 3: /GND -> GND
- MK1301 pad 3: /GND -> GND
- MK1401 pad 3: /GND -> GND
- MK1501 pad 3: /GND -> GND
- MK1601 pad 3: /GND -> GND
- MK1801 pad 3: /GND -> GND
- MK1901 pad 3: /GND -> GND
- MK2001 pad 3: /GND -> GND
- MK2101 pad 3: /GND -> GND
- MK2201 pad 3: /GND -> GND
- MK2301 pad 3: /GND -> GND
- MK2401 pad 3: /GND -> GND
- MK2501 pad 3: /GND -> GND
- MK2601 pad 3: /GND -> GND
- MK2701 pad 3: /GND -> GND
- MK2801 pad 3: /GND -> GND
- MK301 pad 3: /GND -> GND
- MK501 pad 3: /GND -> GND
- MK601 pad 3: /GND -> GND
- MK701 pad 3: /GND -> GND
- MK801 pad 3: /GND -> GND
- MK901 pad 3: /GND -> GND
- R1002 pad 1: Net-(U601B--) -> Net-(U1001B--)
- R1004 pad 1: Net-(U601B--) -> Net-(U1001B--)
- R1005 pad 2: /GND -> GND
- R1102 pad 1: Net-(U701B--) -> Net-(U1101B--)
- R1104 pad 1: Net-(U701B--) -> Net-(U1101B--)
- R1104 pad 2: /eight_transducer_array1/rx_amp.rx.5 -> /eight_transducer_array1/rx_amp.rx.3
- R1105 pad 2: /GND -> GND
- R1202 pad 1: Net-(U801B--) -> Net-(U1201B--)
- R1204 pad 1: Net-(U801B--) -> Net-(U1201B--)
- R1204 pad 2: /eight_transducer_array1/rx_amp.rx.6 -> /eight_transducer_array1/rx_amp.rx.2
- R1205 pad 2: /GND -> GND
- R1302 pad 1: Net-(U802B--) -> Net-(U1301B--)
- R1304 pad 1: Net-(U802B--) -> Net-(U1301B--)
- R1304 pad 2: /eight_transducer_array1/rx_amp.rx.4 -> /eight_transducer_array1/rx_amp.rx.5
- R1305 pad 2: /GND -> GND
- R1402 pad 1: Net-(U803B--) -> Net-(U1401B--)
- R1404 pad 1: Net-(U803B--) -> Net-(U1401B--)
- R1405 pad 2: /GND -> GND
- R1502 pad 1: Net-(U901B--) -> Net-(U1501B--)
- R1504 pad 1: Net-(U901B--) -> Net-(U1501B--)
- R1504 pad 2: /eight_transducer_array1/rx_amp.rx.3 -> /eight_transducer_array1/rx_amp.rx.7
- R1505 pad 2: /GND -> GND
- R1602 pad 1: Net-(U1001B--) -> Net-(U1601B--)
- R1604 pad 1: Net-(U1001B--) -> Net-(U1601B--)
- R1604 pad 2: /eight_transducer_array1/rx_amp.rx.2 -> /eight_transducer_array1/rx_amp.rx.6
- R1605 pad 2: /GND -> GND
- R1703 pad 2: /GND -> GND
- R1704 pad 2: /GND -> GND
- R1802 pad 1: Net-(U1101B--) -> Net-(U1801B--)
- R1804 pad 1: Net-(U1101B--) -> Net-(U1801B--)
- R1805 pad 2: /GND -> GND
- R1901 pad 1: Net-(U1902A-+) -> Net-(U1901A-+)
- R1902 pad 1: Net-(U1901A--) -> Net-(U1901B--)
- R1903 pad 1: Net-(U1902A--) -> Net-(U1901A--)
- R1904 pad 1: Net-(U1901A--) -> Net-(U1901B--)
- R1904 pad 2: /eight_transducer_array2/rx_amp.rx.1 -> /eight_transducer_array2/rx_amp.rx.4
- R1905 pad 1: Net-(U1902A--) -> Net-(U1901A--)
- R1905 pad 2: /GND -> GND
- R2001 pad 1: Net-(U2002A-+) -> Net-(U2001A-+)
- R2002 pad 1: Net-(U2001A--) -> Net-(U2001B--)
- R2003 pad 1: Net-(U2002A--) -> Net-(U2001A--)
- R2004 pad 1: Net-(U2001A--) -> Net-(U2001B--)
- R2005 pad 1: Net-(U2002A--) -> Net-(U2001A--)
- R2005 pad 2: /GND -> GND
- R203 pad 2: /GND -> GND
- R204 pad 2: /GND -> GND
- R2102 pad 1: Net-(U1201B--) -> Net-(U2101B--)
- R2104 pad 1: Net-(U1201B--) -> Net-(U2101B--)
- R2104 pad 2: /eight_transducer_array2/rx_amp.rx.7 -> /eight_transducer_array2/rx_amp.rx.1
- R2105 pad 2: /GND -> GND
- R2202 pad 1: Net-(U1301B--) -> Net-(U2201B--)
- R2204 pad 1: Net-(U1301B--) -> Net-(U2201B--)
- R2205 pad 2: /GND -> GND
- R2302 pad 1: Net-(U1401B--) -> Net-(U2301B--)
- R2304 pad 1: Net-(U1401B--) -> Net-(U2301B--)
- R2304 pad 2: /eight_transducer_array2/rx_amp.rx.5 -> /eight_transducer_array2/rx_amp.rx.3
- R2305 pad 2: /GND -> GND
- R2402 pad 1: Net-(U1501B--) -> Net-(U2401B--)
- R2404 pad 1: Net-(U1501B--) -> Net-(U2401B--)
- R2404 pad 2: /eight_transducer_array2/rx_amp.rx.6 -> /eight_transducer_array2/rx_amp.rx.2
- R2405 pad 2: /GND -> GND
- R2502 pad 1: Net-(U1601B--) -> Net-(U2501B--)
- R2504 pad 1: Net-(U1601B--) -> Net-(U2501B--)
- R2504 pad 2: /eight_transducer_array2/rx_amp.rx.4 -> /eight_transducer_array2/rx_amp.rx.5
- R2505 pad 2: /GND -> GND
- R2602 pad 1: Net-(U1801B--) -> Net-(U2601B--)
- R2604 pad 1: Net-(U1801B--) -> Net-(U2601B--)
- R2605 pad 2: /GND -> GND
- R2702 pad 1: Net-(U1901B--) -> Net-(U2701B--)
- R2704 pad 1: Net-(U1901B--) -> Net-(U2701B--)
- R2704 pad 2: /eight_transducer_array2/rx_amp.rx.3 -> /eight_transducer_array2/rx_amp.rx.7
- R2705 pad 2: /GND -> GND
- R2802 pad 1: Net-(U1902B--) -> Net-(U2801B--)
- R2804 pad 1: Net-(U1902B--) -> Net-(U2801B--)
- R2804 pad 2: /eight_transducer_array2/rx_amp.rx.2 -> /eight_transducer_array2/rx_amp.rx.6
- R2805 pad 2: /GND -> GND
- R305 pad 2: /GND -> GND
- R3101 pad 2: /GND -> /power_supply/5v_12v_boost/GND
- R403 pad 2: /GND -> GND
- R404 pad 2: /GND -> GND
- R501 pad 1: Net-(U502A-+) -> Net-(U501A-+)
- R502 pad 1: Net-(U501A--) -> Net-(U501B--)
- R503 pad 1: Net-(U502A--) -> Net-(U501A--)
- R504 pad 1: Net-(U501A--) -> Net-(U501B--)
- R504 pad 2: /eight_transducer_array1/rx_amp.rx.1 -> /eight_transducer_array1/rx_amp.rx.4
- R505 pad 1: Net-(U502A--) -> Net-(U501A--)
- R505 pad 2: /GND -> GND
- R602 pad 1: Net-(U501B--) -> Net-(U601B--)
- R604 pad 1: Net-(U501B--) -> Net-(U601B--)
- R605 pad 2: /GND -> GND
- R702 pad 1: Net-(U502B--) -> Net-(U701B--)
- R704 pad 1: Net-(U502B--) -> Net-(U701B--)
- R705 pad 2: /GND -> GND
- R801 pad 1: Net-(U802A-+) -> Net-(U801A-+)
- R802 pad 1: Net-(U801A--) -> Net-(U801B--)
- R803 pad 1: Net-(U802A--) -> Net-(U801A--)
- R804 pad 1: Net-(U801A--) -> Net-(U801B--)
- R805 pad 1: Net-(U802A--) -> Net-(U801A--)
- R805 pad 2: /GND -> GND
- R902 pad 1: Net-(U503B--) -> Net-(U901B--)
- R904 pad 1: Net-(U503B--) -> Net-(U901B--)
- R904 pad 2: /eight_transducer_array1/rx_amp.rx.7 -> /eight_transducer_array1/rx_amp.rx.1
- R905 pad 2: /GND -> GND
- TP1101 pad 1: /eight_transducer_array1/rx_amp.rx.5 -> /eight_transducer_array1/rx_amp.rx.3
- TP1201 pad 1: /eight_transducer_array1/rx_amp.rx.6 -> /eight_transducer_array1/rx_amp.rx.2
- TP1301 pad 1: /eight_transducer_array1/rx_amp.rx.4 -> /eight_transducer_array1/rx_amp.rx.5
- TP1501 pad 1: /eight_transducer_array1/rx_amp.rx.3 -> /eight_transducer_array1/rx_amp.rx.7
- TP1601 pad 1: /eight_transducer_array1/rx_amp.rx.2 -> /eight_transducer_array1/rx_amp.rx.6
- TP1901 pad 1: /eight_transducer_array2/rx_amp.rx.1 -> /eight_transducer_array2/rx_amp.rx.4
- TP2101 pad 1: /eight_transducer_array2/rx_amp.rx.7 -> /eight_transducer_array2/rx_amp.rx.1
- TP2301 pad 1: /eight_transducer_array2/rx_amp.rx.5 -> /eight_transducer_array2/rx_amp.rx.3
- TP2401 pad 1: /eight_transducer_array2/rx_amp.rx.6 -> /eight_transducer_array2/rx_amp.rx.2
- TP2501 pad 1: /eight_transducer_array2/rx_amp.rx.4 -> /eight_transducer_array2/rx_amp.rx.5
- TP2701 pad 1: /eight_transducer_array2/rx_amp.rx.3 -> /eight_transducer_array2/rx_amp.rx.7
- TP2801 pad 1: /eight_transducer_array2/rx_amp.rx.2 -> /eight_transducer_array2/rx_amp.rx.6
- TP3102 pad 1: /power_supply/VBUS -> /power_mux/Vout
- TP501 pad 1: /eight_transducer_array1/rx_amp.rx.1 -> /eight_transducer_array1/rx_amp.rx.4
- TP901 pad 1: /eight_transducer_array1/rx_amp.rx.7 -> /eight_transducer_array1/rx_amp.rx.1
- U1001 pad 4: /eight_transducer_array1/-2.5V -> /eight_transducer_array/-2.5V
- U1001 pad 5: /GND -> GND
- U1001 pad 7: /eight_transducer_array1/rx_amp.rx.2 -> /eight_transducer_array/rx_amp.rx.3
- U1001 pad 8: /eight_transducer_array1/2.5V -> /eight_transducer_array/2.5V
- U1101 pad 4: /eight_transducer_array/-2.5V -> /eight_transducer_array1/-2.5V
- U1101 pad 5: /GND -> GND
- U1101 pad 7: /eight_transducer_array/rx_amp.rx.5 -> /eight_transducer_array1/rx_amp.rx.3
- U1101 pad 8: /eight_transducer_array/2.5V -> /eight_transducer_array1/2.5V
- U1201 pad 4: /eight_transducer_array2/-2.5V -> /eight_transducer_array1/-2.5V
- U1201 pad 5: /GND -> GND
- U1201 pad 7: /eight_transducer_array2/rx_amp.rx.7 -> /eight_transducer_array1/rx_amp.rx.2
- U1201 pad 8: /eight_transducer_array2/2.5V -> /eight_transducer_array1/2.5V
- U1301 pad 4: /eight_transducer_array/-2.5V -> /eight_transducer_array1/-2.5V
- U1301 pad 5: /GND -> GND
- U1301 pad 7: /eight_transducer_array/rx_amp.rx.6 -> /eight_transducer_array1/rx_amp.rx.5
- U1301 pad 8: /eight_transducer_array/2.5V -> /eight_transducer_array1/2.5V
- U1401 pad 4: /eight_transducer_array2/-2.5V -> /eight_transducer_array/-2.5V
- U1401 pad 5: /GND -> GND
- U1401 pad 7: /eight_transducer_array2/rx_amp.rx.5 -> /eight_transducer_array/rx_amp.rx.4
- U1401 pad 8: /eight_transducer_array2/2.5V -> /eight_transducer_array/2.5V
- U1501 pad 4: /eight_transducer_array2/-2.5V -> /eight_transducer_array1/-2.5V
- U1501 pad 5: /GND -> GND
- U1501 pad 7: /eight_transducer_array2/rx_amp.rx.6 -> /eight_transducer_array1/rx_amp.rx.7
- U1501 pad 8: /eight_transducer_array2/2.5V -> /eight_transducer_array1/2.5V
- U1601 pad 4: /eight_transducer_array2/-2.5V -> /eight_transducer_array1/-2.5V
- U1601 pad 5: /GND -> GND
- U1601 pad 7: /eight_transducer_array2/rx_amp.rx.4 -> /eight_transducer_array1/rx_amp.rx.6
- U1601 pad 8: /eight_transducer_array2/2.5V -> /eight_transducer_array1/2.5V
- U1701 pad 11: /eight_transducer_array2/refen_~{wr} -> /refen_~{wr}
- U1701 pad 12: /eight_transducer_array2/read -> /synced_read
- U1701 pad 13: /eight_transducer_array2/chip_select_frame_sync -> /chip_select_frame_sync
- U1701 pad 15: /GND -> GND
- U1701 pad 24: /GND -> GND
- U1701 pad 3: /GND -> GND
- U1701 pad 37: /eight_transducer_array2/adc_conv_start -> /start_conv
- U1701 pad 38: /eight_transducer_array2/adc_conv_start -> /start_conv
- U1701 pad 39: /eight_transducer_array2/adc_conv_start -> /start_conv
- U1701 pad 40: /eight_transducer_array2/adc_conv_start -> /start_conv
- U1701 pad 41: /eight_transducer_array2/~{hw}_sw_select -> /~{hw}_sw_select
- U1701 pad 44: /GND -> GND
- U1701 pad 46: /GND -> GND
- U1701 pad 5: /GND -> GND
- U1701 pad 51: /GND -> GND
- U1701 pad 53: /GND -> GND
- U1701 pad 55: /GND -> GND
- U1701 pad 58: /GND -> GND
- U1701 pad 60: /GND -> GND
- U1701 pad 62: /GND -> GND
- U1701 pad 8: /eight_transducer_array2/par_ser_select -> /par_ser_select
- U1801 pad 5: /GND -> GND
- U1801 pad 7: /eight_transducer_array/rx_amp.rx.7 -> /eight_transducer_array/rx_amp.rx.5
- U1901 pad 1: /eight_transducer_array2/rx_amp.rx.1 -> Net-(C1903-Pad1)
- U1901 pad 3: /GND -> Net-(U1901A-+)
- U1901 pad 5: /GND -> GND
- U1901 pad 7: /eight_transducer_array2/rx_amp.rx.3 -> /eight_transducer_array2/rx_amp.rx.4
- U2001 pad 1: /eight_transducer_array2/rx_amp.rx.0 -> Net-(C2003-Pad1)
- U2001 pad 3: /GND -> Net-(U2001A-+)
- U2001 pad 4: (no net) -> /eight_transducer_array2/-2.5V
- U2001 pad 5: (no net) -> GND
- U2001 pad 6: (no net) -> Net-(U2001B--)
- U2001 pad 7: (no net) -> /eight_transducer_array2/rx_amp.rx.0
- U2001 pad 8: (no net) -> /eight_transducer_array2/2.5V
- U201 pad 15: /GND -> GND
- U201 pad 16: /eight_transducer_array/read_out_bus.db15 -> /adc_bus_a.db15
- U201 pad 17: /eight_transducer_array/read_out_bus.db14 -> /adc_bus_a.db14
- U201 pad 18: /eight_transducer_array/read_out_bus.db13 -> /adc_bus_a.db13
- U201 pad 19: /eight_transducer_array/read_out_bus.db12 -> /adc_bus_a.db12
- U201 pad 20: /eight_transducer_array/read_out_bus.db11 -> /adc_bus_a.db11
- U201 pad 21: /eight_transducer_array/read_out_bus.db10 -> /adc_bus_a.db10
- U201 pad 22: /eight_transducer_array/read_out_bus.db9 -> /adc_bus_a.db9
- U201 pad 23: /eight_transducer_array/read_out_bus.db8 -> /adc_bus_a.db8
- U201 pad 24: /GND -> GND
- U201 pad 26: /eight_transducer_array/read_out_bus.db7 -> /adc_bus_a.db7
- U201 pad 27: /eight_transducer_array/read_out_bus.db6 -> /adc_bus_a.db6
- U201 pad 28: /eight_transducer_array/read_out_bus.db5 -> /adc_bus_a.db5
- U201 pad 29: /eight_transducer_array/read_out_bus.db4 -> /adc_bus_a.db4
- U201 pad 3: /GND -> GND
- U201 pad 30: /eight_transducer_array/read_out_bus.db3 -> /adc_bus_a.db3
- U201 pad 31: /eight_transducer_array/read_out_bus.db2 -> /adc_bus_a.db2
- U201 pad 32: /eight_transducer_array/read_out_bus.db1 -> /adc_bus_a.db1
- U201 pad 33: /eight_transducer_array/read_out_bus.db0 -> /adc_bus_a.db0
- U201 pad 44: /GND -> GND
- U201 pad 46: /GND -> GND
- U201 pad 5: /GND -> GND
- U201 pad 51: /GND -> GND
- U201 pad 53: /GND -> GND
- U201 pad 55: /GND -> GND
- U201 pad 58: /GND -> GND
- U201 pad 60: /GND -> GND
- U201 pad 62: /GND -> GND
- U2101 pad 4: (no net) -> /eight_transducer_array2/-2.5V
- U2101 pad 5: (no net) -> GND
- U2101 pad 6: (no net) -> Net-(U2101B--)
- U2101 pad 7: (no net) -> /eight_transducer_array2/rx_amp.rx.1
- U2101 pad 8: (no net) -> /eight_transducer_array2/2.5V
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