File: sonar-v1-pcb/sonar.kicad_sch (KiCad schematic)
At the start: 17 parts

Commit message: ragebait
Parts:
- removed MK1, MK10, MK11, MK12, MK13, MK14, MK15, MK16, MK2, MK3, MK4, MK5, MK6, MK7, MK8, MK9: Microphone_Ultrasound, Sonar:MA40S4, symbol Device:Microphone_Ultrasound
Other:
- added sheet eight_transducer_array (eight_transducer_array.kicad_sch)
- added sheet eight_transducer_array1 (eight_transducer_array.kicad_sch)
- added sheet eight_transducer_array2 (eight_transducer_array.kicad_sch)
- title: (none) -> Phased Fizzing
- moved on the sheet: LS1
