File: sonar-v1-pcb/eight_transducer_array.kicad_sch (KiCad schematic)
At the start: 1 part, among them U1 ADS8568SPM

Commit message: added some adc shit
Parts:
- added C25, C28, C31, C34, C37, C43: 10uF, symbol Device:C
- added C40, C44: 0.1uF, symbol Device:C
- added R121, R124, R127, R130: 100k, symbol Device:R_US
Connections:
- net 20V is gone; now on net 10V: U1.48 (HVDD)
- net 10V: now also C37.2, C40.2; no longer U1.15 (AGND), U1.24 (DGND), U1.44 (AGND), U1.5 (AGND), U1.51 (AGND), U1.58 (AGND), U1.62 (AGND)
- net GND: now also U1.15 (AGND), U1.24 (DGND), U1.3 (REFDN), U1.44 (AGND), U1.46 (REFAN), U1.5 (AGND), U1.51 (AGND), U1.53 (REFBN), U1.58 (AGND), U1.60 (REFCN), U1.62 (AGND), C25.1, C28.1, C31.1, C34.1, C37.1, C40.1, C43.2, C44.2, R121.2, R124.2, R127.2, R130.2; no longer U1.1 (HVSS)
- net reset: now reaches U1.10 (RESET)
- net reset: now also R127.1
- net read_allow: now reaches U1.12 (RD_N)
- net read_allow: now also R124.1
- net chip_select_frame_sync: now reaches U1.13 (CS_FS_N)
- net sleep_select: now reaches U1.36 (ASLEEP)
- net sleep_select: now also R121.1
- net at U1.43 (REFAP): now also C25.2
- net at U1.50 (REFBP): now also C28.2
- net at U1.6 (REFDP): now also C34.2
- net at U1.63 (REFCP): now also C31.2
- net read_out_bus.par_ser_select: now reaches U1.8 (PAR_SER_N)
- net standby: now reaches U1.9 (STBY_N)
- net standby: now also R130.1
- net 15V renamed 5V
- new net -10V: C43.1, C44.1, U1.1 (HVSS)
Other:
- sheet rx_amp_0 ports: added -10V; removed 20V
- sheet rx_amp_1 ports: added -10V; removed 20V
- sheet rx_amp_2 ports: added -10V; removed 20V
- sheet rx_amp_3 ports: added -10V; removed 20V
- sheet rx_amp_4 ports: added -10V; removed 20V
- sheet rx_amp_5 ports: added -10V; removed 20V
- sheet rx_amp_6 ports: added -10V; removed 20V
- sheet rx_amp_7 ports: added -10V; removed 20V
- note added: "Always Permit Reads"
- note added: "DO WE NEED THESE????"
- note added: "Never reset"
- note added: "Never sleep"
- note added: "Never turn off"

Commit message: fix bandpass
Parts:
- C25, C28, C31, C34, C37, C40, C43, C44: footprint (none) -> Capacitor_SMD:C_0402_1005Metric
- R121, R124, R127, R130: footprint (none) -> Resistor_SMD:R_0402_1005Metric
Connections:
- net 5V: no longer U1.25 (DVDD)
- new net 3.3: U1.25 (DVDD)
Changed lines of the file:
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@@
 	)
 	(junction
-		(at 135.89 46.99)
-		(diameter 0)
-		(color 0 0 0 0)
-	)
-	(junction
 		(at 134.62 97.79)
 		(diameter 0)
@@
 	(wire
 		(pts
-			(xy 20.32 132.08) (xy 22.86 132.08)
+			(xy 132.08 52.07) (xy 138.43 52.07)
 		)
 		(stroke
@@
 		)
 	)
-	(bus
+	(wire
 		(pts
-			(xy 224.79 39.37) (xy 224.79 49.53)
+			(xy 20.32 132.08) (xy 22.86 132.08)
 		)
 		(stroke
@@
 	(bus
 		(pts
-			(xy 224.79 80.01) (xy 224.79 82.55)
+			(xy 224.79 39.37) (xy 224.79 49.53)
 		)
 		(stroke
@@
 		)
 	)
-	(wire
+	(bus
 		(pts
-			(xy 134.62 100.33) (xy 134.62 97.79)
+			(xy 224.79 80.01) (xy 224.79 82.55)
 		)
 		(stroke
@@
 	(wire
 		(pts
-			(xy 138.43 52.07) (xy 135.89 52.07)
+			(xy 134.62 100.33) (xy 134.62 97.79)
 		)
 		(stroke
@@
 		)
 	)
-	(wire
-		(pts
-			(xy 135.89 46.99) (xy 135.89 52.07)
-		)
-		(stroke
-			(width 0)
-			(type default)
-		)
-	)
 	(bus
 		(pts
@@
 		)
 	)
+	(hierarchical_label "3.3"
+		(shape input)
+		(at 132.08 52.07 180)
+		(effects
+			(font
+				(size 1.27 1.27)
+			)
+			(justify right)
+		)
+	)
 	(hierarchical_label "GND"
 		(shape input)
@@
 			)
 		)
-		(property "Footprint" ""
+		(property "Footprint" "Resistor_SMD:R_0402_1005Metric"
 			(at 249.936 127.254 90)
 			(effects
@@
 			)
 		)
-		(property "Footprint" ""
+		(property "Footprint" "Capacitor_SMD:C_0402_1005Metric"
 			(at 106.9848 162.56 0)
 			(effects
@@
 			)
 		)
-		(property "Footprint" ""
+		(property "Footprint" "Resistor_SMD:R_0402_1005Metric"
 			(at 229.616 127.254 90)
 			(effects
@@
 			)
 		)
-		(property "Footprint" ""
+		(property "Footprint" "Resistor_SMD:R_0402_1005Metric"
 			(at 229.616 152.654 90)
 			(effects
@@
 			)
 		)
-		(property "Footprint" ""
+		(property "Footprint" "Capacitor_SMD:C_0402_1005Metric"
 			(at 135.89 114.6048 0)
 			(effects
@@
 			)
 		)
-		(property "Footprint" ""
+		(property "Footprint" "Resistor_SMD:R_0402_1005Metric"
 			(at 267.716 127.254 90)
 			(effects
@@
 			)
 		)
-		(property "Footprint" ""
+		(property "Footprint" "Capacitor_SMD:C_0402_1005Metric"
 			(at 135.89 129.8448 0)
 			(effects
@@
 			)
 		)
-		(property "Footprint" ""
+		(property "Footprint" "Capacitor_SMD:C_0402_1005Metric"
 			(at 118.4148 162.56 0)
 			(effects
@@
 			)
 		)
-		(property "Footprint" ""
+		(property "Footprint" "Capacitor_SMD:C_0402_1005Metric"
 			(at 135.89 122.2248 0)
 			(effects
@@
 			)
 		)
-		(property "Footprint" ""
+		(property "Footprint" "Capacitor_SMD:C_0402_1005Metric"
 			(at 118.4148 172.72 0)
 			(effects
@@
 			)
 		)
-		(property "Footprint" ""
+		(property "Footprint" "Capacitor_SMD:C_0402_1005Metric"
 			(at 135.89 106.9848 0)
 			(effects
@@
 			)
 		)
-		(property "Footprint" ""
+		(property "Footprint" "Capacitor_SMD:C_0402_1005Metric"
 			(at 106.9848 172.72 0)
 			(effects

Commit message: Add lowpas filter
Parts:
- U: renamed from U1; footprint Package_QFP:LQFP-64-1EP_10x10mm_P0.5mm_EP6.5x6.5mm_ThermalVias -> PM0064A-IPC_A
- renumbered C25 to C, R121 to R
Other:
- sheet rx_amp_0 ports: added -2.5V, 2.5V; removed -10V, 10V
- sheet rx_amp_1 ports: added -2.5V, 2.5V; removed -10V, 10V
- sheet rx_amp_2 ports: added -2.5V, 2.5V; removed -10V, 10V
- sheet rx_amp_3 ports: added -2.5V, 2.5V; removed -10V, 10V
- sheet rx_amp_4 ports: added -2.5V, 2.5V; removed -10V, 10V
- sheet rx_amp_5 ports: added -2.5V, 2.5V; removed -10V, 10V
- sheet rx_amp_6 ports: added -2.5V, 2.5V; removed -10V, 10V
- sheet rx_amp_7 ports: added -2.5V, 2.5V; removed -10V, 10V

Commit message: finish ADC signals
Parts:
- renumbered C to C57, R to R77, U to U18
Connections:
- net refen_~{wr}: now reaches U18.11 (REFEN_WR_N)
- net range_xclk: now reaches U18.34 (RANGE_XCLK)
- net adc_busy: now reaches U18.35 (BUSY_INT)
- net hw_sw_select: now reaches U18.41 (HW_SW_N)
Other:
- note added: "4.5mA max"
- note added: "430.1mW max power disipation"
- note added: "50.1mA max 37.9mA typ"

Commit message: kept cooking
Parts:
- renumbered C37 to C1, C43 to C2, C40 to C3, C44 to C4, C57 to C5, C28 to C6, C31 to C7, C34 to C8, R127 to R1, R130 to R2, R124 to R3, R77 to R4, U18 to U1
Other:
- note added: "208mA max draw on both rails"
- note added: "ADC Power Consumption"
Changed lines of the file:
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@@
 	)
 	(rectangle
+		(start 91.44 151.13)
+		(end 154.94 186.69)
+		(stroke
+			(width 0)
+			(type default)
+		)
+		(fill
+			(type none)
+		)
+	)
+	(rectangle
 		(start 264.16 113.03)
 		(end 280.67 135.89)
@@
 		)
 	)
+	(text "208mA max draw on both rails"
+		(exclude_from_sim no)
+		(at 77.47 55.626 0)
+		(effects
+			(font
+				(size 1.27 1.27)
+			)
+		)
+	)
+	(text "ADC Power Consumption"
+		(exclude_from_sim no)
+		(at 122.936 153.924 0)
+		(effects
+			(font
+				(size 1.27 1.27)
+			)
+		)
+	)
 	(text "Never reset"
 		(exclude_from_sim no)
@@
 		(dnp no)
 		(fields_autoplaced yes)
-		(property "Reference" "U?"
+		(property "Reference" "U1"
 			(at 166.37 24.13 0)
 			(effects
@@
 			(project "sonar"
 				(path "/f72ceae0-eee4-4385-b0e8-639846bcb5f2/68d332b8-de02-4694-8619-1c5597a76eff"
-					(reference "U18")
+					(reference "U20")
 					(unit 1)
 				)
 				(path "/f72ceae0-eee4-4385-b0e8-639846bcb5f2/d78844ef-eb5d-4b24-a5c3-8824db20c2bc"
-					(reference "U?")
+					(reference "U1")
 					(unit 1)
 				)
 				(path "/f72ceae0-eee4-4385-b0e8-639846bcb5f2/dbee82a7-8e4c-4ab8-a9a7-41d31ebc4a60"
-					(reference "U1")
+					(reference "U3")
 					(unit 1)
 				)
@@
 		(dnp no)
 		(fields_autoplaced yes)
-		(property "Reference" "R124"
+		(property "Reference" "R3"
 			(at 251.46 125.7299 0)
 			(effects
@@
 				)
 				(path "/f72ceae0-eee4-4385-b0e8-639846bcb5f2/d78844ef-eb5d-4b24-a5c3-8824db20c2bc"
-					(reference "R124")
+					(reference "R3")
 					(unit 1)
 				)
 				(path "/f72ceae0-eee4-4385-b0e8-639846bcb5f2/dbee82a7-8e4c-4ab8-a9a7-41d31ebc4a60"
-					(reference "R8")
+					(reference "R12")
 					(unit 1)
 				)
@@
 		(on_board yes)
 		(dnp no)
-		(property "Reference" "C37"
+		(property "Reference" "C1"
 			(at 104.648 167.64 0)
 			(effects
@@
 			(project "sonar"
 				(path "/f72ceae0-eee4-4385-b0e8-639846bcb5f2/68d332b8-de02-4694-8619-1c5597a76eff"
-					(reference "C49")
+					(reference "C56")
 					(unit 1)
 				)
 				(path "/f72ceae0-eee4-4385-b0e8-639846bcb5f2/d78844ef-eb5d-4b24-a5c3-8824db20c2bc"
-					(reference "C37")
+					(reference "C1")
 					(unit 1)
 				)
 				(path "/f72ceae0-eee4-4385-b0e8-639846bcb5f2/dbee82a7-8e4c-4ab8-a9a7-41d31ebc4a60"
-					(reference "C4")
+					(reference "C12")
 					(unit 1)
 				)
@@
 		(dnp no)
 		(fields_autoplaced yes)
-		(property "Reference" "R127"
+		(property "Reference" "R1"
 			(at 231.14 125.7299 0)
 			(effects
@@
 				)
 				(path "/f72ceae0-eee4-4385-b0e8-639846bcb5f2/d78844ef-eb5d-4b24-a5c3-8824db20c2bc"
-					(reference "R127")
+					(reference "R1")
 					(unit 1)
 				)
 				(path "/f72ceae0-eee4-4385-b0e8-639846bcb5f2/dbee82a7-8e4c-4ab8-a9a7-41d31ebc4a60"
-					(reference "R6")
+					(reference "R10")
 					(unit 1)
 				)
@@
 		(dnp no)
 		(fields_autoplaced yes)
-		(property "Reference" "R130"
+		(property "Reference" "R2"
 			(at 231.14 151.1299 0)
 			(effects
@@
 				)
 				(path "/f72ceae0-eee4-4385-b0e8-639846bcb5f2/d78844ef-eb5d-4b24-a5c3-8824db20c2bc"
-					(reference "R130")
+					(reference "R2")
 					(unit 1)
 				)
 				(path "/f72ceae0-eee4-4385-b0e8-639846bcb5f2/dbee82a7-8e4c-4ab8-a9a7-41d31ebc4a60"
-					(reference "R7")
+					(reference "R11")
 					(unit 1)
 				)
@@
 		(on_board yes)
 		(dnp no)
-		(property "Reference" "C28"
+		(property "Reference" "C6"
 			(at 130.81 112.268 90)
 			(effects
@@
 			(project "sonar"
 				(path "/f72ceae0-eee4-4385-b0e8-639846bcb5f2/68d332b8-de02-4694-8619-1c5597a76eff"
-					(reference "C58")
+					(reference "C61")
 					(unit 1)
 				)
 				(path "/f72ceae0-eee4-4385-b0e8-639846bcb5f2/d78844ef-eb5d-4b24-a5c3-8824db20c2bc"
-					(reference "C28")
+					(reference "C6")
 					(unit 1)
 				)
 				(path "/f72ceae0-eee4-4385-b0e8-639846bcb5f2/dbee82a7-8e4c-4ab8-a9a7-41d31ebc4a60"
-					(reference "C9")
+					(reference "C17")
 					(unit 1)
 				)
@@
 		(dnp no)
 		(fields_autoplaced yes)
-		(property "Reference" "R?"
+		(property "Reference" "R4"
 			(at 269.24 125.7299 0)
 			(effects
@@
 				)
 				(path "/f72ceae0-eee4-4385-b0e8-639846bcb5f2/d78844ef-eb5d-4b24-a5c3-8824db20c2bc"
-					(reference "R?")
+					(reference "R4")
 					(unit 1)
 				)
 				(path "/f72ceae0-eee4-4385-b0e8-639846bcb5f2/dbee82a7-8e4c-4ab8-a9a7-41d31ebc4a60"
-					(reference "R9")
+					(reference "R13")
 					(unit 1)
 				)
@@
 		(on_board yes)
 		(dnp no)
-		(property "Reference" "C34"
+		(property "Reference" "C8"
 			(at 130.81 127.508 90)
 			(effects
@@
 			(project "sonar"
 				(path "/f72ceae0-eee4-4385-b0e8-639846bcb5f2/68d332b8-de02-4694-8619-1c5597a76eff"
-					(reference "C60")
+					(reference "C63")
 					(unit 1)
 				)
 				(path "/f72ceae0-eee4-4385-b0e8-639846bcb5f2/d78844ef-eb5d-4b24-a5c3-8824db20c2bc"
-					(reference "C34")
+					(reference "C8")
 					(unit 1)
 				)
 				(path "/f72ceae0-eee4-4385-b0e8-639846bcb5f2/dbee82a7-8e4c-4ab8-a9a7-41d31ebc4a60"
-					(reference "C14")
+					(reference "C19")
 					(unit 1)
 				)
@@
 		(on_board yes)
 		(dnp no)
-		(property "Reference" "C40"
+		(property "Reference" "C3"
 			(at 116.078 167.64 0)
 			(effects
@@
 			(project "sonar"
 				(path "/f72ceae0-eee4-4385-b0e8-639846bcb5f2/68d332b8-de02-4694-8619-1c5597a76eff"
-					(reference "C51")
+					(reference "C58")
 					(unit 1)
 				)
 				(path "/f72ceae0-eee4-4385-b0e8-639846bcb5f2/d78844ef-eb5d-4b24-a5c3-8824db20c2bc"
-					(reference "C40")
+					(reference "C3")
 					(unit 1)
 				)
 				(path "/f72ceae0-eee4-4385-b0e8-639846bcb5f2/dbee82a7-8e4c-4ab8-a9a7-41d31ebc4a60"
-					(reference "C6")
+					(reference "C14")
 					(unit 1)
 				)
@@
 		(on_board yes)
 		(dnp no)
-		(property "Reference" "C31"
+		(property "Reference" "C7"
 			(at 130.81 119.888 90)
 			(effects
@@
 			(project "sonar"
 				(path "/f72ceae0-eee4-4385-b0e8-639846bcb5f2/68d332b8-de02-4694-8619-1c5597a76eff"
-					(reference "C59")
+					(reference "C62")
 					(unit 1)
 				)
 				(path "/f72ceae0-eee4-4385-b0e8-639846bcb5f2/d78844ef-eb5d-4b24-a5c3-8824db20c2bc"
-					(reference "C31")
+					(reference "C7")
 					(unit 1)
 				)
 				(path "/f72ceae0-eee4-4385-b0e8-639846bcb5f2/dbee82a7-8e4c-4ab8-a9a7-41d31ebc4a60"
-					(reference "C10")
+					(reference "C18")
 					(unit 1)
 				)
@@
 		(on_board yes)
 		(dnp no)
-		(property "Reference" "C44"
+		(property "Reference" "C4"
 			(at 116.078 177.8 0)
 			(effects
@@
 			(project "sonar"
 				(path "/f72ceae0-eee4-4385-b0e8-639846bcb5f2/68d332b8-de02-4694-8619-1c5597a76eff"
-					(reference "C53")
+					(reference "C59")
 					(unit 1)
 				)
 				(path "/f72ceae0-eee4-4385-b0e8-639846bcb5f2/d78844ef-eb5d-4b24-a5c3-8824db20c2bc"
-					(reference "C44")
+					(reference "C4")
 					(unit 1)
 				)
 				(path "/f72ceae0-eee4-4385-b0e8-639846bcb5f2/dbee82a7-8e4c-4ab8-a9a7-41d31ebc4a60"
-					(reference "C7")
+					(reference "C15")
 					(unit 1)
 				)
@@
 		(on_board yes)
 		(dnp no)
-		(property "Reference" "C?"
+		(property "Reference" "C5"
 			(at 130.81 104.648 90)
 			(effects
@@
 			(project "sonar"
 				(path "/f72ceae0-eee4-4385-b0e8-639846bcb5f2/68d332b8-de02-4694-8619-1c5597a76eff"
-					(reference "C57")
+					(reference "C60")
 					(unit 1)
 				)
 				(path "/f72ceae0-eee4-4385-b0e8-639846bcb5f2/d78844ef-eb5d-4b24-a5c3-8824db20c2bc"
-					(reference "C?")
+					(reference "C5")
 					(unit 1)
 				)
 				(path "/f72ceae0-eee4-4385-b0e8-639846bcb5f2/dbee82a7-8e4c-4ab8-a9a7-41d31ebc4a60"
-					(reference "C8")
+					(reference "C16")
 					(unit 1)
 				)
@@
 		(on_board yes)
 		(dnp no)
-		(property "Reference" "C43"
+		(property "Reference" "C2"
 			(at 104.648 177.8 0)
 			(effects
@@
 			(project "sonar"
 				(path "/f72ceae0-eee4-4385-b0e8-639846bcb5f2/68d332b8-de02-4694-8619-1c5597a76eff"
-					(reference "C50")
+					(reference "C57")
 					(unit 1)
 				)
 				(path "/f72ceae0-eee4-4385-b0e8-639846bcb5f2/d78844ef-eb5d-4b24-a5c3-8824db20c2bc"
-					(reference "C43")
+					(reference "C2")
 					(unit 1)
 				)
 				(path "/f72ceae0-eee4-4385-b0e8-639846bcb5f2/dbee82a7-8e4c-4ab8-a9a7-41d31ebc4a60"
-					(reference "C5")
+					(reference "C13")
 					(unit 1)
 				)

Commit message: Switch to audio not just ultrasonic.
Parts:
- U1: footprint PM0064A-IPC_A -> Package_QFP:LQFP-64-1EP_10x10mm_P0.5mm_EP5x5mm_ThermalVias
Changed lines of the file:
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@@
 			)
 		)
-		(property "Footprint" "PM0064A-IPC_A"
+		(property "Footprint" "Package_QFP:LQFP-64-1EP_10x10mm_P0.5mm_EP5x5mm_ThermalVias"
 			(at 167.64 32.512 0)
 			(effects

Commit message: Josh cooking some more.
Parts:
- removed R3: 100k, Resistor_SMD:R_0402_1005Metric, symbol Device:R_US
- added C201, C202, C203, C204, C205, C214: 1uF, Capacitor_SMD:C_0402_1005Metric, symbol Device:C
- added C210: 470nF, Capacitor_SMD:C_0402_1005Metric, symbol Device:C
- added C213: 40uF, Capacitor_SMD:C_0402_1005Metric, symbol Device:C
- added R201: 10, Resistor_SMD:R_0402_1005Metric, symbol Device:R_US
- added R202: 100k, Resistor_SMD:R_0402_1005Metric, symbol Device:R_US
- renumbered C5 to C206, C6 to C207, C7 to C208, C8 to C209, C1 to C211, C3 to C212, C2 to C215, C4 to C216, R4 to R203, R1 to R204, R2 to R205, U1 to U201
Connections:
- net 5V: now also C201.2, C202.2, C203.2, C204.2, C205.2, C213.2
- net GND: now also U201.55 (REFN), C201.1, C202.1, C203.1, C204.1, C205.1, C210.2, C213.1, C214.1; no longer R205.2
- net at U201.56 (REFIO): now also C210.1
- net 3.3: no longer names the net of U201.25 (DVDD)
- net 3.3: now also R201.2
- net ADC_CONV_START renamed adc_conv_start
- net hw_sw_select renamed ~{hw}_sw_select
- net range_xclk renamed range_select
- net range_select: now also R202.1
- net read_allow renamed read
- net read_out_bus.par_ser_select renamed par_ser_select
- new net 3.3V: C214.2, R201.1, R202.2, R205.2
Other:
- sheet rx_amp_0 ports: added 2.75V; removed none
- sheet rx_amp_1 ports: added 2.75V; removed none
- sheet rx_amp_2 ports: added 2.75V; removed none
- sheet rx_amp_3 ports: added 2.75V; removed none
- sheet rx_amp_4 ports: added 2.75V; removed none
- sheet rx_amp_5 ports: added 2.75V; removed none
- sheet rx_amp_6 ports: added 2.75V; removed none
- sheet rx_amp_7 ports: added 2.75V; removed none
- note added: "1.4mA max draw on +2.75V rail"
- note added: "208mA max draw on +2.5V and -2.5V rails"
- note added: "50.1mA max"
- note added: "Must be placed directly next to input pins"
- note added: "NOTE: Maybe make them all switchs in case of design error"
- note added: "Set range to +-2 VREF"
- note added: "Using harware and software config with parralel readout. The software confid is to set the ref voltage to 1.25V."
- note removed: "208mA max draw on both rails"
- note removed: "Always Permit Reads"
- note removed: "DO WE NEED THESE????"
- moved on the sheet: C211, C212, C215, C216, R203, R204, R205
