File: sonar-v1-pcb/5_to_10_boost.kicad_sch (KiCad schematic)
At the start: 4 parts, among them U34 TPS55340PWP

Commit message: Switch to audio not just ultrasonic.
Parts:
- R135: footprint (none) -> Resistor_SMD:R_0402_1005Metric
- TP97, TP98: footprint (none) -> TestPoint:TestPoint_Pad_D1.0mm
- U34: footprint PWP14 -> (none)
Changed lines of the file:
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@@
 			)
 		)
-		(property "Footprint" ""
+		(property "Footprint" "Resistor_SMD:R_0402_1005Metric"
 			(at 199.136 141.224 90)
 			(effects
@@
 			)
 		)
-		(property "Footprint" ""
+		(property "Footprint" "TestPoint:TestPoint_Pad_D1.0mm"
 			(at 118.11 57.15 0)
 			(effects
@@
 			)
 		)
-		(property "Footprint" ""
+		(property "Footprint" "TestPoint:TestPoint_Pad_D1.0mm"
 			(at 198.12 49.53 0)
 			(effects
@@
 			)
 		)
-		(property "Footprint" "PWP14"
+		(property "Footprint" ""
 			(at 150.114 113.284 0)
 			(effects

Commit message: Josh cooking some more.
Parts:
- U3101: renamed from U34; footprint (none) -> PWP14
- renumbered R135 to R3101, TP98 to TP3101, TP97 to TP3102
Changed lines of the file:
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@@
 		(dnp no)
 		(fields_autoplaced yes)
-		(property "Reference" "R135"
+		(property "Reference" "R3101"
 			(at 200.66 139.6999 0)
 			(effects
@@
 			(project "sonar"
 				(path "/f72ceae0-eee4-4385-b0e8-639846bcb5f2/0971c334-b681-41ae-ad35-a89520df0687/6814f6cb-3c12-4399-b1d1-2b674ba47631"
-					(reference "R135")
+					(reference "R3101")
 					(unit 1)
 				)
@@
 		(dnp no)
 		(fields_autoplaced yes)
-		(property "Reference" "TP97"
+		(property "Reference" "TP3102"
 			(at 116.84 54.2924 0)
 			(effects
@@
 			(project ""
 				(path "/f72ceae0-eee4-4385-b0e8-639846bcb5f2/0971c334-b681-41ae-ad35-a89520df0687/6814f6cb-3c12-4399-b1d1-2b674ba47631"
-					(reference "TP97")
+					(reference "TP3102")
 					(unit 1)
 				)
@@
 		(dnp no)
 		(fields_autoplaced yes)
-		(property "Reference" "TP98"
+		(property "Reference" "TP3101"
 			(at 196.85 46.6724 0)
 			(effects
@@
 			(project ""
 				(path "/f72ceae0-eee4-4385-b0e8-639846bcb5f2/0971c334-b681-41ae-ad35-a89520df0687/6814f6cb-3c12-4399-b1d1-2b674ba47631"
-					(reference "TP98")
+					(reference "TP3101")
 					(unit 1)
 				)
@@
 		(dnp no)
 		(fields_autoplaced yes)
-		(property "Reference" "U34"
+		(property "Reference" "U3101"
 			(at 149.86 53.34 0)
 			(effects
@@
 			)
 		)
-		(property "Footprint" ""
+		(property "Footprint" "PWP14"
 			(at 150.114 113.284 0)
 			(effects
@@
 			(project "sonar"
 				(path "/f72ceae0-eee4-4385-b0e8-639846bcb5f2/0971c334-b681-41ae-ad35-a89520df0687/6814f6cb-3c12-4399-b1d1-2b674ba47631"
-					(reference "U34")
-					(unit 1)
-				)
+					(reference "U3101")
+					(unit 1)
+				)
