File: sonar-v1-pcb/inverting_buck_boost.kicad_sch (KiCad schematic)
At the start: 13 parts, among them U1 TPS63700

Commit message: Some work on the boost converter
Parts:
- added TP3501: -12V_EN, symbol Connector:TestPoint_Probe
- renumbered U1 to U3501
Connections:
- net at C3504.1, R3503.2, U3501.3 (VIN)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: now also TP3501.1
Changed lines of the file:
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@@
 	)
 	(junction
+		(at 120.65 86.36)
+		(diameter 0)
+		(color 0 0 0 0)
+	)
+	(junction
 		(at 128.27 86.36)
 		(diameter 0)
@@
 	(wire
 		(pts
+			(xy 120.65 86.36) (xy 114.3 86.36)
+		)
+		(stroke
+			(width 0)
+			(type default)
+		)
+	)
+	(wire
+		(pts
 			(xy 163.83 109.22) (xy 166.37 109.22)
 		)
@@
 	(wire
 		(pts
-			(xy 128.27 86.36) (xy 114.3 86.36)
+			(xy 128.27 86.36) (xy 120.65 86.36)
 		)
 		(stroke
@@
 		)
 		(instances
-			(project ""
+			(project "sonar"
 				(path "/f72ceae0-eee4-4385-b0e8-639846bcb5f2/0971c334-b681-41ae-ad35-a89520df0687/b540816d-de86-42bd-acdb-d7039b5ee686"
 					(reference "L3501")
@@
 		)
 		(instances
-			(project ""
+			(project "sonar"
 				(path "/f72ceae0-eee4-4385-b0e8-639846bcb5f2/0971c334-b681-41ae-ad35-a89520df0687/b540816d-de86-42bd-acdb-d7039b5ee686"
 					(reference "C3505")
@@
 		)
 		(instances
-			(project ""
+			(project "sonar"
 				(path "/f72ceae0-eee4-4385-b0e8-639846bcb5f2/0971c334-b681-41ae-ad35-a89520df0687/b540816d-de86-42bd-acdb-d7039b5ee686"
 					(reference "C3502")
@@
 		)
 		(instances
-			(project ""
+			(project "sonar"
 				(path "/f72ceae0-eee4-4385-b0e8-639846bcb5f2/0971c334-b681-41ae-ad35-a89520df0687/b540816d-de86-42bd-acdb-d7039b5ee686"
 					(reference "C3506")
@@
 		)
 		(instances
-			(project ""
+			(project "sonar"
 				(path "/f72ceae0-eee4-4385-b0e8-639846bcb5f2/0971c334-b681-41ae-ad35-a89520df0687/b540816d-de86-42bd-acdb-d7039b5ee686"
 					(reference "R3501")
@@
 		)
 		(instances
-			(project ""
+			(project "sonar"
 				(path "/f72ceae0-eee4-4385-b0e8-639846bcb5f2/0971c334-b681-41ae-ad35-a89520df0687/b540816d-de86-42bd-acdb-d7039b5ee686"
 					(reference "D3501")
@@
 		)
 		(instances
-			(project ""
+			(project "sonar"
 				(path "/f72ceae0-eee4-4385-b0e8-639846bcb5f2/0971c334-b681-41ae-ad35-a89520df0687/b540816d-de86-42bd-acdb-d7039b5ee686"
 					(reference "C3501")
@@
 		(dnp no)
 		(fields_autoplaced yes)
-		(property "Reference" "U?"
+		(property "Reference" "U3501"
 			(at 146.05 74.93 0)
 			(effects
@@
 			(project "sonar"
 				(path "/f72ceae0-eee4-4385-b0e8-639846bcb5f2/0971c334-b681-41ae-ad35-a89520df0687/b540816d-de86-42bd-acdb-d7039b5ee686"
-					(reference "U?")
+					(reference "U3501")
 					(unit 1)
 				)
@@
 		)
 		(instances
-			(project ""
+			(project "sonar"
 				(path "/f72ceae0-eee4-4385-b0e8-639846bcb5f2/0971c334-b681-41ae-ad35-a89520df0687/b540816d-de86-42bd-acdb-d7039b5ee686"
 					(reference "R3503")
@@
 	)
 	(symbol
+		(lib_id "Connector:TestPoint_Probe")
+		(at 120.65 86.36 0)
+		(unit 1)
+		(exclude_from_sim no)
+		(in_bom yes)
+		(on_board yes)
+		(dnp no)
+		(property "Reference" "TP3501"
+			(at 121.92 78.74 0)
+			(effects
+				(font
+					(size 1.27 1.27)
+				)
+			)
+		)
+		(property "Value" "-12V_EN"
+			(at 121.92 81.28 0)
+			(effects
+				(font
+					(size 1.27 1.27)
+				)
+			)
+		)
+		(property "Footprint" ""
+			(at 125.73 86.36 0)
+			(effects
+				(font
+					(size 1.27 1.27)
+				)
+				(hide yes)
+			)
+		)
+		(property "Datasheet" "~"
+			(at 125.73 86.36 0)
+			(effects
+				(font
+					(size 1.27 1.27)
+				)
+				(hide yes)
+			)
+		)
+		(property "Description" "test point (alternative probe-style design)"
+			(at 120.65 86.36 0)
+			(effects
+				(font
+					(size 1.27 1.27)
+				)
+				(hide yes)
+			)
+		)
+		(pin "1"
+		)
+		(instances
+			(project "sonar"
+				(path "/f72ceae0-eee4-4385-b0e8-639846bcb5f2/0971c334-b681-41ae-ad35-a89520df0687/b540816d-de86-42bd-acdb-d7039b5ee686"
+					(reference "TP3501")
+					(unit 1)
+				)
+			)
+		)
+	)
+	(symbol
 		(lib_id "sonar_lib:R_0603_100k")
 		(at 191.77 105.41 0)
@@
 		)
 		(instances
-			(project ""
+			(project "sonar"
 				(path "/f72ceae0-eee4-4385-b0e8-639846bcb5f2/0971c334-b681-41ae-ad35-a89520df0687/b540816d-de86-42bd-acdb-d7039b5ee686"
 					(reference "R3504")
@@
 		)
 		(instances
-			(project ""
+			(project "sonar"
 				(path "/f72ceae0-eee4-4385-b0e8-639846bcb5f2/0971c334-b681-41ae-ad35-a89520df0687/b540816d-de86-42bd-acdb-d7039b5ee686"
 					(reference "NT3501")
@@
 		)
 		(instances
-			(project ""
+			(project "sonar"
 				(path "/f72ceae0-eee4-4385-b0e8-639846bcb5f2/0971c334-b681-41ae-ad35-a89520df0687/b540816d-de86-42bd-acdb-d7039b5ee686"
 					(reference "C3504")
@@
 		)
 		(instances
-			(project ""
+			(project "sonar"
 				(path "/f72ceae0-eee4-4385-b0e8-639846bcb5f2/0971c334-b681-41ae-ad35-a89520df0687/b540816d-de86-42bd-acdb-d7039b5ee686"
 					(reference "C3503")

Commit message: some stuff i forget
Connections:
- net GND: now also C3502.2, C3506.2
- net PGND: no longer C3502.2, C3506.2
Changed lines of the file:
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@@
 	(wire
 		(pts
-			(xy 99.06 132.08) (xy 99.06 116.84)
+			(xy 99.06 127) (xy 99.06 116.84)
 		)
 		(stroke
@@
 	(wire
 		(pts
-			(xy 207.01 124.46) (xy 207.01 132.08)
+			(xy 207.01 124.46) (xy 207.01 127)
 		)
 		(stroke
@@
 	)
 	(label "PGND"
-		(at 207.01 132.08 90)
-		(effects
-			(font
-				(size 1.27 1.27)
-			)
-			(justify left bottom)
-		)
-	)
-	(label "PGND"
 		(at 163.83 132.08 90)
 		(effects
@@
 		)
 	)
-	(label "PGND"
-		(at 99.06 132.08 90)
-		(effects
-			(font
-				(size 1.27 1.27)
-			)
-			(justify left bottom)
-		)
-	)
 	(hierarchical_label "R_set_fb"
 		(shape passive)
@@
 		)
 	)
+	(hierarchical_label "GND"
+		(shape input)
+		(at 207.01 127 270)
+		(effects
+			(font
+				(size 1.27 1.27)
+			)
+			(justify right)
+		)
+	)
 	(hierarchical_label "Vin"
 		(shape input)
@@
 		)
 	)
+	(hierarchical_label "GND"
+		(shape input)
+		(at 99.06 127 270)
+		(effects
+			(font
+				(size 1.27 1.27)
+			)
+			(justify right)
+		)
+	)
