File: sonar-v1-pcb/inverting_buck_boost.kicad_sch (KiCad schematic)
At the start: 14 parts, among them U3501 TPS63700

Commit message: WIP hand-off: rx amp sim project, SPICE models, schematic updates
Adds rx_amp_sim KiCad project, SPICE models, Python setup-kicad.py
(replaces test_py.sh), CLAUDE.md, and a sweep of schematic edits across
the v1 board.

Co-Authored-By: Claude Opus 4.7 <noreply@anthropic.com>
Parts:
- renumbered C3502 to C143, C3504 to C144, C3503 to C145, C3505 to C146, C3501 to C147, C3506 to C148, D3501 to D2, L3501 to L3, NT3501 to NT2, R3503 to R142, R3501 to R143, R3504 to R144, TP3501 to TP83, U3501 to U36
Changed lines of the file:
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@@
 		(dnp no)
 		(fields_autoplaced yes)
-		(property "Reference" "L3501"
+		(property "Reference" "L3"
 			(at 166.37 119.3799 0)
 			(show_name no)
@@
 			(project "sonar"
 				(path "/f72ceae0-eee4-4385-b0e8-639846bcb5f2/0971c334-b681-41ae-ad35-a89520df0687/b540816d-de86-42bd-acdb-d7039b5ee686"
-					(reference "L3501")
+					(reference "L3")
 					(unit 1)
 				)
@@
 		(dnp no)
 		(fields_autoplaced yes)
-		(property "Reference" "C3505"
+		(property "Reference" "C146"
 			(at 195.58 96.5199 0)
 			(show_name no)
@@
 			(project "sonar"
 				(path "/f72ceae0-eee4-4385-b0e8-639846bcb5f2/0971c334-b681-41ae-ad35-a89520df0687/b540816d-de86-42bd-acdb-d7039b5ee686"
-					(reference "C3505")
+					(reference "C146")
 					(unit 1)
 				)
@@
 		(dnp no)
 		(fields_autoplaced yes)
-		(property "Reference" "C3502"
+		(property "Reference" "C143"
 			(at 102.87 111.7599 0)
 			(show_name no)
@@
 			(project "sonar"
 				(path "/f72ceae0-eee4-4385-b0e8-639846bcb5f2/0971c334-b681-41ae-ad35-a89520df0687/b540816d-de86-42bd-acdb-d7039b5ee686"
-					(reference "C3502")
+					(reference "C143")
 					(unit 1)
 				)
@@
 	)
 	(symbol
-		(lib_name "C_0603_22uF_1")
 		(lib_id "sonar_lib:C_0603_22uF")
 		(at 207.01 120.65 0)
@@
 		(dnp no)
 		(fields_autoplaced yes)
-		(property "Reference" "C3506"
+		(property "Reference" "C148"
 			(at 210.82 119.3799 0)
 			(show_name no)
@@
 			(project "sonar"
 				(path "/f72ceae0-eee4-4385-b0e8-639846bcb5f2/0971c334-b681-41ae-ad35-a89520df0687/b540816d-de86-42bd-acdb-d7039b5ee686"
-					(reference "C3506")
+					(reference "C148")
 					(unit 1)
 				)
@@
 		(dnp no)
 		(fields_autoplaced yes)
-		(property "Reference" "R3501"
+		(property "Reference" "R143"
 			(at 179.07 88.8999 0)
 			(show_name no)
@@
 			(project "sonar"
 				(path "/f72ceae0-eee4-4385-b0e8-639846bcb5f2/0971c334-b681-41ae-ad35-a89520df0687/b540816d-de86-42bd-acdb-d7039b5ee686"
-					(reference "R3501")
+					(reference "R143")
 					(unit 1)
 				)
@@
 		(in_pos_files yes)
 		(dnp no)
-		(property "Reference" "D3501"
+		(property "Reference" "D2"
 			(at 170.18 113.03 0)
 			(show_name no)
@@
 		(property "Package" "SOD-123"
 			(at 170.18 99.06 0)
+			(hide yes)
+			(show_name no)
+			(do_not_autoplace no)
+			(effects
+				(font
+					(size 1.27 1.27)
+				)
+			)
+		)
+		(property "Sim.Device" "D"
+			(at 0 0 0)
+			(hide yes)
+			(show_name no)
+			(do_not_autoplace no)
+			(effects
+				(font
+					(size 1.27 1.27)
+				)
+			)
+		)
+		(property "Sim.Name" "DSchottky580"
+			(at 0 0 0)
+			(hide yes)
+			(show_name no)
+			(do_not_autoplace no)
+			(effects
+				(font
+					(size 1.27 1.27)
+				)
+			)
+		)
+		(property "Sim.Params" "is=1e-9 rs=0.05 n=1 cjo=80p"
+			(at 0 0 0)
+			(hide yes)
+			(show_name no)
+			(do_not_autoplace no)
+			(effects
+				(font
+					(size 1.27 1.27)
+				)
+			)
+		)
+		(property "Sim.Pins" "1=K 2=A"
+			(at 0 0 0)
 			(hide yes)
 			(show_name no)
@@
 			(project "sonar"
 				(path "/f72ceae0-eee4-4385-b0e8-639846bcb5f2/0971c334-b681-41ae-ad35-a89520df0687/b540816d-de86-42bd-acdb-d7039b5ee686"
-					(reference "D3501")
+					(reference "D2")
 					(unit 1)
 				)
@@
 		(dnp no)
 		(fields_autoplaced yes)
-		(property "Reference" "C3501"
+		(property "Reference" "C147"
 			(at 210.82 90.1699 0)
 			(show_name no)
@@
 			(project "sonar"
 				(path "/f72ceae0-eee4-4385-b0e8-639846bcb5f2/0971c334-b681-41ae-ad35-a89520df0687/b540816d-de86-42bd-acdb-d7039b5ee686"
-					(reference "C3501")
+					(reference "C147")
 					(unit 1)
 				)
@@
 		(dnp no)
 		(fields_autoplaced yes)
-		(property "Reference" "U3501"
+		(property "Reference" "U36"
 			(at 146.05 74.93 0)
 			(show_name no)
@@
 			(project "sonar"
 				(path "/f72ceae0-eee4-4385-b0e8-639846bcb5f2/0971c334-b681-41ae-ad35-a89520df0687/b540816d-de86-42bd-acdb-d7039b5ee686"
-					(reference "U3501")
+					(reference "U36")
 					(unit 1)
 				)
@@
 		(dnp no)
 		(fields_autoplaced yes)
-		(property "Reference" "R3503"
+		(property "Reference" "R142"
 			(at 106.68 80.01 90)
 			(show_name no)
@@
 			(project "sonar"
 				(path "/f72ceae0-eee4-4385-b0e8-639846bcb5f2/0971c334-b681-41ae-ad35-a89520df0687/b540816d-de86-42bd-acdb-d7039b5ee686"
-					(reference "R3503")
+					(reference "R142")
 					(unit 1)
 				)
@@
 		(unit 1)
 		(body_style 1)
-		(exclude_from_sim no)
+		(exclude_from_sim yes)
 		(in_bom yes)
 		(on_board yes)
 		(in_pos_files yes)
 		(dnp no)
-		(property "Reference" "TP3501"
+		(property "Reference" "TP83"
 			(at 121.92 78.74 0)
 			(show_name no)
@@
 			(project "sonar"
 				(path "/f72ceae0-eee4-4385-b0e8-639846bcb5f2/0971c334-b681-41ae-ad35-a89520df0687/b540816d-de86-42bd-acdb-d7039b5ee686"
-					(reference "TP3501")
+					(reference "TP83")
 					(unit 1)
 				)
@@
 		(dnp no)
 		(fields_autoplaced yes)
-		(property "Reference" "R3504"
+		(property "Reference" "R144"
 			(at 194.31 104.1399 0)
 			(show_name no)
@@
 			(project "sonar"
 				(path "/f72ceae0-eee4-4385-b0e8-639846bcb5f2/0971c334-b681-41ae-ad35-a89520df0687/b540816d-de86-42bd-acdb-d7039b5ee686"
-					(reference "R3504")
+					(reference "R144")
 					(unit 1)
 				)
@@
 		(dnp no)
 		(fields_autoplaced yes)
-		(property "Reference" "NT3501"
+		(property "Reference" "NT2"
 			(at 146.05 156.21 0)
 			(show_name no)
@@
 			(project "sonar"
 				(path "/f72ceae0-eee4-4385-b0e8-639846bcb5f2/0971c334-b681-41ae-ad35-a89520df0687/b540816d-de86-42bd-acdb-d7039b5ee686"
-					(reference "NT3501")
+					(reference "NT2")
 					(unit 1)
 				)
@@
 		(dnp no)
 		(fields_autoplaced yes)
-		(property "Reference" "C3504"
+		(property "Reference" "C144"
 			(at 118.11 90.1699 0)
 			(show_name no)
@@
 			(project "sonar"
 				(path "/f72ceae0-eee4-4385-b0e8-639846bcb5f2/0971c334-b681-41ae-ad35-a89520df0687/b540816d-de86-42bd-acdb-d7039b5ee686"
-					(reference "C3504")
+					(reference "C144")
 					(unit 1)
 				)
@@
 		(dnp no)
 		(fields_autoplaced yes)
-		(property "Reference" "C3503"
+		(property "Reference" "C145"
 			(at 121.92 111.7599 0)
 			(show_name no)
@@
 			(project "sonar"
 				(path "/f72ceae0-eee4-4385-b0e8-639846bcb5f2/0971c334-b681-41ae-ad35-a89520df0687/b540816d-de86-42bd-acdb-d7039b5ee686"
-					(reference "C3503")
+					(reference "C145")
 					(unit 1)
 				)
