File: sonar-v1-pcb/5v_to_12v_boost.kicad_sch (KiCad schematic)
At the start: 0 parts

Commit message: Some work on the boost converter
Parts:
- added NT3301: NetTie_2, NetTie:NetTie-2_SMD_Pad0.5mm, symbol sonar_lib:NetTie_2
- added R3301: 78.7k, Sonar:R_0603_1608Metric, symbol sonar_lib:R_0603_78.7k
- added U3301: TPS55340PWPR, Sonar:Texas_HTSSOP-14-1EP_4.4x5mm_P0.65mm_EP3.4x5mm_Mask3.155x3.255mm, symbol sonar_lib:TPS55340PWPR
Connections:
- new net: U3301.1 (SW), U3301.2 (SW)
- new net: R3301.1, U3301.10 (FREQ)
- new net GND: NT3301.1, R3301.2, U3301.11 (NC), U3301.15 (EP), U3301.6 (SYNC), U3301.7 (AGND)
- new net PGND: NT3301.2, U3301.12 (PGND), U3301.13 (PGND), U3301.14 (PGND)
Other:
- title: (none) -> Vin to 12V Boost

Commit message: some stuff i forget
Parts:
- added C3301: 47nF, Sonar:C_0603_1608Metric, symbol sonar_lib:C_0603_47nF
- added C3302, C3303: 4.7uF, Sonar:C_0603_1608Metric, symbol sonar_lib:C_0603_4.7uF
- added D3301: 550mV, 3A, Sonar:D_SMA, symbol sonar_lib:D_Schottky_550mV_3A
- added L3301: 27uH, Sonar:L_12x12mm_H8mm, symbol sonar_lib:L_12x12mm_27uH
- added R3302: 10k, Sonar:R_0603_1608Metric, symbol sonar_lib:R_0603_10k
- added R3303: 86.6k, Sonar:R_0603_1608Metric, symbol sonar_lib:R_0603_86.6k
Connections:
- net GND: now also C3301.2, C3302.2, C3303.2, R3302.2
- net at U3301.1 (SW), U3301.2 (SW): now also D3301.2 (A), L3301.2
- net Vin: now reaches U3301.3 (VIN)
- net Vin: now also U3301.4 (EN), C3302.1, L3301.1
- net at U3301.5 (SS): now also C3301.1
- net at U3301.9 (FB): now also R3302.1, R3303.2
- new net Vout: C3303.1, D3301.1 (K), R3303.1
Other:
- moved on the sheet: NT3301, R3301, U3301
