File: sonar-v1-pcb/5v_to_12v_boost.kicad_sch (KiCad schematic)
At the start: 10 parts, among them U3301 TPS55340PWPR

Commit message: WIP hand-off: rx amp sim project, SPICE models, schematic updates
Adds rx_amp_sim KiCad project, SPICE models, Python setup-kicad.py
(replaces test_py.sh), CLAUDE.md, and a sweep of schematic edits across
the v1 board.

Co-Authored-By: Claude Opus 4.7 <noreply@anthropic.com>
Parts:
- renumbered C3302 to C140, C3301 to C141, C3303 to C142, D3301 to D1, L3301 to L2, NT3301 to NT1, R3301 to R139, R3303 to R140, R3302 to R141, U3301 to U35
Changed lines of the file:
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@@
 		(dnp no)
 		(fields_autoplaced yes)
-		(property "Reference" "C3302"
+		(property "Reference" "C140"
 			(at 119.38 96.5199 0)
 			(show_name no)
@@
 			(project "sonar"
 				(path "/f72ceae0-eee4-4385-b0e8-639846bcb5f2/0971c334-b681-41ae-ad35-a89520df0687/3221bd23-5073-46fa-ae01-536305e89f25"
-					(reference "C3302")
+					(reference "C140")
 					(unit 1)
 				)
@@
 		(dnp no)
 		(fields_autoplaced yes)
-		(property "Reference" "L3301"
+		(property "Reference" "L2"
 			(at 153.67 85.09 90)
 			(show_name no)
@@
 			(project "sonar"
 				(path "/f72ceae0-eee4-4385-b0e8-639846bcb5f2/0971c334-b681-41ae-ad35-a89520df0687/3221bd23-5073-46fa-ae01-536305e89f25"
-					(reference "L3301")
+					(reference "L2")
 					(unit 1)
 				)
@@
 		(dnp no)
 		(fields_autoplaced yes)
-		(property "Reference" "U3301"
+		(property "Reference" "U35"
 			(at 153.67 93.98 0)
 			(show_name no)
@@
 		)
 		(property "Sim.Library" "/home/george-sleen/Documents/projects/gs-kicad-lib/spice-models/TPS55340/TPS55340_TRANS_ngspice.lib"
+			(at 153.67 72.39 0)
+			(hide yes)
+			(show_name no)
+			(do_not_autoplace no)
+			(effects
+				(font
+					(size 1.27 1.27)
+				)
+			)
+		)
+		(property "Sim.Device" "SUBCKT"
+			(at 153.67 72.39 0)
+			(hide yes)
+			(show_name no)
+			(do_not_autoplace no)
+			(effects
+				(font
+					(size 1.27 1.27)
+				)
+			)
+		)
+		(property "Sim.Name" "TPS55340_TRANS"
+			(at 153.67 72.39 0)
+			(hide yes)
+			(show_name no)
+			(do_not_autoplace no)
+			(effects
+				(font
+					(size 1.27 1.27)
+				)
+			)
+		)
+		(property "Sim.Pins" "1=SW_0 2=SW_1 15=PWPD 1=SW_2 3=VIN 4=EN 5=SS 6=SYNC 7=AGND 11=NC_0 12=PGND_0 13=PGND_1 14=PGND_2 11=NC_1 10=FREQ 9=FB 8=COMP"
 			(at 153.67 72.39 0)
 			(hide yes)
@@
 			(project "sonar"
 				(path "/f72ceae0-eee4-4385-b0e8-639846bcb5f2/0971c334-b681-41ae-ad35-a89520df0687/3221bd23-5073-46fa-ae01-536305e89f25"
-					(reference "U3301")
+					(reference "U35")
 					(unit 1)
 				)
@@
 		(dnp no)
 		(fields_autoplaced yes)
-		(property "Reference" "D3301"
+		(property "Reference" "D1"
 			(at 180.6575 83.82 0)
 			(show_name no)
@@
 		(property "Package" "SMA"
 			(at 180.34 100.33 0)
+			(hide yes)
+			(show_name no)
+			(do_not_autoplace no)
+			(effects
+				(font
+					(size 1.27 1.27)
+				)
+			)
+		)
+		(property "Sim.Device" "D"
+			(at 0 0 0)
+			(hide yes)
+			(show_name no)
+			(do_not_autoplace no)
+			(effects
+				(font
+					(size 1.27 1.27)
+				)
+			)
+		)
+		(property "Sim.Name" "DSchottky550"
+			(at 0 0 0)
+			(hide yes)
+			(show_name no)
+			(do_not_autoplace no)
+			(effects
+				(font
+					(size 1.27 1.27)
+				)
+			)
+		)
+		(property "Sim.Params" "is=1e-8 rs=0.02 n=1 cjo=200p"
+			(at 0 0 0)
+			(hide yes)
+			(show_name no)
+			(do_not_autoplace no)
+			(effects
+				(font
+					(size 1.27 1.27)
+				)
+			)
+		)
+		(property "Sim.Pins" "1=K 2=A"
+			(at 0 0 0)
 			(hide yes)
 			(show_name no)
@@
 			(project "sonar"
 				(path "/f72ceae0-eee4-4385-b0e8-639846bcb5f2/0971c334-b681-41ae-ad35-a89520df0687/3221bd23-5073-46fa-ae01-536305e89f25"
-					(reference "D3301")
+					(reference "D1")
 					(unit 1)
 				)
@@
 		(dnp no)
 		(fields_autoplaced yes)
-		(property "Reference" "NT3301"
+		(property "Reference" "NT1"
 			(at 140.97 161.29 0)
 			(show_name no)
@@
 			(project "sonar"
 				(path "/f72ceae0-eee4-4385-b0e8-639846bcb5f2/0971c334-b681-41ae-ad35-a89520df0687/3221bd23-5073-46fa-ae01-536305e89f25"
-					(reference "NT3301")
+					(reference "NT1")
 					(unit 1)
 				)
@@
 		(dnp no)
 		(fields_autoplaced yes)
-		(property "Reference" "R3303"
+		(property "Reference" "R140"
 			(at 195.58 109.2199 0)
 			(show_name no)
@@
 			(project "sonar"
 				(path "/f72ceae0-eee4-4385-b0e8-639846bcb5f2/0971c334-b681-41ae-ad35-a89520df0687/3221bd23-5073-46fa-ae01-536305e89f25"
-					(reference "R3303")
+					(reference "R140")
 					(unit 1)
 				)
@@
 		(dnp no)
 		(fields_autoplaced yes)
-		(property "Reference" "C3301"
+		(property "Reference" "C141"
 			(at 119.38 124.4599 0)
 			(show_name no)
@@
 			(project "sonar"
 				(path "/f72ceae0-eee4-4385-b0e8-639846bcb5f2/0971c334-b681-41ae-ad35-a89520df0687/3221bd23-5073-46fa-ae01-536305e89f25"
-					(reference "C3301")
+					(reference "C141")
 					(unit 1)
 				)
@@
 		(dnp no)
 		(fields_autoplaced yes)
-		(property "Reference" "C3303"
+		(property "Reference" "C142"
 			(at 210.82 96.5199 0)
 			(show_name no)
@@
 			(project "sonar"
 				(path "/f72ceae0-eee4-4385-b0e8-639846bcb5f2/0971c334-b681-41ae-ad35-a89520df0687/3221bd23-5073-46fa-ae01-536305e89f25"
-					(reference "C3303")
+					(reference "C142")
 					(unit 1)
 				)
@@
 		(dnp no)
 		(fields_autoplaced yes)
-		(property "Reference" "R3302"
+		(property "Reference" "R141"
 			(at 195.58 116.8399 0)
 			(show_name no)
@@
 			(project "sonar"
 				(path "/f72ceae0-eee4-4385-b0e8-639846bcb5f2/0971c334-b681-41ae-ad35-a89520df0687/3221bd23-5073-46fa-ae01-536305e89f25"
-					(reference "R3302")
+					(reference "R141")
 					(unit 1)
 				)
@@
 		(dnp no)
 		(fields_autoplaced yes)
-		(property "Reference" "R3301"
+		(property "Reference" "R139"
 			(at 130.81 124.4599 0)
 			(show_name no)
@@
 			(project "sonar"
 				(path "/f72ceae0-eee4-4385-b0e8-639846bcb5f2/0971c334-b681-41ae-ad35-a89520df0687/3221bd23-5073-46fa-ae01-536305e89f25"
-					(reference "R3301")
+					(reference "R139")
 					(unit 1)
 				)
