File: sonar-v1-pcb/5v_to_12v_boost.kicad_sch (KiCad schematic)
At the start: 10 parts, among them U35 TPS55340PWPR

Commit message: T-012: prune power tree to four rails (drop 6 legacy sheets, rewire supply/top)
Parts:
- added C261: 4.7nF, Sonar:C_0603_1608Metric, symbol sonar_lib:C_0603_4.7nF
- added R163: 10k, Sonar:R_0603_1608Metric, symbol sonar_lib:R_0603_10k
- added R164: 100k, Sonar:R_0603_1608Metric, symbol sonar_lib:R_0603_100k
Connections:
- net GND: now also C261.2
- net Vin: no longer U35.4 (EN)
- net at U35.8 (COMP): now also R163.1
- new net: C261.1, R163.2
- new net: R164.2, U35.4 (EN)
- new net +3.3V: R164.1
