File: sonar-v1-pcb/power_mux.kicad_sch (KiCad schematic)
At the start: 0 parts

Commit message: Do some more power work and add a few components
Other:
- added sheet ideal_diode0 (ideal_diode.kicad_sch)
- added sheet ideal_diode1 (ideal_diode.kicad_sch)
- title: (none) -> Power MUX
