File: sonar-v1-pcb/-10v_negative_ldo.kicad_sch (KiCad schematic)
At the start: 5 parts, among them U2906 LM337IMPX-TP

Commit message: WIP hand-off: rx amp sim project, SPICE models, schematic updates
Adds rx_amp_sim KiCad project, SPICE models, Python setup-kicad.py
(replaces test_py.sh), CLAUDE.md, and a sweep of schematic edits across
the v1 board.

Co-Authored-By: Claude Opus 4.7 <noreply@anthropic.com>
Parts:
- renumbered C3802 to C149, C3801 to C150, R3802 to R149, R3801 to R150, U2906 to U39
Changed lines of the file:
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@@
 		(dnp no)
 		(fields_autoplaced yes)
-		(property "Reference" "C3801"
+		(property "Reference" "C150"
 			(at 132.08 58.4199 0)
 			(show_name no)
@@
 			(project "sonar"
 				(path "/f72ceae0-eee4-4385-b0e8-639846bcb5f2/0971c334-b681-41ae-ad35-a89520df0687/9158f2d6-597a-4405-857f-4829a945af57"
-					(reference "C3801")
+					(reference "C150")
 					(unit 1)
 				)
@@
 		(dnp no)
 		(fields_autoplaced yes)
-		(property "Reference" "C3802"
+		(property "Reference" "C149"
 			(at 85.09 58.4199 0)
 			(show_name no)
@@
 			(project "sonar"
 				(path "/f72ceae0-eee4-4385-b0e8-639846bcb5f2/0971c334-b681-41ae-ad35-a89520df0687/9158f2d6-597a-4405-857f-4829a945af57"
-					(reference "C3802")
+					(reference "C149")
 					(unit 1)
 				)
@@
 		(in_pos_files yes)
 		(dnp no)
-		(property "Reference" "R3801"
+		(property "Reference" "R150"
 			(at 115.57 63.4999 0)
 			(show_name no)
@@
 			(project "sonar"
 				(path "/f72ceae0-eee4-4385-b0e8-639846bcb5f2/0971c334-b681-41ae-ad35-a89520df0687/9158f2d6-597a-4405-857f-4829a945af57"
-					(reference "R3801")
+					(reference "R150")
 					(unit 1)
 				)
@@
 		(dnp no)
 		(fields_autoplaced yes)
-		(property "Reference" "U2906"
+		(property "Reference" "U39"
 			(at 100.33 76.2 0)
 			(show_name no)
@@
 			(project "sonar"
 				(path "/f72ceae0-eee4-4385-b0e8-639846bcb5f2/0971c334-b681-41ae-ad35-a89520df0687/9158f2d6-597a-4405-857f-4829a945af57"
-					(reference "U2906")
+					(reference "U39")
 					(unit 1)
 				)
@@
 		(in_pos_files yes)
 		(dnp no)
-		(property "Reference" "R3802"
+		(property "Reference" "R149"
 			(at 115.57 53.3399 0)
 			(show_name no)
@@
 			(project "sonar"
 				(path "/f72ceae0-eee4-4385-b0e8-639846bcb5f2/0971c334-b681-41ae-ad35-a89520df0687/9158f2d6-597a-4405-857f-4829a945af57"
-					(reference "R3802")
+					(reference "R149")
 					(unit 1)
 				)
