File: sonar-v1-pcb/2.75V_ldo.kicad_sch (KiCad schematic)
At the start: 5 parts, among them U4 AP2127K-ADJTRG1

Commit message: WIP hand-off: rx amp sim project, SPICE models, schematic updates
Adds rx_amp_sim KiCad project, SPICE models, Python setup-kicad.py
(replaces test_py.sh), CLAUDE.md, and a sweep of schematic edits across
the v1 board.

Co-Authored-By: Claude Opus 4.7 <noreply@anthropic.com>
Parts:
- renumbered C2 to C151, C5 to C152, R8 to R151, R7 to R152, U4 to U40
Changed lines of the file:
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@@
 		(dnp no)
 		(fields_autoplaced yes)
-		(property "Reference" "#PWR019"
+		(property "Reference" "#PWR015"
 			(at 125.73 88.9 0)
 			(hide yes)
@@
 			(project "sonar"
 				(path "/f72ceae0-eee4-4385-b0e8-639846bcb5f2/0971c334-b681-41ae-ad35-a89520df0687/ee73137f-d5eb-4789-88c4-4482e951aa01"
-					(reference "#PWR019")
+					(reference "#PWR015")
 					(unit 1)
 				)
@@
 		(dnp no)
 		(fields_autoplaced yes)
-		(property "Reference" "#PWR017"
+		(property "Reference" "#PWR013"
 			(at 74.93 88.9 0)
 			(hide yes)
@@
 			(project "sonar"
 				(path "/f72ceae0-eee4-4385-b0e8-639846bcb5f2/0971c334-b681-41ae-ad35-a89520df0687/ee73137f-d5eb-4789-88c4-4482e951aa01"
-					(reference "#PWR017")
+					(reference "#PWR013")
 					(unit 1)
 				)
@@
 		(dnp no)
 		(fields_autoplaced yes)
-		(property "Reference" "#PWR014"
+		(property "Reference" "#PWR012"
 			(at 62.23 71.12 0)
 			(hide yes)
@@
 			(project "sonar"
 				(path "/f72ceae0-eee4-4385-b0e8-639846bcb5f2/0971c334-b681-41ae-ad35-a89520df0687/ee73137f-d5eb-4789-88c4-4482e951aa01"
-					(reference "#PWR014")
+					(reference "#PWR012")
 					(unit 1)
 				)
@@
 		(in_pos_files yes)
 		(dnp no)
-		(property "Reference" "C2"
+		(property "Reference" "C151"
 			(at 71.12 74.9299 0)
 			(show_name no)
@@
 			(project "sonar"
 				(path "/f72ceae0-eee4-4385-b0e8-639846bcb5f2/0971c334-b681-41ae-ad35-a89520df0687/ee73137f-d5eb-4789-88c4-4482e951aa01"
-					(reference "C2")
+					(reference "C151")
 					(unit 1)
 				)
@@
 		(dnp no)
 		(fields_autoplaced yes)
-		(property "Reference" "#PWR012"
+		(property "Reference" "#PWR011"
 			(at 43.18 88.9 0)
 			(hide yes)
@@
 			(project "sonar"
 				(path "/f72ceae0-eee4-4385-b0e8-639846bcb5f2/0971c334-b681-41ae-ad35-a89520df0687/ee73137f-d5eb-4789-88c4-4482e951aa01"
-					(reference "#PWR012")
+					(reference "#PWR011")
 					(unit 1)
 				)
@@
 		(dnp no)
 		(fields_autoplaced yes)
-		(property "Reference" "#PWR015"
+		(property "Reference" "#PWR017"
 			(at 156.21 71.12 0)
 			(hide yes)
@@
 			(project "sonar"
 				(path "/f72ceae0-eee4-4385-b0e8-639846bcb5f2/0971c334-b681-41ae-ad35-a89520df0687/ee73137f-d5eb-4789-88c4-4482e951aa01"
-					(reference "#PWR015")
+					(reference "#PWR017")
 					(unit 1)
 				)
@@
 		(in_pos_files yes)
 		(dnp no)
-		(property "Reference" "U4"
+		(property "Reference" "U40"
 			(at 102.87 60.96 0)
 			(show_name no)
@@
 			(project "sonar"
 				(path "/f72ceae0-eee4-4385-b0e8-639846bcb5f2/0971c334-b681-41ae-ad35-a89520df0687/ee73137f-d5eb-4789-88c4-4482e951aa01"
-					(reference "U4")
+					(reference "U40")
 					(unit 1)
 				)
@@
 		(dnp no)
 		(fields_autoplaced yes)
-		(property "Reference" "#PWR09"
+		(property "Reference" "#PWR014"
 			(at 102.87 88.9 0)
 			(hide yes)
@@
 			(project "sonar"
 				(path "/f72ceae0-eee4-4385-b0e8-639846bcb5f2/0971c334-b681-41ae-ad35-a89520df0687/ee73137f-d5eb-4789-88c4-4482e951aa01"
-					(reference "#PWR09")
+					(reference "#PWR014")
 					(unit 1)
 				)
@@
 		(in_pos_files yes)
 		(dnp no)
-		(property "Reference" "C5"
+		(property "Reference" "C152"
 			(at 139.7 74.9299 0)
 			(show_name no)
@@
 			(project "sonar"
 				(path "/f72ceae0-eee4-4385-b0e8-639846bcb5f2/0971c334-b681-41ae-ad35-a89520df0687/ee73137f-d5eb-4789-88c4-4482e951aa01"
-					(reference "C5")
+					(reference "C152")
 					(unit 1)
 				)
@@
 		(dnp no)
 		(fields_autoplaced yes)
-		(property "Reference" "R8"
+		(property "Reference" "R151"
 			(at 128.27 69.8499 0)
 			(show_name no)
@@
 			(project "sonar"
 				(path "/f72ceae0-eee4-4385-b0e8-639846bcb5f2/0971c334-b681-41ae-ad35-a89520df0687/ee73137f-d5eb-4789-88c4-4482e951aa01"
-					(reference "R8")
+					(reference "R151")
 					(unit 1)
 				)
@@
 		(dnp no)
 		(fields_autoplaced yes)
-		(property "Reference" "R7"
+		(property "Reference" "R152"
 			(at 128.27 77.4699 0)
 			(show_name no)
@@
 			(project "sonar"
 				(path "/f72ceae0-eee4-4385-b0e8-639846bcb5f2/0971c334-b681-41ae-ad35-a89520df0687/ee73137f-d5eb-4789-88c4-4482e951aa01"
-					(reference "R7")
+					(reference "R152")
 					(unit 1)
 				)
@@
 		(dnp no)
 		(fields_autoplaced yes)
-		(property "Reference" "#PWR018"
+		(property "Reference" "#PWR016"
 			(at 143.51 88.9 0)
 			(hide yes)
@@
 			(project "sonar"
 				(path "/f72ceae0-eee4-4385-b0e8-639846bcb5f2/0971c334-b681-41ae-ad35-a89520df0687/ee73137f-d5eb-4789-88c4-4482e951aa01"
-					(reference "#PWR018")
-					(unit 1)
-				)
+					(reference "#PWR016")
+					(unit 1)
+				)
