File: sonar-v1-pcb/2.75V_ldo.kicad_sch (KiCad schematic)
At the start: 5 parts, among them U40 AP2127K-ADJTRG1

Commit message: Do some power work
Other:
- moved on the sheet: C151, C152, R151, R152, U40
