File: sonar-v1-pcb/power_supply.kicad_sch (KiCad schematic)
At the start: 30 parts, among them SW2901 SW_SPDT, U2901 TPS7A2033DQN, U2902 TPS7A2028DQN, U2903 TPS62912, U2904 TPS7A205DQN, U2905 TPS7A91

Commit message: WIP hand-off: rx amp sim project, SPICE models, schematic updates
Adds rx_amp_sim KiCad project, SPICE models, Python setup-kicad.py
(replaces test_py.sh), CLAUDE.md, and a sweep of schematic edits across
the v1 board.

Co-Authored-By: Claude Opus 4.7 <noreply@anthropic.com>
Parts:
- removed C2901, C2902, C2914, C2915: 1uF, Capacitor_SMD:C_0402_1005Metric, symbol Device:C
- removed C2903, C2904: 1uF, symbol Device:C
- removed C2905, C2906, C2907, C2908, C2909: 22uF, Capacitor_SMD:C_0402_1005Metric, symbol Device:C
- removed C2910: 470nF, Capacitor_SMD:C_0402_1005Metric, symbol Device:C
- removed C2911: 2.2nF, Capacitor_SMD:C_0402_1005Metric, symbol Device:C
- removed C2912, C2913: 10uF, Capacitor_SMD:C_0402_1005Metric, symbol Device:C
- removed C2917: 0.1uF, Capacitor_SMD:C_0402_1005Metric, symbol Device:C
- removed FB2901: FerriteBead, symbol Device:FerriteBead
- removed L2901: 2.2uH, Inductor_SMD:L_0402_1005Metric, symbol Device:L
- removed SW2901: SW_SPDT, symbol Switch:SW_SPDT
- removed TP2901, TP2902, TP2905, TP2907: TestPoint_Probe, TestPoint:TestPoint_Pad_D1.0mm, symbol Connector:TestPoint_Probe
- removed U2901: TPS7A2033DQN, Package_SON:Texas_X2SON-4_1x1mm_P0.65mm, symbol Regulator_Linear:TPS7A20xxxDQN
- removed U2902: TPS7A2028DQN, Package_SON:Texas_X2SON-4_1x1mm_P0.65mm, symbol Regulator_Linear:TPS7A20xxxDQN
- removed U2903: TPS62912, Package_DFN_QFN:Texas_RPU0010A_VQFN-HR-10_2x2mm_P0.5mm, symbol Regulator_Switching:TPS62912
- removed U2904: TPS7A205DQN, Package_SON:Texas_X2SON-4_1x1mm_P0.65mm, symbol Regulator_Linear:TPS7A20xxxDQN
- removed U2905: TPS7A91, Package_DFN_QFN:Texas_S-PDSO-N10_EP1.2x2mm, symbol Regulator_Linear:TPS7A91
- renumbered R2901 to R138, TP2903 to TP78
Other:
- note removed: "600mA required for 2.5V bus, so use a TPS7A91 instead"
- note removed: "Holy fucking yikes is this gonna be a mess"
- note removed: "Holy lost in the sauce... I am gonna let you fix this one George"
- note removed: "Max 1.5mA from audio RX"
- note removed: "Max 150mA from ADC AVDD"
- note removed: "TODO: design the feedback loop"
- note removed: "TPS629210 to buck down to 4V"
- note removed: "TPS629210 to buck down to 5.5V"
- note removed: "TPS7A20 looks sick as fuck for an LDO"
- note removed: "TPS7A30 NEGTAIVE LDO for -2.5V"
- note removed: "look at https://www.ti.com/lit/an/sbva042/sbva042.pdf?ts=1773012729035 before connecting to the LDOs"
