File: sonar-v1-pcb/ideal_diode.kicad_sch (KiCad schematic)
At the start: 7 parts, among them Q1 AO3415, U37 DZDH0401DW-7

Commit message: T-012: prune power tree to four rails (drop 6 legacy sheets, rewire supply/top)
Parts:
- U37: footprint GS_SO:SOT-363_SC-70-6 -> Package_TO_SOT_SMD:SOT-363_SC-70-6; symbol GS_PMIC:DZDH0401DW-7 -> sonar_lib:DZDH0401DW-7
Changed lines of the file:
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@@
 	)
 	(symbol
-		(lib_id "GS_PMIC:DZDH0401DW-7")
+		(lib_id "sonar_lib:DZDH0401DW-7")
 		(at 110.49 59.69 0)
 		(unit 1)
@@
 			)
 		)
-		(property "Footprint" "GS_SO:SOT-363_SC-70-6"
+		(property "Footprint" "Package_TO_SOT_SMD:SOT-363_SC-70-6"
 			(at 110.49 21.59 0)
 			(hide yes)
