File: spikes/eda-zener/deep-port/sonar_v1_deep_port/layout/layout.kicad_pcb (KiCad board)
At the start: 4 copper layers, 67 parts, among them J1 1935161, U1 OPA4171IDR, U2 AP63301WU-7, U3 DRV8876PWPR

Commit message: T-017 session 2: authenticated BOM coverage survey, registry swap, verdict strengthens
Parts:
- U1: value OPA4171IDR -> OPA4171AIDR; footprint localhost_sonar_deep-port_footprints:SOIC-14_3.9x8.7mm_P1.27mm -> localhost_sonar_deep-port_components_registry_OPA4171AIDR:lcsc
- U2: footprint localhost_sonar_deep-port_footprints:TSOT-23-6 -> localhost_sonar_deep-port_components_registry_AP63301WU-7:lcsc
- U3: footprint localhost_sonar_deep-port_footprints:HTSSOP-16-1EP_4.4x5mm_P0.65mm_EP3.4x5mm_Mask2.46x2.31mm -> localhost_sonar_deep-port_components_registry_DRV8876PWPR:lcsc
